Commit message: update grippers config

File: xacro/grippers.xacro (robot description, xacro)
@@ -32,6 +32,6 @@
         <xacro:if value="${type == 'rg75'}">
             <xacro:include filename="$(find jodell_description)/xacro/RG75-300.xacro"/>
-            <xacro:RG75-300 name="left" use_flange="true"/>
-            <xacro:RG75-300 name="right" use_flange="true"/>
+            <xacro:RG75-300 name="left" use_flange="true" pad="leapmotor"/>
+            <xacro:RG75-300 name="right" use_flange="true" pad="leapmotor"/>
             <joint name="left_gripper_base_joint" type="fixed">
                 <parent link="left_tcp"/>

File: xacro/ros2_control/robot.xacro (robot description, xacro)
@@ -13,4 +13,18 @@
 			<xacro:m6_interfaces name="left"/>
 			<xacro:m6_interfaces name="right"/>
+			<xacro:if value="${'$(arg type)' != ''}">
+				<joint name="left_gripper_joint">
+					<command_interface name="position"/>
+					<state_interface name="position">
+						<param name="initial_value">0</param>
+					</state_interface>
+				</joint>
+				<joint name="right_gripper_joint">
+					<command_interface name="position"/>
+					<state_interface name="position">
+						<param name="initial_value">0</param>
+					</state_interface>
+				</joint>
+			</xacro:if>
 		</ros2_control>
 		<ros2_control name="juxie_body" type="system">
