Commit message: Update configuration and documentation

File: xacro/body.xacro (robot description, xacro)
@@ -115,5 +115,5 @@
 		<parent link="body_link2" />
 		<child link="body_link3" />
-		<axis xyz="0 -1 0" />
+		<axis xyz="0 1 0" />
 		<limit lower="-1.745" upper="1.745" effort="100" velocity="1" />
 	</joint>

File: xacro/ros2_control/body.xacro (robot description, xacro)
@@ -7,5 +7,5 @@
       <state_interface name="position"/>
       <state_interface name="velocity"/>
-      <state_interface name="effort"/>
+      <!-- <state_interface name="effort"/> -->
     </joint>
     <joint name="body_joint2">
@@ -13,5 +13,5 @@
       <state_interface name="position"/>
       <state_interface name="velocity"/>
-      <state_interface name="effort"/>
+      <!-- <state_interface name="effort"/> -->
     </joint>
     <joint name="body_joint3">
@@ -19,5 +19,5 @@
       <state_interface name="position"/>
       <state_interface name="velocity"/>
-      <state_interface name="effort"/>
+      <!-- <state_interface name="effort"/> -->
     </joint>
     <joint name="body_joint4">
@@ -25,7 +25,7 @@
       <state_interface name="position"/>
       <state_interface name="velocity"/>
-      <state_interface name="effort"/>
+      <!-- <state_interface name="effort"/> -->
     </joint>
-    <joint name="head_joint1">
+    <!-- <joint name="head_joint1">
       <command_interface name="position"/>
       <state_interface name="position"/>
@@ -38,5 +38,5 @@
       <state_interface name="velocity"/>
       <state_interface name="effort"/>
-    </joint>
+    </joint> -->
   </xacro:macro>
 </robot>

File: xacro/ros2_control/robot.xacro (robot description, xacro)
@@ -1,38 +1,63 @@
 <?xml version="1.0"?>
 <robot name="fiveages_w2" xmlns:xacro="http://www.ros.org/wiki/xacro">
-	<xacro:arg name="ros2_control_hardware_type" default="mock_components"/>
-	<xacro:include filename="$(find fiveages_w2_description)/xacro/robot.xacro"/>
-	<xacro:include filename="$(find m6_ccs_description)/xacro/ros2_control/interfaces.xacro"/>
-	<xacro:include filename="$(find fiveages_w2_description)/xacro/ros2_control/body.xacro"/>
-	<!-- <xacro:include filename="$(find fiveages_w2_description)/xacro/ros2_control/chassis.xacro"/> -->
-	<ros2_control name="fiveages_w2_system" type="system">
-		<hardware>
-			<xacro:if value="${'$(arg ros2_control_hardware_type)' == 'gz'}">
-				<plugin>gz_ros2_control/GazeboSimSystem</plugin>
-			</xacro:if>
-			<xacro:if value="${'$(arg ros2_control_hardware_type)' == 'mock_components'}">
-				<plugin>mock_components/GenericSystem</plugin>
-			</xacro:if>
-			<xacro:if value="${'$(arg ros2_control_hardware_type)' == 'isaac'}">
-				<plugin>topic_based_ros2_control/TopicBasedSystem</plugin>
-				<param name="joint_commands_topic">/isaac/joint_command</param>
-				<param name="joint_states_topic">/isaac/joint_states</param>
-				<param name="sum_wrapped_joint_states">false</param>
-				<param name="initialize_commands_from_state">true</param>
-			</xacro:if>
-		</hardware>
-		<xacro:body_interfaces/>
-		<xacro:m6_interfaces name="left"/>
-		<xacro:m6_interfaces name="right"/>
-	</ros2_control>
-	<!-- Gazebo plugin configuration -->
-	<xacro:arg name="gazebo" default="false"/>
-	<xacro:if value="$(arg gazebo)">
-		<xacro:property name="ros2_control_config_basename" value="ros2_controllers.yaml"/>
-		<gazebo>
-			<plugin filename="gz_ros2_control-system" name="gz_ros2_control::GazeboSimROS2ControlPlugin">
-				<parameters>$(find fiveages_w2_description)/config/ros2_control/${ros2_control_config_basename}</parameters>
-			</plugin>
-		</gazebo>
-	</xacro:if>
+    <xacro:arg name="ros2_control_hardware_type" default="mock_components"/>
+    <xacro:include filename="$(find fiveages_w2_description)/xacro/robot.xacro"/>
+    <xacro:include filename="$(find m6_ccs_description)/xacro/ros2_control/interfaces.xacro"/>
+    <xacro:include filename="$(find fiveages_w2_description)/xacro/ros2_control/body.xacro"/>
+    <!-- <xacro:include filename="$(find fiveages_w2_description)/xacro/ros2_control/chassis.xacro"/> -->
+    <xacro:if value="${'$(arg ros2_control_hardware_type)' == 'real'}">
+        <ros2_control name="M6_CCS_System" type="system">
+            <hardware>
+                <plugin>marvin_ros2_control/MarvinHardware</plugin>
+                <param name="left_right_arm">2</param>
+            </hardware>
+            <xacro:m6_interfaces name="left"/>
+            <xacro:m6_interfaces name="right"/>
+        </ros2_control>
+        <ros2_control name="juxie_body" type="system">
+            <hardware>
+                <plugin>juxie_ros2_control/JxHardware</plugin>
+                <!-- CAN 接口配置 -->
+                <param name="can_interface">canfd</param>
+                <!-- 电机 ID 列表（最多 8 个） -->
+                <param name="motor_ids">1,2,3,4</param>
+                <!-- 控制周期（毫秒） -->
+                <param name="control_period_ms">1</param>
+            </hardware>
+            <xacro:body_interfaces/>
+        </ros2_control>
+    </xacro:if>
+    <xacro:unless value="${'$(arg ros2_control_hardware_type)' == 'real'}">
+        <ros2_control name="fiveages_w2_system" type="system">
+            <hardware>
+                <xacro:if value="${'$(arg ros2_control_hardware_type)' == 'gz'}">
+                    <plugin>gz_ros2_control/GazeboSimSystem</plugin>
+                </xacro:if>
+                <xacro:if value="${'$(arg ros2_control_hardware_type)' == 'mock_components'}">
+                    <plugin>mock_components/GenericSystem</plugin>
+                </xacro:if>
+                <xacro:if value="${'$(arg ros2_control_hardware_type)' == 'isaac'}">
+                    <plugin>topic_based_ros2_control/TopicBasedSystem</plugin>
+                    <param name="joint_commands_topic">/isaac/joint_command</param>
+                    <param name="joint_states_topic">/isaac/joint_states</param>
+                    <param name="sum_wrapped_joint_states">false</param>
+                    <param name="initialize_commands_from_state">true</param>
+                </xacro:if>
+            </hardware>
+            <xacro:body_interfaces/>
+            <xacro:m6_interfaces name="left"/>
+            <xacro:m6_interfaces name="right"/>
+        </ros2_control>
+    </xacro:unless>
+    <!-- Gazebo plugin configuration -->
+    <xacro:arg name="gazebo" default="false"/>
+    <xacro:if value="$(arg gazebo)">
+        <xacro:property name="ros2_control_config_basename" value="ros2_controllers.yaml"/>
+        <gazebo>
+            <plugin filename="gz_ros2_control-system" name="gz_ros2_control::GazeboSimROS2ControlPlugin">
+                <parameters>$(find fiveages_w2_description)/config/ros2_control/${ros2_control_config_basename}
+                </parameters>
+            </plugin>
+        </gazebo>
+    </xacro:if>
 </robot>

Commit message: update head joint

File: xacro/body.xacro (robot description, xacro)
@@ -4,5 +4,5 @@
 		<inertial>
 			<origin xyz="-0.000200488559999101 -0.000273639516978452 -0.146062494992026"/>
-			<mass value="8.23744177260185" />
+			<mass value="8.23744177260185"/>
 			<inertia
 					ixx="0.0427044289140212"
@@ -11,14 +11,14 @@
 					iyy="0.0344639116909607"
 					iyz="-1.07902056768718E-05"
-					izz="0.0490685771548297" />
-		</inertial>
-		<visual>
-			<geometry>
-				<mesh filename="file://$(find fiveages_w2_description)/meshes/body/base.obj" />
-			</geometry>
-		</visual>
-		<collision>
-			<geometry>
-				<mesh filename="file://$(find fiveages_w2_description)/meshes/body/base.obj" />
+					izz="0.0490685771548297"/>
+		</inertial>
+		<visual>
+			<geometry>
+				<mesh filename="file://$(find fiveages_w2_description)/meshes/body/base.obj"/>
+			</geometry>
+		</visual>
+		<collision>
+			<geometry>
+				<mesh filename="file://$(find fiveages_w2_description)/meshes/body/base.obj"/>
 			</geometry>
 		</collision>
@@ -26,11 +26,11 @@
 	<joint name="body_fixed_joint" type="fixed">
 		<origin xyz="0.10525 0 0.2295"/>
-		<parent link="base_link" />
-		<child link="body_base" />
+		<parent link="base_link"/>
+		<child link="body_base"/>
 	</joint>
 	<link name="body_link1">
 		<inertial>
 			<origin xyz="-5.26269080900477E-05 -0.000546927086993554 0.159848926806017"/>
-			<mass value="5.6518910145446" />
+			<mass value="5.6518910145446"/>
 			<inertia
 					ixx="0.129446325951384"
@@ -39,27 +39,27 @@
 					iyy="0.118974430850637"
 					iyz="0.000463913896532557"
-					izz="0.0161870223281112" />
-		</inertial>
-		<visual>
-			<geometry>
-				<mesh filename="file://$(find fiveages_w2_description)/meshes/body/link1.obj" />
-			</geometry>
-		</visual>
-		<collision>
-			<geometry>
-				<mesh filename="file://$(find fiveages_w2_description)/meshes/body/link1.obj" />
+					izz="0.0161870223281112"/>
+		</inertial>
+		<visual>
+			<geometry>
+				<mesh filename="file://$(find fiveages_w2_description)/meshes/body/link1.obj"/>
+			</geometry>
+		</visual>
+		<collision>
+			<geometry>
+				<mesh filename="file://$(find fiveages_w2_description)/meshes/body/link1.obj"/>
 			</geometry>
 		</collision>
 	</link>
 	<joint name="body_joint1" type="revolute">
-		<parent link="body_base" />
-		<child link="body_link1" />
-		<axis xyz="0 1 0" />
-		<limit lower="-1.352633" upper="0.567" effort="100" velocity="1" />
+		<parent link="body_base"/>
+		<child link="body_link1"/>
+		<axis xyz="0 1 0"/>
+		<limit lower="-1.352633" upper="0.567" effort="100" velocity="1"/>
 	</joint>
 	<link name="body_link2">
 		<inertial>
 			<origin xyz="-5.06261699229071E-14 -1.0902390101819E-13 0.172448903272911"/>
-			<mass value="7.6108743790626" />
+			<mass value="7.6108743790626"/>
 			<inertia
 					ixx="0.168898657844891"
@@ -68,14 +68,14 @@
 					iyy="0.189588222903554"
 					iyz="-2.80537312130624E-15"
-					izz="0.0218547815193579" />
-		</inertial>
-		<visual>
-			<geometry>
-				<mesh filename="file://$(find fiveages_w2_description)/meshes/body/link2.obj" />
-			</geometry>
-		</visual>
-		<collision>
-			<geometry>
-				<mesh filename="file://$(find fiveages_w2_description)/meshes/body/link2.obj" />
+					izz="0.0218547815193579"/>
+		</inertial>
+		<visual>
+			<geometry>
+				<mesh filename="file://$(find fiveages_w2_description)/meshes/body/link2.obj"/>
+			</geometry>
+		</visual>
+		<collision>
+			<geometry>
+				<mesh filename="file://$(find fiveages_w2_description)/meshes/body/link2.obj"/>
 			</geometry>
 		</collision>
@@ -83,13 +83,13 @@
 	<joint name="body_joint2" type="revolute">
 		<origin xyz="0 0 0.323"/>
-		<parent link="body_link1" />
-		<child link="body_link2" />
-		<axis xyz="0 -1 0" />
-		<limit lower="-2.66" upper="1.605" effort="100" velocity="1" />
+		<parent link="body_link1"/>
+		<child link="body_link2"/>
+		<axis xyz="0 -1 0"/>
+		<limit lower="-2.66" upper="1.605" effort="100" velocity="1"/>
 	</joint>
 	<link name="body_link3">
 		<inertial>
 			<origin xyz="2.24765231915391E-06 -0.017843126813746 0.0199837851518558"/>
-			<mass value="13.7293315804368" />
+			<mass value="13.7293315804368"/>
 			<inertia
 					ixx="0.0380691419113999"
@@ -98,14 +98,14 @@
 					iyy="0.0443960808652778"
 					iyz="8.97911264129812E-06"
-					izz="0.0332593124725221" />
-		</inertial>
-		<visual>
-			<geometry>
-				<mesh filename="file://$(find fiveages_w2_description)/meshes/body/link3.obj" />
-			</geometry>
-		</visual>
-		<collision>
-			<geometry>
-				<mesh filename="file://$(find fiveages_w2_description)/meshes/body/link3.obj" />
+					izz="0.0332593124725221"/>
+		</inertial>
+		<visual>
+			<geometry>
+				<mesh filename="file://$(find fiveages_w2_description)/meshes/body/link3.obj"/>
+			</geometry>
+		</visual>
+		<collision>
+			<geometry>
+				<mesh filename="file://$(find fiveages_w2_description)/meshes/body/link3.obj"/>
 			</geometry>
 		</collision>
@@ -113,43 +113,43 @@
 	<joint name="body_joint3" type="revolute">
 		<origin xyz="0 0.0019 0.35294"/>
-		<parent link="body_link2" />
-		<child link="body_link3" />
-		<axis xyz="0 1 0" />
-		<limit lower="-1.745" upper="1.745" effort="100" velocity="1" />
+		<parent link="body_link2"/>
+		<child link="body_link3"/>
+		<axis xyz="0 1 0"/>
+		<limit lower="-1.745" upper="1.745" effort="100" velocity="1"/>
 	</joint>
 	<link name="body_link4">
 		<inertial>
-			<origin xyz="-0.0249769763515 0.00261378092766984 0.273685327435851"/>
-			<mass value="23.7446873792875" />
-			<inertia
-					ixx="0.32004495936722"
-					ixy="8.27745275816937E-05"
-					ixz="0.0072338104417254"
-					iyy="0.228581680748554"
-					iyz="8.86157129443541E-05"
-					izz="0.136693312472866" />
-		</inertial>
-		<visual>
-			<geometry>
-				<mesh filename="file://$(find fiveages_w2_description)/meshes/body/link4.obj" />
-			</geometry>
-		</visual>
-		<collision>
-			<geometry>
-				<mesh filename="file://$(find fiveages_w2_description)/meshes/body/link4.obj" />
+			<origin xyz="-0.0150844595179076 0.00261332042527829 0.274407850772391"/>
+			<mass value="23.7446394325596"/>
+			<inertia
+					ixx="0.320326293119484"
+					ixy="8.41740202015408E-05"
+					ixz="0.000603743723020676"
+					iyy="0.228575723449718"
+					iyz="8.78726038347342E-05"
+					izz="0.136416117968312"/>
+		</inertial>
+		<visual>
+			<geometry>
+				<mesh filename="file://$(find fiveages_w2_description)/meshes/body/link4.obj"/>
+			</geometry>
+		</visual>
+		<collision>
+			<geometry>
+				<mesh filename="file://$(find fiveages_w2_description)/meshes/body/link4.obj"/>
 			</geometry>
 		</collision>
 	</link>
 	<joint name="body_joint4" type="revolute">
-		<origin xyz="0 -0.0019 0.1443"/>
-		<parent link="body_link3" />
-		<child link="body_link4" />
-		<axis xyz="0 0 -1" />
-		<limit lower="-3.14" upper="3.14" effort="100" velocity="1" />
+		<origin xyz="-7.1612E-05 -0.0019 0.14441"/>
+		<parent link="body_link3"/>
+		<child link="body_link4"/>
+		<axis xyz="0 0 -1"/>
+		<limit lower="-3.14" upper="3.14" effort="100" velocity="1"/>
 	</joint>
 	<link name="head_link1">
 		<inertial>
 			<origin xyz="0.0110684120335558 0.0270955929655894 -0.0849037421704728"/>
-			<mass value="1.76592019732553" />
+			<mass value="1.76592019732553"/>
 			<inertia
 					ixx="0.00540494211688139"
@@ -158,59 +158,59 @@
 					iyy="0.0045794535946287"
 					iyz="5.71011553188605E-05"
-					izz="0.00441063426341843" />
-		</inertial>
-		<visual>
-			<geometry>
-				<mesh filename="file://$(find fiveages_w2_description)/meshes/body/head_yaw.obj" />
-			</geometry>
-		</visual>
-		<collision>
-			<geometry>
-				<mesh filename="file://$(find fiveages_w2_description)/meshes/body/head_yaw.obj" />
+					izz="0.00441063426341843"/>
+		</inertial>
+		<visual>
+			<geometry>
+				<mesh filename="file://$(find fiveages_w2_description)/meshes/body/head_yaw.obj"/>
+			</geometry>
+		</visual>
+		<collision>
+			<geometry>
+				<mesh filename="file://$(find fiveages_w2_description)/meshes/body/head_yaw.obj"/>
 			</geometry>
 		</collision>
 	</link>
 	<joint name="head_joint1" type="revolute">
-		<origin xyz="-0.046314 -0.0272 0.63334"/>
-		<parent link="body_link4" />
-		<child link="head_link1" />
-		<axis xyz="0.036088 0 -0.99935" />
-		<limit lower="-3.14" upper="3.14" effort="100" velocity="1" />
+		<origin xyz="-0.023428 0 0.48475"/>
+		<parent link="body_link4"/>
+		<child link="head_link1"/>
+		<axis xyz="0 0 1"/>
+		<limit lower="-3.14" upper="3.14" effort="100" velocity="1"/>
 	</joint>
 	<link name="head_link2">
 		<inertial>
-			<origin xyz="0.0106970783153679 -0.00153937526954917 0.0535386876730146"/>
-			<mass value="1.96837023227358" />
-			<inertia
-					ixx="0.00378109514744319"
-					ixy="-1.35306059382265E-05"
-					ixz="-4.33373870574624E-05"
-					iyy="0.0035236676197971"
-					iyz="9.33508804534738E-06"
-					izz="0.00568993406575938" />
-		</inertial>
-		<visual>
-			<geometry>
-				<mesh filename="file://$(find fiveages_w2_description)/meshes/body/head_pitch.obj" />
-			</geometry>
-		</visual>
-		<collision>
-			<geometry>
-				<mesh filename="file://$(find fiveages_w2_description)/meshes/body/head_pitch.obj" />
+			<origin xyz="-0.0151771428301439 -0.00143945296196635 -0.0524451271193214"/>
+			<mass value="1.96836671464479"/>
+			<inertia
+					ixx="0.00378737345531871"
+					ixy="1.23509442005848E-05"
+					ixz="0.000117982756207023"
+					iyy="0.00352320847778892"
+					iyz="-1.03942260573708E-05"
+					izz="0.00568300818653482"/>
+		</inertial>
+		<visual>
+			<geometry>
+				<mesh filename="file://$(find fiveages_w2_description)/meshes/body/head_pitch.obj"/>
+			</geometry>
+		</visual>
+		<collision>
+			<geometry>
+				<mesh filename="file://$(find fiveages_w2_description)/meshes/body/head_pitch.obj"/>
 			</geometry>
 		</collision>
 	</link>
 	<joint name="head_joint2" type="revolute">
-		<origin xyz="0 0.0315 0"/>
-		<parent link="head_link1" />
-		<child link="head_link2" />
-		<axis xyz="0 -1 0" />
-		<limit lower="-3.14" upper="3.14" effort="100" velocity="1" />
+		<origin xyz="0 0.0042 0.15" rpy="3.1416 0 3.1416"/>
+		<parent link="head_link1"/>
+		<child link="head_link2"/>
+		<axis xyz="0 -1 0"/>
+		<limit lower="-3.14" upper="3.14" effort="100" velocity="1"/>
 	</joint>
 	<link name="arm_base"/>
 	<joint name="arm_base_joint" type="fixed">
-		<origin xyz="-0.0164439628111166 0 0.457354971463696"/>
-		<parent link="body_link4" />
-		<child link="arm_base" />
+		<origin xyz="7.1612E-05 0 0.45765"/>
+		<parent link="body_link4"/>
+		<child link="arm_base"/>
 	</joint>
 </robot>

Commit message: using high precision pi

File: xacro/body.xacro (robot description, xacro)
@@ -1,4 +1,5 @@
 <?xml version="1.0"?>
 <robot name="FiveAges W2" xmlns:xacro="http://www.ros.org/wiki/xacro">
+	<xacro:property name="PI" value="3.1415926535897931"/>
 	<link name="body_base">
 		<inertial>
@@ -146,5 +147,5 @@
 		<child link="body_link4"/>
 		<axis xyz="0 0 -1"/>
-		<limit lower="-3.14" upper="3.14" effort="100" velocity="1"/>
+		<limit lower="-${PI}" upper="${PI}" effort="100" velocity="1"/>
 	</joint>
 	<link name="head_link1">
@@ -202,5 +203,5 @@
 	</link>
 	<joint name="head_joint2" type="revolute">
-		<origin xyz="0 0.0042 0.15" rpy="3.1416 0 3.1416"/>
+		<origin xyz="0 0.0042 0.15" rpy="${PI} 0 ${PI}"/>
 		<parent link="head_link1"/>
 		<child link="head_link2"/>

File: xacro/chassis/linkhou_s2.xacro (robot description, xacro)
@@ -1,8 +1,9 @@
 <robot name="LinkHou_S2" xmlns:xacro="http://www.ros.org/wiki/xacro">
 	<link name="base_link"/>
+	<xacro:property name="PI" value="3.1415926535897931"/>
 	<joint name="base_link_mount" type="fixed">
 		<parent link="base_link"/>
 		<child link="chassis_base"/>
-		<origin rpy="0 0 3.1415926535"/>
+		<origin rpy="0 0 ${PI}"/>
 	</joint>
 	<link name="chassis_base">
@@ -72,6 +73,7 @@
 		</visual>
 		<collision>
-			<geometry>
-				<mesh filename="file://$(find fiveages_w2_description)/meshes/linkhou_s2/wheel.obj" scale="1 -1 1"/>
+			<origin rpy="${PI/2.0} 0 0"/>
+			<geometry>
+				<cylinder radius="0.07" length="0.046"/>
 			</geometry>
 		</collision>
@@ -127,6 +129,7 @@
 		</visual>
 		<collision>
-			<geometry>
-				<mesh filename="file://$(find fiveages_w2_description)/meshes/linkhou_s2/wheel.obj"/>
+			<origin rpy="${PI/2.0} 0 0"/>
+			<geometry>
+				<cylinder radius="0.07" length="0.046"/>
 			</geometry>
 		</collision>
@@ -182,6 +185,7 @@
 		</visual>
 		<collision>
-			<geometry>
-				<mesh filename="file://$(find fiveages_w2_description)/meshes/linkhou_s2/wheel.obj" scale="1 -1 1"/>
+			<origin rpy="${PI/2.0} 0 0"/>
+			<geometry>
+				<cylinder radius="0.07" length="0.046"/>
 			</geometry>
 		</collision>
@@ -237,6 +241,7 @@
 		</visual>
 		<collision>
-			<geometry>
-				<mesh filename="file://$(find fiveages_w2_description)/meshes/linkhou_s2/wheel.obj"/>
+			<origin rpy="${PI/2.0} 0 0"/>
+			<geometry>
+				<cylinder radius="0.07" length="0.046"/>
 			</geometry>
 		</collision>
@@ -273,5 +278,5 @@
 	</link>
 	<joint name="rr_lidar_joint" type="fixed">
-		<origin xyz="0.21412 0.19406 0.32957" rpy="1.5708 -1.309 0"/>
+		<origin xyz="0.21412 0.19406 0.32957" rpy="${PI/2.0} -1.309 0"/>
 		<parent link="chassis_base"/>
 		<child link="rr_lidar"/>
@@ -301,5 +306,5 @@
 	</link>
 	<joint name="fl_lidar_joint" type="fixed">
-		<origin xyz="-0.21412 -0.19406 0.32957" rpy="1.5708 -1.309 3.1416"/>
+		<origin xyz="-0.21412 -0.19406 0.32957" rpy="${PI/2.0} -1.309 3.1416"/>
 		<parent link="chassis_base"/>
 		<child link="fl_lidar"/>
@@ -318,5 +323,5 @@
 	</link>
 	<joint name="chassis_camera_joint" type="fixed">
-		<origin xyz="-0.3438 -0.00032028 0.159" rpy="0 0 3.1416"/>
+		<origin xyz="-0.3438 -0.00032028 0.159" rpy="0 0 ${PI}"/>
 		<parent link="chassis_base"/>
 		<child link="chassis_camera"/>

File: xacro/robot.xacro (robot description, xacro)
@@ -8,5 +8,5 @@
 		<parent link="arm_base"/>
 		<child link="left_base_link"/>
-		<origin rpy="-1.5708 0 0" xyz="0.0 0.062 0"/>
+		<origin rpy="-${PI/2} 0 0" xyz="0.0 0.062 0"/>
 	</joint>
 	<!-- Right Arm -->
@@ -14,5 +14,5 @@
 		<parent link="arm_base"/>
 		<child link="right_base_link"/>
-		<origin rpy="1.5708 0 0" xyz="0 -0.062 0"/>
+		<origin rpy="${PI/2} 0 0" xyz="0 -0.062 0"/>
 	</joint>
 	<xacro:include filename="$(find m6_ccs_description)/xacro/arm.xacro"/>

Commit message: add head top camera

File: xacro/body.xacro (robot description, xacro)
@@ -216,5 +216,5 @@
 	</link>
 	<joint name="head_joint2" type="revolute">
-		<origin xyz="0 0.0042 0.15" rpy="${PI} 0 ${PI}"/>
+		<origin xyz="0 0.0042 0.15"/>
 		<parent link="head_link1"/>
 		<child link="head_link2"/>
@@ -230,5 +230,5 @@
 	</link>
 	<joint name="head_camera_joint" type="fixed">
-		<origin xyz="-0.097847  0.046703 -0.12364" rpy="0 -0.64460396 ${PI}"/>
+		<origin xyz="0.097847  0.046703 0.12364" rpy="${PI} 0.64460396 0"/>
 		<parent link="head_link2"/>
 		<child link="head_camera"/>
@@ -240,3 +240,9 @@
 		<child link="arm_base"/>
 	</joint>
+	<link name="head_top_camera"/>
+	<joint name="head_top_camera_joint" type="fixed">
+		<origin xyz="0.0877736 0.0245687 0.107989" rpy="-2.100227811211368 0.0016038446958035316 -1.583610269343787"/>
+		<parent link="head_link2"/>
+		<child link="head_top_camera"/>
+	</joint>
 </robot>
