Commit message: add sinopec style

File: xacro/body.xacro (robot description, xacro)
@@ -216,5 +216,5 @@
 	</link>
 	<joint name="head_joint2" type="revolute">
-		<origin xyz="0 0.0042 0.15"/>
+		<origin xyz="0 0.0 0.15"/>
 		<parent link="head_link1"/>
 		<child link="head_link2"/>

File: xacro/component.xacro (robot description, xacro)
@@ -8,5 +8,5 @@
 	<xacro:arg name="chassis_joints_movable" default="true"/>
 	<xacro:if value="${'$(arg type)' == 'linkhou_q2'}">
-		<xacro:include filename="$(find fiveages_w2_description)/xacro/chassis/linkhou_s2.xacro"/>
+		<xacro:include filename="$(find fiveages_w2_description)/xacro/components/linkhou_s2.xacro"/>
 		<xacro:linkhou_s2 joints_movable="$(arg chassis_joints_movable)"/>
 	</xacro:if>

File: xacro/robot.xacro (robot description, xacro)
@@ -3,5 +3,5 @@
 	<xacro:arg name="collider" default="convex"/>
 	<xacro:arg name="chassis_joints_movable" default="false"/>
-	<xacro:include filename="$(find fiveages_w2_description)/xacro/chassis/linkhou_s2.xacro"/>
+	<xacro:include filename="$(find fiveages_w2_description)/xacro/components/linkhou_s2.xacro"/>
 	<xacro:linkhou_s2 joints_movable="$(arg chassis_joints_movable)"/>
 	<xacro:include filename="$(find fiveages_w2_description)/xacro/body.xacro"/>
@@ -18,5 +18,5 @@
 		<origin rpy="${PI/2} 0 0" xyz="0 -0.062 0"/>
 	</joint>
-	<xacro:include filename="$(find m6_ccs_description)/xacro/arm.xacro"/>
+	<xacro:include filename="$(find fiveages_w2_description)/xacro/components/arm.xacro"/>
 	<xacro:M6_CCS name="left" collider="$(arg collider)"/>
 	<xacro:M6_CCS name="right" direction="-1" collider="$(arg collider)"/>
