Commit message: 实现全身控制

File: xacro/robot.xacro (robot description, xacro)
@@ -210,4 +210,11 @@
 		<limit lower="-3.14" upper="3.14" effort="100" velocity="1" />
 	</joint>
+	<!-- Alias link for compatibility with arms_target_manager (which expects head_link2) -->
+	<link name="head_link2"/>
+	<joint name="head_link2_alias_joint" type="fixed">
+		<parent link="head_pitch"/>
+		<child link="head_link2"/>
+		<origin xyz="0 0 0" rpy="0 0 0"/>
+	</joint>
 	<link name="arm_base"/>
 	<joint name="arm_base_joint" type="fixed">

Commit message: add movej dialog

File: xacro/robot.xacro (robot description, xacro)
@@ -19,3 +19,7 @@
 	<xacro:M6_CCS name="left" collider="$(arg collider)"/>
 	<xacro:M6_CCS name="right" direction="-1" collider="$(arg collider)"/>
+	<xacro:arg name="type" default=""/>
+	<xacro:property name="selected_gripper_type" value="$(arg type)"/>
+	<xacro:include filename="$(find fiveages_w2_description)/xacro/grippers.xacro"/>
+	<xacro:Grippers type="${selected_gripper_type}"/>
 </robot>

Commit message: add o6

File: xacro/robot.xacro (robot description, xacro)
@@ -21,10 +21,12 @@
 	<xacro:M6_CCS name="left" collider="$(arg collider)"/>
 	<xacro:M6_CCS name="right" direction="-1" collider="$(arg collider)"/>
-	<!-- 从 type 参数解析出 gripper_type -->
+	<!-- 从 type 参数解析出 hand_type 和 gripper_type -->
 	<xacro:arg name="type" default=""/>
 	<xacro:property name="type_arg" value="$(arg type)"/>
 	<!-- 默认值 -->
+	<xacro:property name="selected_hand_type" value=""/>
 	<xacro:property name="selected_gripper_type" value=""/>
-	<!-- 从 type 解析 gripper_type -->
+	<!-- 从 type 解析 hand_type 和 gripper_type -->
+	<!-- 夹爪类型：selected_gripper_type 不为空即表示使用夹爪 -->
 	<xacro:if value="${type_arg == 'rg75'}">
 		<xacro:property name="selected_gripper_type" value="rg75"/>
@@ -39,5 +41,9 @@
 		<xacro:property name="selected_gripper_type" value="ag2f90_d"/>
 	</xacro:if>
-	<xacro:include filename="$(find fiveages_w2_description)/xacro/grippers.xacro"/>
-	<xacro:Grippers type="${selected_gripper_type}"/>
+	<!-- 灵巧手类型 -->
+	<xacro:if value="${type_arg == 'linkerhand_o6'}">
+		<xacro:property name="selected_hand_type" value="linkerhand_o6"/>
+	</xacro:if>
+	<xacro:include filename="$(find fiveages_w2_description)/xacro/eefs.xacro"/>
+	<xacro:EndEffectors hand_type="${selected_hand_type}" gripper_type="${selected_gripper_type}"/>
 </robot>

File: xacro/ros2_control/robot.xacro (robot description, xacro)
@@ -17,4 +17,5 @@
 			<xacro:m6_interfaces name="left"/>
 			<xacro:m6_interfaces name="right"/>
+			<!-- 夹爪接口：selected_gripper_type 不为空即表示使用夹爪 -->
 			<xacro:if value="${selected_gripper_type != ''}">
 				<joint name="left_gripper_joint">
@@ -30,4 +31,10 @@
 					</state_interface>
 				</joint>
+			</xacro:if>
+			<!-- 灵巧手接口 -->
+			<xacro:if value="${selected_hand_type == 'linkerhand_o6'}">
+				<xacro:include filename="$(find linkerhand_description)/xacro/ros2_control/o6.xacro"/>
+				<xacro:linkerhand_o6_interfaces name="left_hand"/>
+				<xacro:linkerhand_o6_interfaces name="right_hand"/>
 			</xacro:if>
 		</ros2_control>
@@ -65,15 +72,20 @@
 			<xacro:m6_interfaces name="left"/>
 			<xacro:m6_interfaces name="right"/>
-			<xacro:if
-					value="${selected_gripper_type == 'rg75'}">
+			<!-- 夹爪接口：selected_gripper_type 不为空即表示使用夹爪 -->
+			<xacro:if value="${selected_gripper_type == 'rg75'}">
 				<xacro:include filename="$(find jodell_description)/xacro/ros2_control/RG75-300.xacro"/>
 				<xacro:rg75_interfaces name="left"/>
 				<xacro:rg75_interfaces name="right"/>
 			</xacro:if>
-			<xacro:if
-					value="${selected_gripper_type == 'ag2f90_c' or selected_gripper_type == 'ag2f90_d'}">
+			<xacro:if value="${selected_gripper_type == 'ag2f90_c' or selected_gripper_type == 'ag2f90_d'}">
 				<xacro:include filename="$(find changingtek_description)/xacro/ros2_control/AG2F90-C.xacro"/>
 				<xacro:ag2f90c_interfaces name="left"/>
 				<xacro:ag2f90c_interfaces name="right"/>
+			</xacro:if>
+			<!-- 灵巧手接口 -->
+			<xacro:if value="${selected_hand_type == 'linkerhand_o6'}">
+				<xacro:include filename="$(find linkerhand_description)/xacro/ros2_control/o6.xacro"/>
+				<xacro:linkerhand_o6_interfaces name="left_hand"/>
+				<xacro:linkerhand_o6_interfaces name="right_hand"/>
 			</xacro:if>
 		</ros2_control>

Commit message: Merge pull request #1 from fiveages-sim/feature/o6
Feature/o6

File: xacro/robot.xacro (robot description, xacro)
@@ -21,10 +21,12 @@
 	<xacro:M6_CCS name="left" collider="$(arg collider)"/>
 	<xacro:M6_CCS name="right" direction="-1" collider="$(arg collider)"/>
-	<!-- 从 type 参数解析出 gripper_type -->
+	<!-- 从 type 参数解析出 hand_type 和 gripper_type -->
 	<xacro:arg name="type" default=""/>
 	<xacro:property name="type_arg" value="$(arg type)"/>
 	<!-- 默认值 -->
+	<xacro:property name="selected_hand_type" value=""/>
 	<xacro:property name="selected_gripper_type" value=""/>
-	<!-- 从 type 解析 gripper_type -->
+	<!-- 从 type 解析 hand_type 和 gripper_type -->
+	<!-- 夹爪类型：selected_gripper_type 不为空即表示使用夹爪 -->
 	<xacro:if value="${type_arg == 'rg75'}">
 		<xacro:property name="selected_gripper_type" value="rg75"/>
@@ -39,5 +41,12 @@
 		<xacro:property name="selected_gripper_type" value="ag2f90_d"/>
 	</xacro:if>
-	<xacro:include filename="$(find fiveages_w2_description)/xacro/grippers.xacro"/>
-	<xacro:Grippers type="${selected_gripper_type}"/>
+	<!-- 灵巧手类型 -->
+	<xacro:if value="${type_arg == 'linkerhand_o6'}">
+		<xacro:property name="selected_hand_type" value="linkerhand_o6"/>
+	</xacro:if>
+	<xacro:if value="${type_arg == 'linkerhand_l6'}">
+		<xacro:property name="selected_hand_type" value="linkerhand_l6"/>
+	</xacro:if>
+	<xacro:include filename="$(find fiveages_w2_description)/xacro/eefs.xacro"/>
+	<xacro:EndEffectors hand_type="${selected_hand_type}" gripper_type="${selected_gripper_type}"/>
 </robot>

File: xacro/ros2_control/robot.xacro (robot description, xacro)
@@ -17,4 +17,5 @@
 			<xacro:m6_interfaces name="left"/>
 			<xacro:m6_interfaces name="right"/>
+			<!-- 夹爪接口：selected_gripper_type 不为空即表示使用夹爪 -->
 			<xacro:if value="${selected_gripper_type != ''}">
 				<joint name="left_gripper_joint">
@@ -30,4 +31,10 @@
 					</state_interface>
 				</joint>
+			</xacro:if>
+			<!-- 灵巧手接口 -->
+			<xacro:if value="${selected_hand_type == 'linkerhand_o6' or selected_hand_type == 'linkerhand_l6'}">
+				<xacro:include filename="$(find linkerhand_description)/xacro/ros2_control/o6.xacro"/>
+				<xacro:linkerhand_o6_interfaces name="left_hand"/>
+				<xacro:linkerhand_o6_interfaces name="right_hand"/>
 			</xacro:if>
 		</ros2_control>
@@ -65,15 +72,20 @@
 			<xacro:m6_interfaces name="left"/>
 			<xacro:m6_interfaces name="right"/>
-			<xacro:if
-					value="${selected_gripper_type == 'rg75'}">
+			<!-- 夹爪接口：selected_gripper_type 不为空即表示使用夹爪 -->
+			<xacro:if value="${selected_gripper_type == 'rg75'}">
 				<xacro:include filename="$(find jodell_description)/xacro/ros2_control/RG75-300.xacro"/>
 				<xacro:rg75_interfaces name="left"/>
 				<xacro:rg75_interfaces name="right"/>
 			</xacro:if>
-			<xacro:if
-					value="${selected_gripper_type == 'ag2f90_c' or selected_gripper_type == 'ag2f90_d'}">
+			<xacro:if value="${selected_gripper_type == 'ag2f90_c' or selected_gripper_type == 'ag2f90_d'}">
 				<xacro:include filename="$(find changingtek_description)/xacro/ros2_control/AG2F90-C.xacro"/>
 				<xacro:ag2f90c_interfaces name="left"/>
 				<xacro:ag2f90c_interfaces name="right"/>
+			</xacro:if>
+			<!-- 灵巧手接口 -->
+			<xacro:if value="${selected_hand_type == 'linkerhand_o6' or selected_hand_type == 'linkerhand_l6'}">
+				<xacro:include filename="$(find linkerhand_description)/xacro/ros2_control/o6.xacro"/>
+				<xacro:linkerhand_o6_interfaces name="left_hand"/>
+				<xacro:linkerhand_o6_interfaces name="right_hand"/>
 			</xacro:if>
 		</ros2_control>

Commit message: update xacro file for IP and hand ctrl

File: xacro/robot.xacro (robot description, xacro)
@@ -6,5 +6,5 @@
 	<xacro:arg name="type" default=""/>
 	<xacro:property name="type_arg" value="$(arg type)"/>
-	<!-- 手部控制方式：usb 或 marvin -->
+	<!-- 手部控制模式：通过 type 后缀选择（_usb -> modbus, _marvin -> marvin 485） -->
 	<xacro:arg name="hand_control_mode" default="usb"/>
 	<xacro:property name="hand_control_mode_arg" value="$(arg hand_control_mode)"/>
@@ -26,13 +26,22 @@
 		<xacro:property name="selected_gripper_type" value="ag2f90_d"/>
 	</xacro:if>
-	<!-- 灵巧手类型 -->
-	<xacro:if value="${type_arg == 'linkerhand_o6'}">
+	<!-- 灵巧手类型解析：支持格式 linkerhand_{o6,l6,o7}[_usb|_marvin] -->
+	<!-- O6 -->
+	<xacro:if value="${type_arg == 'linkerhand_o6' or type_arg == 'linkerhand_o6_usb' or type_arg == 'linkerhand_o6_marvin'}">
 		<xacro:property name="selected_hand_type" value="linkerhand_o6"/>
+		<xacro:if value="${type_arg == 'linkerhand_o6_usb'}"><xacro:property name="hand_control_mode_arg" value="usb"/></xacro:if>
+		<xacro:if value="${type_arg == 'linkerhand_o6_marvin'}"><xacro:property name="hand_control_mode_arg" value="marvin"/></xacro:if>
 	</xacro:if>
-	<xacro:if value="${type_arg == 'linkerhand_l6'}">
+	<!-- L6 -->
+	<xacro:if value="${type_arg == 'linkerhand_l6' or type_arg == 'linkerhand_l6_usb' or type_arg == 'linkerhand_l6_marvin'}">
 		<xacro:property name="selected_hand_type" value="linkerhand_l6"/>
+		<xacro:if value="${type_arg == 'linkerhand_l6_usb'}"><xacro:property name="hand_control_mode_arg" value="usb"/></xacro:if>
+		<xacro:if value="${type_arg == 'linkerhand_l6_marvin'}"><xacro:property name="hand_control_mode_arg" value="marvin"/></xacro:if>
 	</xacro:if>
-	<xacro:if value="${type_arg == 'linkerhand_o7'}">
+	<!-- O7 -->
+	<xacro:if value="${type_arg == 'linkerhand_o7' or type_arg == 'linkerhand_o7_usb' or type_arg == 'linkerhand_o7_marvin'}">
 		<xacro:property name="selected_hand_type" value="linkerhand_o7"/>
+		<xacro:if value="${type_arg == 'linkerhand_o7_usb'}"><xacro:property name="hand_control_mode_arg" value="usb"/></xacro:if>
+		<xacro:if value="${type_arg == 'linkerhand_o7_marvin'}"><xacro:property name="hand_control_mode_arg" value="marvin"/></xacro:if>
 	</xacro:if>
 	<xacro:include filename="$(find fiveages_w2_description)/xacro/components/linkhou_s2.xacro"/>

File: xacro/ros2_control/robot.xacro (robot description, xacro)
@@ -2,12 +2,27 @@
 <robot name="fiveages_w2" xmlns:xacro="http://www.ros.org/wiki/xacro">
 	<xacro:arg name="ros2_control_hardware_type" default="mock_components"/>
+	<xacro:arg name="device_ip" default="192.168.1.190"/>
+	<xacro:property name="device_ip_arg" value="$(arg device_ip)"/>
 	<xacro:include filename="$(find fiveages_w2_description)/xacro/robot.xacro"/>
 	<xacro:include filename="$(find m6_ccs_description)/xacro/ros2_control/interfaces.xacro"/>
 	<xacro:include filename="$(find fiveages_w2_description)/xacro/ros2_control/body.xacro"/>
+	<!-- 宏：创建单个 modbus 灵巧手系统（USB 模式） -->
+	<xacro:macro name="create_modbus_hand_single" params="hand_type system_suffix side serial_port">
+		<ros2_control name="linkerhand_${system_suffix}_${side}_system" type="system">
+			<hardware>
+				<plugin>modbus_ros2_control/DexterousHandHardware</plugin>
+				<param name="serial_port">${serial_port}</param>
+				<param name="hand_type">${hand_type}</param>
+				<param name="hand_side">${side}</param>
+				<param name="max_speed_ratio">1.0</param>
+			</hardware>
+			<xacro:insert_block/>
+		</ros2_control>
+	</xacro:macro>
 	<xacro:if value="${'$(arg ros2_control_hardware_type)' == 'real'}">
 		<!-- 确定传递给 marvin_ros2_control 的 gripper_type 参数 -->
 		<!--
 			Marvin 模式下的手部控制逻辑：
-			1. 如果 hand_control_mode == 'marvin' 且 selected_hand_type 不为空，
+			1. 如果 hand_control_mode_arg == 'marvin'（由 type 后缀 _marvin 设定）且 selected_hand_type 不为空，
 			   则将 selected_hand_type (如 linkerhand_o7) 传递给 MarvinHardware 的 gripper_type 参数
 			2. MarvinHardware 会通过 normalizeString() 将 gripper_type 转换为大写
@@ -38,5 +53,5 @@
 				<param name="left_dyn_param">0.4,0,0,50.65,0,0,0,0,0,0</param>
 				<param name="right_dyn_param">0.4,0,0,50.85,0,0,0,0,0,0</param>
-				<param name="device_ip"></param>
+				<param name="device_ip">${device_ip_arg}</param>
 			</hardware>
 			<xacro:m6_interfaces name="left"/>
@@ -57,10 +72,5 @@
 				</joint>
 			</xacro:if>
-			<!--
-				灵巧手接口：通过天机硬件控制（marvin 模式）
-				注意：这些接口会被添加到 M6_CCS_System 中，MarvinHardware 会通过 gripper_type 参数
-				检测到手部类型，并创建对应的 DexterousHand 对象来控制这些关节。
-				控制通过 485 总线完成，不需要 modbus_ros2_control。
-			-->
+			<!-- 灵巧手接口：marvin 模式（485 总线，通过 M6_CCS_System） -->
 			<xacro:if value="${selected_hand_type != '' and hand_control_mode_arg == 'marvin'}">
 				<xacro:if value="${selected_hand_type == 'linkerhand_o6' or selected_hand_type == 'linkerhand_l6'}">
@@ -88,53 +98,25 @@
 			<xacro:body_interfaces/>
 		</ros2_control>
-		<!-- 灵巧手接口：通过 USB (modbus_ros2_control) -->
-		<!-- 只有在 hand_control_mode 明确为 'usb' 时才创建 modbus 系统 -->
-		<!-- 注意：marvin 模式下，手的控制通过 M6_CCS_System 中的 MarvinHardware 完成，不需要 modbus 系统 -->
+		<!-- 灵巧手接口：USB 模式（modbus_ros2_control） -->
 		<xacro:if value="${selected_hand_type != '' and hand_control_mode_arg == 'usb'}">
+			<!-- O6/L6: 6-DOF 手 -->
 			<xacro:if value="${selected_hand_type == 'linkerhand_o6' or selected_hand_type == 'linkerhand_l6'}">
 				<xacro:include filename="$(find linkerhand_description)/xacro/ros2_control/o6.xacro"/>
-				<ros2_control name="linkerhand_6_left_system" type="system">
-					<hardware>
-						<plugin>modbus_ros2_control/DexterousHandHardware</plugin>
-						<param name="serial_port">/dev/ttyUSB1</param>
-						<param name="hand_type">${selected_hand_type}</param>
-						<param name="hand_side">left</param>
-						<param name="max_speed_ratio">1.0</param>
-					</hardware>
+				<xacro:create_modbus_hand_single hand_type="${selected_hand_type}" system_suffix="6" side="left" serial_port="/dev/ttyUSB1">
 					<xacro:linkerhand_o6_interfaces name="left_hand"/>
-				</ros2_control>
-				<ros2_control name="linkerhand_6_right_system" type="system">
-					<hardware>
-						<plugin>modbus_ros2_control/DexterousHandHardware</plugin>
-						<param name="serial_port">/dev/ttyUSB0</param>
-						<param name="hand_type">${selected_hand_type}</param>
-						<param name="hand_side">right</param>
-						<param name="max_speed_ratio">1.0</param>
-					</hardware>
+				</xacro:create_modbus_hand_single>
+				<xacro:create_modbus_hand_single hand_type="${selected_hand_type}" system_suffix="6" side="right" serial_port="/dev/ttyUSB0">
 					<xacro:linkerhand_o6_interfaces name="right_hand"/>
-				</ros2_control>
+				</xacro:create_modbus_hand_single>
 			</xacro:if>
+			<!-- O7: 7-DOF 手 -->
 			<xacro:if value="${selected_hand_type == 'linkerhand_o7'}">
 				<xacro:include filename="$(find linkerhand_description)/xacro/ros2_control/o7.xacro"/>
-				<ros2_control name="linkerhand_7_left_system" type="system">
-					<hardware>
-						<plugin>modbus_ros2_control/DexterousHandHardware</plugin>
-						<param name="serial_port">/dev/ttyUSB1</param>
-						<param name="hand_type">${selected_hand_type}</param>
-						<param name="hand_side">left</param>
-						<param name="max_speed_ratio">1.0</param>
-					</hardware>
+				<xacro:create_modbus_hand_single hand_type="${selected_hand_type}" system_suffix="7" side="left" serial_port="/dev/ttyUSB1">
 					<xacro:linkerhand_o7_interfaces name="left_hand"/>
-				</ros2_control>
-				<ros2_control name="linkerhand_7_right_system" type="system">
-					<hardware>
-						<plugin>modbus_ros2_control/DexterousHandHardware</plugin>
-						<param name="serial_port">/dev/ttyUSB0</param>
-						<param name="hand_type">${selected_hand_type}</param>
-						<param name="hand_side">right</param>
-						<param name="max_speed_ratio">1.0</param>
-					</hardware>
+				</xacro:create_modbus_hand_single>
+				<xacro:create_modbus_hand_single hand_type="${selected_hand_type}" system_suffix="7" side="right" serial_port="/dev/ttyUSB0">
 					<xacro:linkerhand_o7_interfaces name="right_hand"/>
-				</ros2_control>
+				</xacro:create_modbus_hand_single>
 			</xacro:if>
 		</xacro:if>
