Commit message: Update xacro file to support marvin 485 communication

File: xacro/robot.xacro (robot description, xacro)
@@ -1,58 +1,99 @@
 <?xml version="1.0"?>
-<robot name="FiveAges W2" xmlns:xacro="http://www.ros.org/wiki/xacro">
-	<xacro:arg name="collider" default="convex"/>
-	<xacro:arg name="chassis_joints_movable" default="false"/>
-	<!-- 从 type 参数解析出 hand_type 和 gripper_type -->
-	<xacro:arg name="type" default=""/>
-	<xacro:property name="type_arg" value="$(arg type)"/>
-	<!-- 手部控制方式：usb 或 marvin -->
-	<xacro:arg name="hand_control_mode" default="usb"/>
-	<xacro:property name="hand_control_mode_arg" value="$(arg hand_control_mode)"/>
-	<!-- 默认值 -->
-	<xacro:property name="selected_hand_type" value=""/>
-	<xacro:property name="selected_gripper_type" value=""/>
-	<!-- 从 type 解析 hand_type 和 gripper_type -->
-	<!-- 夹爪类型：selected_gripper_type 不为空即表示使用夹爪 -->
-	<xacro:if value="${type_arg == 'rg75'}">
-		<xacro:property name="selected_gripper_type" value="rg75"/>
-	</xacro:if>
-	<xacro:if value="${type_arg == 'ag2f90'}">
-		<xacro:property name="selected_gripper_type" value="ag2f90_d"/>
-	</xacro:if>
-	<xacro:if value="${type_arg == 'ag2f90_c'}">
-		<xacro:property name="selected_gripper_type" value="ag2f90_c"/>
-	</xacro:if>
-	<xacro:if value="${type_arg == 'ag2f90_d'}">
-		<xacro:property name="selected_gripper_type" value="ag2f90_d"/>
-	</xacro:if>
-	<!-- 灵巧手类型 -->
-	<xacro:if value="${type_arg == 'linkerhand_o6'}">
-		<xacro:property name="selected_hand_type" value="linkerhand_o6"/>
-	</xacro:if>
-	<xacro:if value="${type_arg == 'linkerhand_l6'}">
-		<xacro:property name="selected_hand_type" value="linkerhand_l6"/>
-	</xacro:if>
-	<xacro:if value="${type_arg == 'linkerhand_o7'}">
-		<xacro:property name="selected_hand_type" value="linkerhand_o7"/>
-	</xacro:if>
-	<xacro:include filename="$(find fiveages_w2_description)/xacro/components/linkhou_s2.xacro"/>
-	<xacro:linkhou_s2 joints_movable="$(arg chassis_joints_movable)"/>
-	<xacro:include filename="$(find fiveages_w2_description)/xacro/components/body.xacro"/>
-	<!-- Left Arm -->
-	<joint name="left_arm_base_joint" type="fixed">
-		<parent link="arm_base"/>
-		<child link="left_base_link"/>
-		<origin rpy="-${PI/2} 0 0" xyz="0.0 0.062 0"/>
-	</joint>
-	<!-- Right Arm -->
-	<joint name="right_arm_base_joint" type="fixed">
-		<parent link="arm_base"/>
-		<child link="right_base_link"/>
-		<origin rpy="${PI/2} 0 0" xyz="0 -0.062 0"/>
-	</joint>
-	<xacro:include filename="$(find m6_ccs_description)/xacro/arm.xacro"/>
-	<xacro:M6_CCS name="left" style="fiveages_w2"/>
-	<xacro:M6_CCS name="right" direction="-1" style="fiveages_w2"/>
-	<xacro:include filename="$(find fiveages_w2_description)/xacro/eefs.xacro"/>
-	<xacro:EndEffectors hand_type="${selected_hand_type}" gripper_type="${selected_gripper_type}"/>
+<robot xmlns:xacro="http://www.ros.org/wiki/xacro">
+    <xacro:macro name="EndEffectors" params="hand_type:='' gripper_type:=''">
+        <!-- Note:
+             - gripper_type 不为空时表示使用夹爪（保持原有逻辑）
+             - hand_type 只在需要区分灵巧手时使用（如 linkerhand_o6）
+             - 两者都为空时表示无末端执行器配置
+        -->
+        <!-- 无末端执行器配置 -->
+        <xacro:if value="${hand_type == '' and gripper_type == ''}">
+            <link name="left_eef"/>
+            <link name="right_eef"/>
+            <joint name="left_eef_joint" type="fixed">
+                <parent link="left_tcp"/>
+                <child link="left_eef"/>
+            </joint>
+            <joint name="right_eef_joint" type="fixed">
+                <parent link="right_tcp"/>
+                <child link="right_eef"/>
+            </joint>
+        </xacro:if>
+        <!-- 夹爪类型：gripper_type 不为空即表示使用夹爪 -->
+        <xacro:if value="${gripper_type == 'ag2f90_c' or gripper_type == 'ag2f90_d'}">
+            <xacro:include filename="$(find changingtek_description)/xacro/AG2F90-C.xacro"/>
+            <xacro:AG2F90-C name="left" use_flange="true"/>
+            <joint name="left_gripper_fix" type="fixed">
+                <parent link="left_tcp"/>
+                <child link="left_flange"/>
+                <origin xyz="0 0 0.0045"/>
+            </joint>
+            <xacro:AG2F90-C name="right" use_flange="true"/>
+            <joint name="right_gripper_fix" type="fixed">
+                <parent link="right_tcp"/>
+                <child link="right_flange"/>
+                <origin xyz="0 0 0.0045"/>
+            </joint>
+        </xacro:if>
+        <xacro:if value="${gripper_type == 'rg75'}">
+            <xacro:include filename="$(find jodell_description)/xacro/RG75-300.xacro"/>
+            <xacro:RG75-300 name="left" use_flange="true"/>
+            <xacro:RG75-300 name="right" use_flange="true"/>
+            <joint name="left_gripper_base_joint" type="fixed">
+                <parent link="left_tcp"/>
+                <child link="left_flange"/>
+            </joint>
+            <joint name="right_gripper_base_joint" type="fixed">
+                <parent link="right_tcp"/>
+                <child link="right_flange"/>
+            </joint>
+        </xacro:if>
+        <!-- 灵巧手类型 -->
+        <xacro:if value="${hand_type == 'linkerhand_o6'}">
+            <xacro:include filename="$(find linkerhand_description)/xacro/o6.xacro"/>
+            <xacro:LinkerHandO6 name="left_hand" direction="1" use_flange="true" fixed_joints="false"/>
+            <joint name="left_hand_base_joint" type="fixed">
+                <origin xyz="0 0 0.0045" rpy="0 0 ${PI}"/>
+                <parent link="left_tcp"/>
+                <child link="left_hand_flange"/>
+            </joint>
+            <xacro:LinkerHandO6 name="right_hand" direction="-1" use_flange="true" fixed_joints="false"/>
+            <joint name="right_hand_base_joint" type="fixed">
+                <parent link="right_tcp"/>
+                <child link="right_hand_flange"/>
+                <origin xyz="0 0 0.0045"/>
+            </joint>
+        </xacro:if>
+        <xacro:if value="${hand_type == 'linkerhand_o7'}">
+            <xacro:include filename="$(find linkerhand_description)/xacro/o7.xacro"/>
+            <xacro:LinkerHandO7 name="left_hand" direction="1" use_flange="true" fixed_joints="false"/>
+            <joint name="left_hand_base_joint" type="fixed">
+                <origin rpy="0 0 ${PI/2}"/>
+                <parent link="left_tcp"/>
+                <child link="left_hand_flange"/>
+            </joint>
+            <xacro:LinkerHandO7 name="right_hand" direction="-1" use_flange="true" fixed_joints="false"/>
+            <joint name="right_hand_base_joint" type="fixed">
+                <origin rpy="0 0 ${-PI/2}"/>
+                <parent link="right_tcp"/>
+                <child link="right_hand_flange"/>
+            </joint>
+        </xacro:if>
+        <!-- 灵巧手类型 -->
+        <xacro:if value="${hand_type == 'linkerhand_l6'}">
+            <xacro:include filename="$(find linkerhand_description)/xacro/l6.xacro"/>
+            <xacro:LinkerHandL6 name="left_hand" direction="1" use_flange="true" fixed_joints="false"/>
+            <joint name="left_hand_base_joint" type="fixed">
+                <origin xyz="0 0 0.0045" rpy="0 0 ${PI}"/>
+                <parent link="left_tcp"/>
+                <child link="left_hand_flange"/>
+            </joint>
+            <xacro:LinkerHandL6 name="right_hand" direction="-1" use_flange="true" fixed_joints="false"/>
+            <joint name="right_hand_base_joint" type="fixed">
+                <parent link="right_tcp"/>
+                <child link="right_hand_flange"/>
+                <origin xyz="0 0 0.0045"/>
+            </joint>
+        </xacro:if>
+    </xacro:macro>
 </robot>

File: xacro/ros2_control/robot.xacro (robot description, xacro)
@@ -2,23 +2,16 @@
 <robot name="fiveages_w2" xmlns:xacro="http://www.ros.org/wiki/xacro">
 	<xacro:arg name="ros2_control_hardware_type" default="mock_components"/>
+	<xacro:arg name="device_ip" default="192.168.1.190"/>
+	<xacro:property name="device_ip_arg" value="$(arg device_ip)"/>
 	<xacro:include filename="$(find fiveages_w2_description)/xacro/robot.xacro"/>
 	<xacro:include filename="$(find m6_ccs_description)/xacro/ros2_control/interfaces.xacro"/>
 	<xacro:include filename="$(find fiveages_w2_description)/xacro/ros2_control/body.xacro"/>
-	<xacro:if value="${'$(arg ros2_control_hardware_type)' == 'real'}">
+	<xacro:if value="${'$(arg ros2_control_hardware_type)' == 'real' or '$(arg ros2_control_hardware_type)' == 'real_usb'}">
 		<!-- 确定传递给 marvin_ros2_control 的 gripper_type 参数 -->
 		<!--
-			Marvin 模式下的手部控制逻辑：
-			1. 如果 hand_control_mode == 'marvin' 且 selected_hand_type 不为空，
-			   则将 selected_hand_type (如 linkerhand_o7) 传递给 MarvinHardware 的 gripper_type 参数
-			2. MarvinHardware 会通过 normalizeString() 将 gripper_type 转换为大写
-			3. 在 createTool() 和 contains_gripper() 中检测 gripper_type 是否包含 "LINKERHAND" 或 "HAND"
-			4. 如果检测到手部类型，MarvinHardware 会创建对应的 DexterousHand 对象（O7/O6/L6）
-			5. 手的控制通过 485 总线完成，不需要独立的 modbus_ros2_control 系统
+			手部控制模式由 ros2_control_hardware_type 决定：
+			- hardware=real      : 485/marvin（手作为 MarvinHardware 的 tool，由 gripper_type 传入）
+			- hardware=real_usb  : USB/modbus（手由独立 modbus_ros2_control 系统控制，MarvinHardware 只管机械臂）
 		-->
-		<xacro:property name="marvin_gripper_type" value="${selected_gripper_type}"/>
-		<xacro:if value="${selected_hand_type != '' and hand_control_mode_arg == 'marvin'}">
-			<!-- marvin 模式下，将手部类型传递给 gripper_type，让 MarvinHardware 检测并创建手部对象 -->
-			<xacro:property name="marvin_gripper_type" value="${selected_hand_type}"/>
-		</xacro:if>
 		<ros2_control name="M6_CCS_System" type="system">
 			<hardware>
@@ -32,5 +25,6 @@
 					- MarvinHardware 会自动检测 gripper_type 中是否包含 "LINKERHAND" 或 "HAND" 来判断是手部还是夹爪
 				-->
-				<param name="gripper_type">${marvin_gripper_type}</param>
+				<!-- 485/marvin(real) + hand: pass hand type; otherwise pass gripper type (or empty). -->
+				<param name="gripper_type">${selected_hand_type if (selected_hand_type != '' and '$(arg ros2_control_hardware_type)' == 'real') else selected_gripper_type}</param>
 				<param name="max_joint_speed">50</param>
 				<param name="max_joint_acceleration">30</param>
@@ -38,5 +32,5 @@
 				<param name="left_dyn_param">0.4,0,0,50.65,0,0,0,0,0,0</param>
 				<param name="right_dyn_param">0.4,0,0,50.85,0,0,0,0,0,0</param>
-				<param name="device_ip"></param>
+				<param name="device_ip">${device_ip_arg}</param>
 			</hardware>
 			<xacro:m6_interfaces name="left"/>
@@ -57,11 +51,6 @@
 				</joint>
 			</xacro:if>
-			<!--
-				灵巧手接口：通过天机硬件控制（marvin 模式）
-				注意：这些接口会被添加到 M6_CCS_System 中，MarvinHardware 会通过 gripper_type 参数
-				检测到手部类型，并创建对应的 DexterousHand 对象来控制这些关节。
-				控制通过 485 总线完成，不需要 modbus_ros2_control。
-			-->
-			<xacro:if value="${selected_hand_type != '' and hand_control_mode_arg == 'marvin'}">
+			<!-- 灵巧手接口：485/marvin（通过 M6_CCS_System） -->
+			<xacro:if value="${selected_hand_type != '' and '$(arg ros2_control_hardware_type)' == 'real'}">
 				<xacro:if value="${selected_hand_type == 'linkerhand_o6' or selected_hand_type == 'linkerhand_l6'}">
 					<xacro:include filename="$(find linkerhand_description)/xacro/ros2_control/o6.xacro"/>
@@ -88,8 +77,7 @@
 			<xacro:body_interfaces/>
 		</ros2_control>
-		<!-- 灵巧手接口：通过 USB (modbus_ros2_control) -->
-		<!-- 只有在 hand_control_mode 明确为 'usb' 时才创建 modbus 系统 -->
-		<!-- 注意：marvin 模式下，手的控制通过 M6_CCS_System 中的 MarvinHardware 完成，不需要 modbus 系统 -->
-		<xacro:if value="${selected_hand_type != '' and hand_control_mode_arg == 'usb'}">
+		<!-- 灵巧手接口：USB 模式（hardware=real_usb，modbus_ros2_control），直接内联 ros2_control 配置 -->
+		<xacro:if value="${selected_hand_type != '' and '$(arg ros2_control_hardware_type)' == 'real_usb'}">
+			<!-- O6/L6: 6-DOF 手 -->
 			<xacro:if value="${selected_hand_type == 'linkerhand_o6' or selected_hand_type == 'linkerhand_l6'}">
 				<xacro:include filename="$(find linkerhand_description)/xacro/ros2_control/o6.xacro"/>
@@ -115,4 +103,5 @@
 				</ros2_control>
 			</xacro:if>
+			<!-- O7: 7-DOF 手 -->
 			<xacro:if value="${selected_hand_type == 'linkerhand_o7'}">
 				<xacro:include filename="$(find linkerhand_description)/xacro/ros2_control/o7.xacro"/>
@@ -140,5 +129,5 @@
 		</xacro:if>
 	</xacro:if>
-	<xacro:unless value="${'$(arg ros2_control_hardware_type)' == 'real'}">
+	<xacro:unless value="${'$(arg ros2_control_hardware_type)' == 'real' or '$(arg ros2_control_hardware_type)' == 'real_usb'}">
 		<ros2_control name="fiveages_w2_system" type="system">
 			<hardware>
@@ -182,9 +171,4 @@
 				<xacro:linkerhand_o7_interfaces name="right_hand"/>
 			</xacro:if>
-			<xacro:if value="${selected_hand_type == 'linkerhand_o7'}">
-				<xacro:include filename="$(find linkerhand_description)/xacro/ros2_control/o7.xacro"/>
-				<xacro:linkerhand_o7_interfaces name="left_hand"/>
-				<xacro:linkerhand_o7_interfaces name="right_hand"/>
-			</xacro:if>
 		</ros2_control>
 	</xacro:unless>
