Commit message: Feature/add o7 hand (#2)
* update xacro file for IP and hand ctrl

* add support for o7 hand

* Update xacro file to support marvin 485 communication

* Update xacro file to support marvin 485 communication

* Update xacro file to support marvin 485 communication

* fix xacro problem

* fix xacro hand usb interface selection

Normalize usb hand series comparisons to string values so o6/o7 interface macros are expanded reliably in real_usb mode.

Made-with: Cursor

---------

Co-authored-by: hja <2486401522@qq.com>
Co-authored-by: wuyidong <wuyidong@fiveages.com>

File: xacro/robot.xacro (robot description, xacro)
@@ -1,60 +1,60 @@
 <?xml version="1.0"?>
 <robot name="FiveAges W2" xmlns:xacro="http://www.ros.org/wiki/xacro">
-	<xacro:arg name="collider" default="convex"/>
-	<xacro:arg name="chassis_joints_movable" default="false"/>
-	<!-- 从 type 参数解析出 hand_type 和 gripper_type -->
-	<xacro:arg name="type" default=""/>
-	<xacro:property name="type_arg" value="$(arg type)"/>
-	<!-- 默认值 -->
-	<xacro:property name="selected_hand_type" value=""/>
-	<xacro:property name="selected_gripper_type" value=""/>
-	<xacro:property name="selected_gripper_pad" value="default"/>
-	<!-- 从 type 解析 hand_type 和 gripper_type -->
-	<!-- 夹爪类型：selected_gripper_type 不为空即表示使用夹爪 -->
-	<xacro:if value="${type_arg == 'rg75'}">
-		<xacro:property name="selected_gripper_type" value="rg75"/>
-	</xacro:if>
-	<xacro:if value="${type_arg == 'rg75_heavy'}">
-		<xacro:property name="selected_gripper_type" value="rg75"/>
-		<xacro:property name="selected_gripper_pad" value="heavy_carry"/>
-	</xacro:if>
-	<xacro:if value="${type_arg == 'ag2f90'}">
-		<xacro:property name="selected_gripper_type" value="ag2f90_d"/>
-	</xacro:if>
-	<xacro:if value="${type_arg == 'ag2f90_c'}">
-		<xacro:property name="selected_gripper_type" value="ag2f90_c"/>
-	</xacro:if>
-	<xacro:if value="${type_arg == 'ag2f90_d'}">
-		<xacro:property name="selected_gripper_type" value="ag2f90_d"/>
-	</xacro:if>
-	<!-- 灵巧手类型 -->
-	<xacro:if value="${type_arg == 'linkerhand_o6'}">
-		<xacro:property name="selected_hand_type" value="linkerhand_o6"/>
-	</xacro:if>
-	<xacro:if value="${type_arg == 'linkerhand_l6'}">
-		<xacro:property name="selected_hand_type" value="linkerhand_l6"/>
-	</xacro:if>
-	<xacro:if value="${type_arg == 'linkerhand_o7'}">
-		<xacro:property name="selected_hand_type" value="linkerhand_o7"/>
-	</xacro:if>
-	<xacro:include filename="$(find fiveages_w2_description)/xacro/components/linkhou_s2.xacro"/>
-	<xacro:linkhou_s2 joints_movable="$(arg chassis_joints_movable)"/>
-	<xacro:include filename="$(find fiveages_w2_description)/xacro/components/body.xacro"/>
-	<!-- Left Arm -->
-	<joint name="left_arm_base_joint" type="fixed">
-		<parent link="arm_base"/>
-		<child link="left_base_link"/>
-		<origin rpy="-${PI/2} 0 0" xyz="0.0 0.062 0"/>
-	</joint>
-	<!-- Right Arm -->
-	<joint name="right_arm_base_joint" type="fixed">
-		<parent link="arm_base"/>
-		<child link="right_base_link"/>
-		<origin rpy="${PI/2} 0 0" xyz="0 -0.062 0"/>
-	</joint>
-	<xacro:include filename="$(find m6_ccs_description)/xacro/arm.xacro"/>
-	<xacro:M6_CCS name="left" style="fiveages_w2"/>
-	<xacro:M6_CCS name="right" direction="-1" style="fiveages_w2"/>
-	<xacro:include filename="$(find fiveages_w2_description)/xacro/eefs.xacro"/>
-	<xacro:EndEffectors hand_type="${selected_hand_type}" gripper_type="${selected_gripper_type}"/>
+    <xacro:arg name="collider" default="convex"/>
+    <xacro:arg name="chassis_joints_movable" default="false"/>
+    <!-- 从 type 参数解析出 hand_type 和 gripper_type -->
+    <xacro:arg name="type" default=""/>
+    <xacro:property name="type_arg" value="$(arg type)"/>
+    <!-- 默认值 -->
+    <xacro:property name="selected_hand_type" value=""/>
+    <xacro:property name="selected_gripper_type" value=""/>
+    <xacro:property name="selected_gripper_pad" value="default"/>
+    <!-- 从 type 解析 hand_type 和 gripper_type -->
+    <!-- 夹爪类型：selected_gripper_type 不为空即表示使用夹爪 -->
+    <xacro:if value="${type_arg == 'rg75'}">
+        <xacro:property name="selected_gripper_type" value="rg75"/>
+    </xacro:if>
+    <xacro:if value="${type_arg == 'rg75_heavy'}">
+        <xacro:property name="selected_gripper_type" value="rg75"/>
+        <xacro:property name="selected_gripper_pad" value="heavy_carry"/>
+    </xacro:if>
+    <xacro:if value="${type_arg == 'ag2f90'}">
+        <xacro:property name="selected_gripper_type" value="ag2f90_d"/>
+    </xacro:if>
+    <xacro:if value="${type_arg == 'ag2f90_c'}">
+        <xacro:property name="selected_gripper_type" value="ag2f90_c"/>
+    </xacro:if>
+    <xacro:if value="${type_arg == 'ag2f90_d'}">
+        <xacro:property name="selected_gripper_type" value="ag2f90_d"/>
+    </xacro:if>
+    <!-- 灵巧手类型 -->
+    <xacro:if value="${type_arg == 'linkerhand_o6'}">
+        <xacro:property name="selected_hand_type" value="linkerhand_o6"/>
+    </xacro:if>
+    <xacro:if value="${type_arg == 'linkerhand_l6'}">
+        <xacro:property name="selected_hand_type" value="linkerhand_l6"/>
+    </xacro:if>
+    <xacro:if value="${type_arg == 'linkerhand_o7'}">
+        <xacro:property name="selected_hand_type" value="linkerhand_o7"/>
+    </xacro:if>
+    <xacro:include filename="$(find fiveages_w2_description)/xacro/components/linkhou_s2.xacro"/>
+    <xacro:linkhou_s2 joints_movable="$(arg chassis_joints_movable)"/>
+    <xacro:include filename="$(find fiveages_w2_description)/xacro/components/body.xacro"/>
+    <!-- Left Arm -->
+    <joint name="left_arm_base_joint" type="fixed">
+        <parent link="arm_base"/>
+        <child link="left_base_link"/>
+        <origin rpy="-${PI/2} 0 0" xyz="0.0 0.062 0"/>
+    </joint>
+    <!-- Right Arm -->
+    <joint name="right_arm_base_joint" type="fixed">
+        <parent link="arm_base"/>
+        <child link="right_base_link"/>
+        <origin rpy="${PI/2} 0 0" xyz="0 -0.062 0"/>
+    </joint>
+    <xacro:include filename="$(find m6_ccs_description)/xacro/arm.xacro"/>
+    <xacro:M6_CCS name="left" style="fiveages_w2"/>
+    <xacro:M6_CCS name="right" direction="-1" style="fiveages_w2"/>
+    <xacro:include filename="$(find fiveages_w2_description)/xacro/eefs.xacro"/>
+    <xacro:EndEffectors hand_type="${selected_hand_type}" gripper_type="${selected_gripper_type}"/>
 </robot>

File: xacro/ros2_control/robot.xacro (robot description, xacro)
@@ -2,8 +2,16 @@
 <robot name="fiveages_w2" xmlns:xacro="http://www.ros.org/wiki/xacro">
 	<xacro:arg name="ros2_control_hardware_type" default="mock_components"/>
+	<xacro:property name="is_real_hardware" value="${'$(arg ros2_control_hardware_type)' == 'real' or '$(arg ros2_control_hardware_type)' == 'real_usb'}"/>
+	<xacro:property name="ee_drive_type" value="${'usb' if '$(arg ros2_control_hardware_type)' == 'real_usb' else ('marvin' if '$(arg ros2_control_hardware_type)' == 'real' else '')}"/>
 	<xacro:include filename="$(find fiveages_w2_description)/xacro/robot.xacro"/>
 	<xacro:include filename="$(find m6_ccs_description)/xacro/ros2_control/interfaces.xacro"/>
 	<xacro:include filename="$(find fiveages_w2_description)/xacro/ros2_control/body.xacro"/>
-	<xacro:if value="${'$(arg ros2_control_hardware_type)' == 'real'}">
+	<xacro:if value="${is_real_hardware}">
+		<!-- 确定传递给 marvin_ros2_control 的 gripper_type 参数 -->
+		<!--
+			手部控制模式由 ros2_control_hardware_type 决定：
+			- hardware=real      : 485/marvin（手作为 MarvinHardware 的 tool，由 gripper_type 传入）
+			- hardware=real_usb  : USB/modbus（手由独立 modbus_ros2_control 系统控制，MarvinHardware 只管机械臂）
+		-->
 		<ros2_control name="M6_CCS_System" type="system">
 			<hardware>
@@ -11,5 +19,12 @@
 				<param name="arm_type">dual</param>
 				<param name="ctrl_mode">position</param>
-				<param name="gripper_type">${selected_gripper_type}</param>
+				<!--
+					gripper_type 参数说明：
+					- 如果是夹爪：传递夹爪类型（如 rg75, ag2f90_c 等）
+					- 如果是 marvin 模式的手部：传递手部类型（如 linkerhand_o7, linkerhand_o6, linkerhand_l6）
+					- MarvinHardware 会自动检测 gripper_type 中是否包含 "LINKERHAND" 或 "HAND" 来判断是手部还是夹爪
+				-->
+				<!-- 485/marvin(real) + hand: pass hand type; otherwise pass gripper type (or empty). -->
+				<param name="gripper_type">${selected_hand_type if ee_drive_type == 'marvin' else selected_gripper_type}</param>
 				<param name="max_joint_speed">50</param>
 				<param name="max_joint_acceleration">30</param>
@@ -17,4 +32,5 @@
 				<param name="left_dyn_param">0.4,0,0,50.65,0,0,0,0,0,0</param>
 				<param name="right_dyn_param">0.4,0,0,50.85,0,0,0,0,0,0</param>
+				<param name="device_ip">192.168.1.190</param>
 			</hardware>
 			<xacro:m6_interfaces name="left"/>
@@ -35,5 +51,17 @@
 				</joint>
 			</xacro:if>
-			<!-- 灵巧手接口 -->
+			<!-- 灵巧手接口：485/marvin（通过 M6_CCS_System） -->
+			<xacro:if value="${ee_drive_type == 'marvin'}">
+				<xacro:if value="${selected_hand_type in ['linkerhand_o6', 'linkerhand_l6']}">
+					<xacro:include filename="$(find linkerhand_description)/xacro/ros2_control/o6.xacro"/>
+					<xacro:linkerhand_o6_interfaces name="left_hand"/>
+					<xacro:linkerhand_o6_interfaces name="right_hand"/>
+				</xacro:if>
+				<xacro:if value="${selected_hand_type == 'linkerhand_o7'}">
+					<xacro:include filename="$(find linkerhand_description)/xacro/ros2_control/o7.xacro"/>
+					<xacro:linkerhand_o7_interfaces name="left_hand"/>
+					<xacro:linkerhand_o7_interfaces name="right_hand"/>
+				</xacro:if>
+			</xacro:if>
 		</ros2_control>
 		<ros2_control name="juxie_body" type="system">
@@ -49,29 +77,48 @@
 			<xacro:body_interfaces/>
 		</ros2_control>
-		<xacro:if value="${selected_hand_type == 'linkerhand_o6' or selected_hand_type == 'linkerhand_l6'}">
-			<xacro:include filename="$(find linkerhand_description)/xacro/ros2_control/o6.xacro"/>
-			<ros2_control name="linkerhand_6_left_system" type="system">
-				<hardware>
-					<plugin>modbus_ros2_control/DexterousHandHardware</plugin>
-					<param name="serial_port">/dev/ttyUSB1</param>
-					<param name="hand_type">${selected_hand_type}</param>
-					<param name="hand_side">left</param>
-					<param name="max_speed_ratio">1.0</param>
-				</hardware>
-				<xacro:linkerhand_o6_interfaces name="left_hand"/>
-			</ros2_control>
-			<ros2_control name="linkerhand_6_right_system" type="system">
-				<hardware>
-					<plugin>modbus_ros2_control/DexterousHandHardware</plugin>
-					<param name="serial_port">/dev/ttyUSB0</param>
-					<param name="hand_type">${selected_hand_type}</param>
-					<param name="hand_side">right</param>
-					<param name="max_speed_ratio">1.0</param>
-				</hardware>
-				<xacro:linkerhand_o6_interfaces name="right_hand"/>
-			</ros2_control>
+		<!-- 灵巧手接口：USB 模式（hardware=real_usb，modbus_ros2_control），直接内联 ros2_control 配置 -->
+		<xacro:if value="${ee_drive_type == 'usb'}">
+			<xacro:if value="${selected_hand_type in ('linkerhand_o6', 'linkerhand_l6', 'linkerhand_o7')}">
+				<xacro:property name="usb_hand_series" value="${str('7' if selected_hand_type == 'linkerhand_o7' else '6')}"/>
+				<xacro:if value="${str(usb_hand_series) == '6'}">
+					<xacro:include filename="$(find linkerhand_description)/xacro/ros2_control/o6.xacro"/>
+				</xacro:if>
+				<xacro:if value="${str(usb_hand_series) == '7'}">
+					<xacro:include filename="$(find linkerhand_description)/xacro/ros2_control/o7.xacro"/>
+				</xacro:if>
+				<ros2_control name="linkerhand_${usb_hand_series}_left_system" type="system">
+					<hardware>
+						<plugin>modbus_ros2_control/DexterousHandHardware</plugin>
+						<param name="serial_port">/dev/ttyUSB0</param>
+						<param name="hand_type">${selected_hand_type}</param>
+						<param name="hand_side">left</param>
+						<param name="max_speed_ratio">1.0</param>
+					</hardware>
+					<xacro:if value="${str(usb_hand_series) == '6'}">
+						<xacro:linkerhand_o6_interfaces name="left_hand"/>
+					</xacro:if>
+					<xacro:if value="${str(usb_hand_series) == '7'}">
+						<xacro:linkerhand_o7_interfaces name="left_hand"/>
+					</xacro:if>
+				</ros2_control>
+				<ros2_control name="linkerhand_${usb_hand_series}_right_system" type="system">
+					<hardware>
+						<plugin>modbus_ros2_control/DexterousHandHardware</plugin>
+						<param name="serial_port">/dev/ttyUSB2</param>
+						<param name="hand_type">${selected_hand_type}</param>
+						<param name="hand_side">right</param>
+						<param name="max_speed_ratio">1.0</param>
+					</hardware>
+					<xacro:if value="${str(usb_hand_series) == '6'}">
+						<xacro:linkerhand_o6_interfaces name="right_hand"/>
+					</xacro:if>
+					<xacro:if value="${str(usb_hand_series) == '7'}">
+						<xacro:linkerhand_o7_interfaces name="right_hand"/>
+					</xacro:if>
+				</ros2_control>
+			</xacro:if>
 		</xacro:if>
 	</xacro:if>
-	<xacro:unless value="${'$(arg ros2_control_hardware_type)' == 'real'}">
+	<xacro:unless value="${is_real_hardware}">
 		<ros2_control name="fiveages_w2_system" type="system">
 			<hardware>
@@ -99,5 +146,5 @@
 				<xacro:rg75_interfaces name="right"/>
 			</xacro:if>
-			<xacro:if value="${selected_gripper_type == 'ag2f90_c' or selected_gripper_type == 'ag2f90_d'}">
+			<xacro:if value="${selected_gripper_type in ('ag2f90_c', 'ag2f90_d')}">
 				<xacro:include filename="$(find changingtek_description)/xacro/ros2_control/AG2F90-C.xacro"/>
 				<xacro:ag2f90c_interfaces name="left"/>
@@ -105,5 +152,5 @@
 			</xacro:if>
 			<!-- 灵巧手接口 -->
-			<xacro:if value="${selected_hand_type == 'linkerhand_o6' or selected_hand_type == 'linkerhand_l6'}">
+			<xacro:if value="${selected_hand_type in ['linkerhand_o6', 'linkerhand_l6']}">
 				<xacro:include filename="$(find linkerhand_description)/xacro/ros2_control/o6.xacro"/>
 				<xacro:linkerhand_o6_interfaces name="left_hand"/>
