Commit message: add linkerhand l6

File: xacro/eefs.xacro (robot description, xacro)
@@ -54,5 +54,5 @@
             <xacro:LinkerHandO6 name="left_hand" direction="1" use_flange="true" fixed_joints="false"/>
             <joint name="left_hand_base_joint" type="fixed">
-                <origin xyz="0 0 0.0045" rpy="0 0 3.1415926535"/>
+                <origin xyz="0 0 0.0045" rpy="0 0 ${PI/2}"/>
                 <parent link="left_tcp"/>
                 <child link="left_hand_flange"/>
@@ -62,5 +62,21 @@
                 <parent link="right_tcp"/>
                 <child link="right_hand_flange"/>
-                <origin xyz="0 0 0.0045"/>
+                <origin xyz="0 0 0.0045" rpy="0 0 ${-PI/2}"/>
+            </joint>
+        </xacro:if>
+        <!-- 灵巧手类型 -->
+        <xacro:if value="${hand_type == 'linkerhand_l6'}">
+            <xacro:include filename="$(find linkerhand_description)/xacro/l6.xacro"/>
+            <xacro:LinkerHandL6 name="left_hand" direction="1" use_flange="true" fixed_joints="false"/>
+            <joint name="left_hand_base_joint" type="fixed">
+                <origin xyz="0 0 0.0045" rpy="0 0 ${PI/2}"/>
+                <parent link="left_tcp"/>
+                <child link="left_hand_flange"/>
+            </joint>
+            <xacro:LinkerHandL6 name="right_hand" direction="-1" use_flange="true" fixed_joints="false"/>
+            <joint name="right_hand_base_joint" type="fixed">
+                <parent link="right_tcp"/>
+                <child link="right_hand_flange"/>
+                <origin xyz="0 0 0.0045" rpy="0 0 ${-PI/2}"/>
             </joint>
         </xacro:if>

File: xacro/robot.xacro (robot description, xacro)
@@ -45,4 +45,7 @@
 		<xacro:property name="selected_hand_type" value="linkerhand_o6"/>
 	</xacro:if>
+	<xacro:if value="${type_arg == 'linkerhand_l6'}">
+		<xacro:property name="selected_hand_type" value="linkerhand_l6"/>
+	</xacro:if>
 	<xacro:include filename="$(find fiveages_w2_description)/xacro/eefs.xacro"/>
 	<xacro:EndEffectors hand_type="${selected_hand_type}" gripper_type="${selected_gripper_type}"/>

File: xacro/ros2_control/robot.xacro (robot description, xacro)
@@ -33,5 +33,5 @@
 			</xacro:if>
 			<!-- 灵巧手接口 -->
-			<xacro:if value="${selected_hand_type == 'linkerhand_o6'}">
+			<xacro:if value="${selected_hand_type == 'linkerhand_o6' or selected_hand_type == 'linkerhand_l6'}">
 				<xacro:include filename="$(find linkerhand_description)/xacro/ros2_control/o6.xacro"/>
 				<xacro:linkerhand_o6_interfaces name="left_hand"/>
@@ -84,5 +84,5 @@
 			</xacro:if>
 			<!-- 灵巧手接口 -->
-			<xacro:if value="${selected_hand_type == 'linkerhand_o6'}">
+			<xacro:if value="${selected_hand_type == 'linkerhand_o6' or selected_hand_type == 'linkerhand_l6'}">
 				<xacro:include filename="$(find linkerhand_description)/xacro/ros2_control/o6.xacro"/>
 				<xacro:linkerhand_o6_interfaces name="left_hand"/>

Commit message: modified default pose

File: xacro/eefs.xacro (robot description, xacro)
@@ -54,5 +54,5 @@
             <xacro:LinkerHandO6 name="left_hand" direction="1" use_flange="true" fixed_joints="false"/>
             <joint name="left_hand_base_joint" type="fixed">
-                <origin xyz="0 0 0.0045" rpy="0 0 ${PI/2}"/>
+                <origin xyz="0 0 0.0045" rpy="0 0 ${PI}"/>
                 <parent link="left_tcp"/>
                 <child link="left_hand_flange"/>
@@ -62,5 +62,5 @@
                 <parent link="right_tcp"/>
                 <child link="right_hand_flange"/>
-                <origin xyz="0 0 0.0045" rpy="0 0 ${-PI/2}"/>
+                <origin xyz="0 0 0.0045"/>
             </joint>
         </xacro:if>
@@ -70,5 +70,5 @@
             <xacro:LinkerHandL6 name="left_hand" direction="1" use_flange="true" fixed_joints="false"/>
             <joint name="left_hand_base_joint" type="fixed">
-                <origin xyz="0 0 0.0045" rpy="0 0 ${PI/2}"/>
+                <origin xyz="0 0 0.0045" rpy="0 0 ${PI}"/>
                 <parent link="left_tcp"/>
                 <child link="left_hand_flange"/>
@@ -78,5 +78,5 @@
                 <parent link="right_tcp"/>
                 <child link="right_hand_flange"/>
-                <origin xyz="0 0 0.0045" rpy="0 0 ${-PI/2}"/>
+                <origin xyz="0 0 0.0045"/>
             </joint>
         </xacro:if>

Commit message: add support for o7 hand

File: xacro/eefs.xacro (robot description, xacro)
@@ -96,4 +96,20 @@
             </joint>
         </xacro:if>
+        <!-- 灵巧手类型 -->
+        <xacro:if value="${hand_type == 'linkerhand_o7'}">
+            <xacro:include filename="$(find linkerhand_description)/xacro/o7.xacro"/>
+            <xacro:LinkerHandO7 name="left_hand" direction="1" use_flange="true" fixed_joints="false"/>
+            <joint name="left_hand_base_joint" type="fixed">
+                <origin xyz="0 0 0.0045" rpy="0 0 ${PI/2}"/>
+                <parent link="left_tcp"/>
+                <child link="left_hand_flange"/>
+            </joint>
+            <xacro:LinkerHandO7 name="right_hand" direction="-1" use_flange="true" fixed_joints="false"/>
+            <joint name="right_hand_base_joint" type="fixed">
+                <parent link="right_tcp"/>
+                <child link="right_hand_flange"/>
+                <origin xyz="0 0 0.0045" rpy="0 0 ${-PI/2}"/>
+            </joint>
+        </xacro:if>
     </xacro:macro>
 </robot>

File: xacro/robot.xacro (robot description, xacro)
@@ -6,4 +6,7 @@
 	<xacro:arg name="type" default=""/>
 	<xacro:property name="type_arg" value="$(arg type)"/>
+	<!-- 手部控制方式：usb 或 marvin -->
+	<xacro:arg name="hand_control_mode" default="usb"/>
+	<xacro:property name="hand_control_mode_arg" value="$(arg hand_control_mode)"/>
 	<!-- 默认值 -->
 	<xacro:property name="selected_hand_type" value=""/>

File: xacro/ros2_control/robot.xacro (robot description, xacro)
@@ -6,4 +6,19 @@
 	<xacro:include filename="$(find fiveages_w2_description)/xacro/ros2_control/body.xacro"/>
 	<xacro:if value="${'$(arg ros2_control_hardware_type)' == 'real'}">
+		<!-- 确定传递给 marvin_ros2_control 的 gripper_type 参数 -->
+		<!--
+			Marvin 模式下的手部控制逻辑：
+			1. 如果 hand_control_mode == 'marvin' 且 selected_hand_type 不为空，
+			   则将 selected_hand_type (如 linkerhand_o7) 传递给 MarvinHardware 的 gripper_type 参数
+			2. MarvinHardware 会通过 normalizeString() 将 gripper_type 转换为大写
+			3. 在 createTool() 和 contains_gripper() 中检测 gripper_type 是否包含 "LINKERHAND" 或 "HAND"
+			4. 如果检测到手部类型，MarvinHardware 会创建对应的 DexterousHand 对象（O7/O6/L6）
+			5. 手的控制通过 485 总线完成，不需要独立的 modbus_ros2_control 系统
+		-->
+		<xacro:property name="marvin_gripper_type" value="${selected_gripper_type}"/>
+		<xacro:if value="${selected_hand_type != '' and hand_control_mode_arg == 'marvin'}">
+			<!-- marvin 模式下，将手部类型传递给 gripper_type，让 MarvinHardware 检测并创建手部对象 -->
+			<xacro:property name="marvin_gripper_type" value="${selected_hand_type}"/>
+		</xacro:if>
 		<ros2_control name="M6_CCS_System" type="system">
 			<hardware>
@@ -11,5 +26,11 @@
 				<param name="arm_type">dual</param>
 				<param name="ctrl_mode">position</param>
-				<param name="gripper_type">${selected_gripper_type}</param>
+				<!--
+					gripper_type 参数说明：
+					- 如果是夹爪：传递夹爪类型（如 rg75, ag2f90_c 等）
+					- 如果是 marvin 模式的手部：传递手部类型（如 linkerhand_o7, linkerhand_o6, linkerhand_l6）
+					- MarvinHardware 会自动检测 gripper_type 中是否包含 "LINKERHAND" 或 "HAND" 来判断是手部还是夹爪
+				-->
+				<param name="gripper_type">${marvin_gripper_type}</param>
 				<param name="max_joint_speed">50</param>
 				<param name="max_joint_acceleration">30</param>
@@ -17,4 +38,5 @@
 				<param name="left_dyn_param">0.4,0,0,50.65,0,0,0,0,0,0</param>
 				<param name="right_dyn_param">0.4,0,0,50.85,0,0,0,0,0,0</param>
+				<param name="device_ip"></param>
 			</hardware>
 			<xacro:m6_interfaces name="left"/>
@@ -35,5 +57,22 @@
 				</joint>
 			</xacro:if>
-			<!-- 灵巧手接口 -->
+			<!--
+				灵巧手接口：通过天机硬件控制（marvin 模式）
+				注意：这些接口会被添加到 M6_CCS_System 中，MarvinHardware 会通过 gripper_type 参数
+				检测到手部类型，并创建对应的 DexterousHand 对象来控制这些关节。
+				控制通过 485 总线完成，不需要 modbus_ros2_control。
+			-->
+			<xacro:if value="${selected_hand_type != '' and hand_control_mode_arg == 'marvin'}">
+				<xacro:if value="${selected_hand_type == 'linkerhand_o6' or selected_hand_type == 'linkerhand_l6'}">
+					<xacro:include filename="$(find linkerhand_description)/xacro/ros2_control/o6.xacro"/>
+					<xacro:linkerhand_o6_interfaces name="left_hand"/>
+					<xacro:linkerhand_o6_interfaces name="right_hand"/>
+				</xacro:if>
+				<xacro:if value="${selected_hand_type == 'linkerhand_o7'}">
+					<xacro:include filename="$(find linkerhand_description)/xacro/ros2_control/o7.xacro"/>
+					<xacro:linkerhand_o7_interfaces name="left_hand"/>
+					<xacro:linkerhand_o7_interfaces name="right_hand"/>
+				</xacro:if>
+			</xacro:if>
 		</ros2_control>
 		<ros2_control name="juxie_body" type="system">
@@ -49,26 +88,54 @@
 			<xacro:body_interfaces/>
 		</ros2_control>
-		<xacro:if value="${selected_hand_type == 'linkerhand_o6' or selected_hand_type == 'linkerhand_l6'}">
-			<xacro:include filename="$(find linkerhand_description)/xacro/ros2_control/o6.xacro"/>
-			<ros2_control name="linkerhand_6_left_system" type="system">
-				<hardware>
-					<plugin>modbus_ros2_control/DexterousHandHardware</plugin>
-					<param name="serial_port">/dev/ttyUSB1</param>
-					<param name="hand_type">${selected_hand_type}</param>
-					<param name="hand_side">left</param>
-					<param name="max_speed_ratio">1.0</param>
-				</hardware>
-				<xacro:linkerhand_o6_interfaces name="left_hand"/>
-			</ros2_control>
-			<ros2_control name="linkerhand_6_right_system" type="system">
-				<hardware>
-					<plugin>modbus_ros2_control/DexterousHandHardware</plugin>
-					<param name="serial_port">/dev/ttyUSB0</param>
-					<param name="hand_type">${selected_hand_type}</param>
-					<param name="hand_side">right</param>
-					<param name="max_speed_ratio">1.0</param>
-				</hardware>
-				<xacro:linkerhand_o6_interfaces name="right_hand"/>
-			</ros2_control>
+		<!-- 灵巧手接口：通过 USB (modbus_ros2_control) -->
+		<!-- 只有在 hand_control_mode 明确为 'usb' 时才创建 modbus 系统 -->
+		<!-- 注意：marvin 模式下，手的控制通过 M6_CCS_System 中的 MarvinHardware 完成，不需要 modbus 系统 -->
+		<xacro:if value="${selected_hand_type != '' and hand_control_mode_arg == 'usb'}">
+			<xacro:if value="${selected_hand_type == 'linkerhand_o6' or selected_hand_type == 'linkerhand_l6'}">
+				<xacro:include filename="$(find linkerhand_description)/xacro/ros2_control/o6.xacro"/>
+				<ros2_control name="linkerhand_6_left_system" type="system">
+					<hardware>
+						<plugin>modbus_ros2_control/DexterousHandHardware</plugin>
+						<param name="serial_port">/dev/ttyUSB1</param>
+						<param name="hand_type">${selected_hand_type}</param>
+						<param name="hand_side">left</param>
+						<param name="max_speed_ratio">1.0</param>
+					</hardware>
+					<xacro:linkerhand_o6_interfaces name="left_hand"/>
+				</ros2_control>
+				<ros2_control name="linkerhand_6_right_system" type="system">
+					<hardware>
+						<plugin>modbus_ros2_control/DexterousHandHardware</plugin>
+						<param name="serial_port">/dev/ttyUSB0</param>
+						<param name="hand_type">${selected_hand_type}</param>
+						<param name="hand_side">right</param>
+						<param name="max_speed_ratio">1.0</param>
+					</hardware>
+					<xacro:linkerhand_o6_interfaces name="right_hand"/>
+				</ros2_control>
+			</xacro:if>
+			<xacro:if value="${selected_hand_type == 'linkerhand_o7'}">
+				<xacro:include filename="$(find linkerhand_description)/xacro/ros2_control/o7.xacro"/>
+				<ros2_control name="linkerhand_7_left_system" type="system">
+					<hardware>
+						<plugin>modbus_ros2_control/DexterousHandHardware</plugin>
+						<param name="serial_port">/dev/ttyUSB1</param>
+						<param name="hand_type">${selected_hand_type}</param>
+						<param name="hand_side">left</param>
+						<param name="max_speed_ratio">1.0</param>
+					</hardware>
+					<xacro:linkerhand_o7_interfaces name="left_hand"/>
+				</ros2_control>
+				<ros2_control name="linkerhand_7_right_system" type="system">
+					<hardware>
+						<plugin>modbus_ros2_control/DexterousHandHardware</plugin>
+						<param name="serial_port">/dev/ttyUSB0</param>
+						<param name="hand_type">${selected_hand_type}</param>
+						<param name="hand_side">right</param>
+						<param name="max_speed_ratio">1.0</param>
+					</hardware>
+					<xacro:linkerhand_o7_interfaces name="right_hand"/>
+				</ros2_control>
+			</xacro:if>
 		</xacro:if>
 	</xacro:if>
@@ -109,4 +176,9 @@
 				<xacro:linkerhand_o6_interfaces name="left_hand"/>
 				<xacro:linkerhand_o6_interfaces name="right_hand"/>
+			</xacro:if>
+			<xacro:if value="${selected_hand_type == 'linkerhand_o7'}">
+				<xacro:include filename="$(find linkerhand_description)/xacro/ros2_control/o7.xacro"/>
+				<xacro:linkerhand_o7_interfaces name="left_hand"/>
+				<xacro:linkerhand_o7_interfaces name="right_hand"/>
 			</xacro:if>
 			<xacro:if value="${selected_hand_type == 'linkerhand_o7'}">
