Commit message: Update xacro file to support marvin 485 communication

File: xacro/eefs.xacro (robot description, xacro)
@@ -96,20 +96,4 @@
             </joint>
         </xacro:if>
-        <!-- 灵巧手类型 -->
-        <xacro:if value="${hand_type == 'linkerhand_o7'}">
-            <xacro:include filename="$(find linkerhand_description)/xacro/o7.xacro"/>
-            <xacro:LinkerHandO7 name="left_hand" direction="1" use_flange="true" fixed_joints="false"/>
-            <joint name="left_hand_base_joint" type="fixed">
-                <origin xyz="0 0 0.0045" rpy="0 0 ${PI/2}"/>
-                <parent link="left_tcp"/>
-                <child link="left_hand_flange"/>
-            </joint>
-            <xacro:LinkerHandO7 name="right_hand" direction="-1" use_flange="true" fixed_joints="false"/>
-            <joint name="right_hand_base_joint" type="fixed">
-                <parent link="right_tcp"/>
-                <child link="right_hand_flange"/>
-                <origin xyz="0 0 0.0045" rpy="0 0 ${-PI/2}"/>
-            </joint>
-        </xacro:if>
     </xacro:macro>
 </robot>

File: xacro/robot.xacro (robot description, xacro)
@@ -1,67 +1,99 @@
 <?xml version="1.0"?>
-<robot name="FiveAges W2" xmlns:xacro="http://www.ros.org/wiki/xacro">
-	<xacro:arg name="collider" default="convex"/>
-	<xacro:arg name="chassis_joints_movable" default="false"/>
-	<!-- 从 type 参数解析出 hand_type 和 gripper_type -->
-	<xacro:arg name="type" default=""/>
-	<xacro:property name="type_arg" value="$(arg type)"/>
-	<!-- 手部控制模式：通过 type 后缀选择（_usb -> modbus, _marvin -> marvin 485） -->
-	<xacro:arg name="hand_control_mode" default="usb"/>
-	<xacro:property name="hand_control_mode_arg" value="$(arg hand_control_mode)"/>
-	<!-- 默认值 -->
-	<xacro:property name="selected_hand_type" value=""/>
-	<xacro:property name="selected_gripper_type" value=""/>
-	<!-- 从 type 解析 hand_type 和 gripper_type -->
-	<!-- 夹爪类型：selected_gripper_type 不为空即表示使用夹爪 -->
-	<xacro:if value="${type_arg == 'rg75'}">
-		<xacro:property name="selected_gripper_type" value="rg75"/>
-	</xacro:if>
-	<xacro:if value="${type_arg == 'ag2f90'}">
-		<xacro:property name="selected_gripper_type" value="ag2f90_d"/>
-	</xacro:if>
-	<xacro:if value="${type_arg == 'ag2f90_c'}">
-		<xacro:property name="selected_gripper_type" value="ag2f90_c"/>
-	</xacro:if>
-	<xacro:if value="${type_arg == 'ag2f90_d'}">
-		<xacro:property name="selected_gripper_type" value="ag2f90_d"/>
-	</xacro:if>
-	<!-- 灵巧手类型解析：支持格式 linkerhand_{o6,l6,o7}[_usb|_marvin] -->
-	<!-- O6 -->
-	<xacro:if value="${type_arg == 'linkerhand_o6' or type_arg == 'linkerhand_o6_usb' or type_arg == 'linkerhand_o6_marvin'}">
-		<xacro:property name="selected_hand_type" value="linkerhand_o6"/>
-		<xacro:if value="${type_arg == 'linkerhand_o6_usb'}"><xacro:property name="hand_control_mode_arg" value="usb"/></xacro:if>
-		<xacro:if value="${type_arg == 'linkerhand_o6_marvin'}"><xacro:property name="hand_control_mode_arg" value="marvin"/></xacro:if>
-	</xacro:if>
-	<!-- L6 -->
-	<xacro:if value="${type_arg == 'linkerhand_l6' or type_arg == 'linkerhand_l6_usb' or type_arg == 'linkerhand_l6_marvin'}">
-		<xacro:property name="selected_hand_type" value="linkerhand_l6"/>
-		<xacro:if value="${type_arg == 'linkerhand_l6_usb'}"><xacro:property name="hand_control_mode_arg" value="usb"/></xacro:if>
-		<xacro:if value="${type_arg == 'linkerhand_l6_marvin'}"><xacro:property name="hand_control_mode_arg" value="marvin"/></xacro:if>
-	</xacro:if>
-	<!-- O7 -->
-	<xacro:if value="${type_arg == 'linkerhand_o7' or type_arg == 'linkerhand_o7_usb' or type_arg == 'linkerhand_o7_marvin'}">
-		<xacro:property name="selected_hand_type" value="linkerhand_o7"/>
-		<xacro:if value="${type_arg == 'linkerhand_o7_usb'}"><xacro:property name="hand_control_mode_arg" value="usb"/></xacro:if>
-		<xacro:if value="${type_arg == 'linkerhand_o7_marvin'}"><xacro:property name="hand_control_mode_arg" value="marvin"/></xacro:if>
-	</xacro:if>
-	<xacro:include filename="$(find fiveages_w2_description)/xacro/components/linkhou_s2.xacro"/>
-	<xacro:linkhou_s2 joints_movable="$(arg chassis_joints_movable)"/>
-	<xacro:include filename="$(find fiveages_w2_description)/xacro/components/body.xacro"/>
-	<!-- Left Arm -->
-	<joint name="left_arm_base_joint" type="fixed">
-		<parent link="arm_base"/>
-		<child link="left_base_link"/>
-		<origin rpy="-${PI/2} 0 0" xyz="0.0 0.062 0"/>
-	</joint>
-	<!-- Right Arm -->
-	<joint name="right_arm_base_joint" type="fixed">
-		<parent link="arm_base"/>
-		<child link="right_base_link"/>
-		<origin rpy="${PI/2} 0 0" xyz="0 -0.062 0"/>
-	</joint>
-	<xacro:include filename="$(find m6_ccs_description)/xacro/arm.xacro"/>
-	<xacro:M6_CCS name="left" style="fiveages_w2"/>
-	<xacro:M6_CCS name="right" direction="-1" style="fiveages_w2"/>
-	<xacro:include filename="$(find fiveages_w2_description)/xacro/eefs.xacro"/>
-	<xacro:EndEffectors hand_type="${selected_hand_type}" gripper_type="${selected_gripper_type}"/>
+<robot xmlns:xacro="http://www.ros.org/wiki/xacro">
+    <xacro:macro name="EndEffectors" params="hand_type:='' gripper_type:=''">
+        <!-- Note:
+             - gripper_type 不为空时表示使用夹爪（保持原有逻辑）
+             - hand_type 只在需要区分灵巧手时使用（如 linkerhand_o6）
+             - 两者都为空时表示无末端执行器配置
+        -->
+        <!-- 无末端执行器配置 -->
+        <xacro:if value="${hand_type == '' and gripper_type == ''}">
+            <link name="left_eef"/>
+            <link name="right_eef"/>
+            <joint name="left_eef_joint" type="fixed">
+                <parent link="left_tcp"/>
+                <child link="left_eef"/>
+            </joint>
+            <joint name="right_eef_joint" type="fixed">
+                <parent link="right_tcp"/>
+                <child link="right_eef"/>
+            </joint>
+        </xacro:if>
+        <!-- 夹爪类型：gripper_type 不为空即表示使用夹爪 -->
+        <xacro:if value="${gripper_type == 'ag2f90_c' or gripper_type == 'ag2f90_d'}">
+            <xacro:include filename="$(find changingtek_description)/xacro/AG2F90-C.xacro"/>
+            <xacro:AG2F90-C name="left" use_flange="true"/>
+            <joint name="left_gripper_fix" type="fixed">
+                <parent link="left_tcp"/>
+                <child link="left_flange"/>
+                <origin xyz="0 0 0.0045"/>
+            </joint>
+            <xacro:AG2F90-C name="right" use_flange="true"/>
+            <joint name="right_gripper_fix" type="fixed">
+                <parent link="right_tcp"/>
+                <child link="right_flange"/>
+                <origin xyz="0 0 0.0045"/>
+            </joint>
+        </xacro:if>
+        <xacro:if value="${gripper_type == 'rg75'}">
+            <xacro:include filename="$(find jodell_description)/xacro/RG75-300.xacro"/>
+            <xacro:RG75-300 name="left" use_flange="true"/>
+            <xacro:RG75-300 name="right" use_flange="true"/>
+            <joint name="left_gripper_base_joint" type="fixed">
+                <parent link="left_tcp"/>
+                <child link="left_flange"/>
+            </joint>
+            <joint name="right_gripper_base_joint" type="fixed">
+                <parent link="right_tcp"/>
+                <child link="right_flange"/>
+            </joint>
+        </xacro:if>
+        <!-- 灵巧手类型 -->
+        <xacro:if value="${hand_type == 'linkerhand_o6'}">
+            <xacro:include filename="$(find linkerhand_description)/xacro/o6.xacro"/>
+            <xacro:LinkerHandO6 name="left_hand" direction="1" use_flange="true" fixed_joints="false"/>
+            <joint name="left_hand_base_joint" type="fixed">
+                <origin xyz="0 0 0.0045" rpy="0 0 ${PI}"/>
+                <parent link="left_tcp"/>
+                <child link="left_hand_flange"/>
+            </joint>
+            <xacro:LinkerHandO6 name="right_hand" direction="-1" use_flange="true" fixed_joints="false"/>
+            <joint name="right_hand_base_joint" type="fixed">
+                <parent link="right_tcp"/>
+                <child link="right_hand_flange"/>
+                <origin xyz="0 0 0.0045"/>
+            </joint>
+        </xacro:if>
+        <xacro:if value="${hand_type == 'linkerhand_o7'}">
+            <xacro:include filename="$(find linkerhand_description)/xacro/o7.xacro"/>
+            <xacro:LinkerHandO7 name="left_hand" direction="1" use_flange="true" fixed_joints="false"/>
+            <joint name="left_hand_base_joint" type="fixed">
+                <origin rpy="0 0 ${PI/2}"/>
+                <parent link="left_tcp"/>
+                <child link="left_hand_flange"/>
+            </joint>
+            <xacro:LinkerHandO7 name="right_hand" direction="-1" use_flange="true" fixed_joints="false"/>
+            <joint name="right_hand_base_joint" type="fixed">
+                <origin rpy="0 0 ${-PI/2}"/>
+                <parent link="right_tcp"/>
+                <child link="right_hand_flange"/>
+            </joint>
+        </xacro:if>
+        <!-- 灵巧手类型 -->
+        <xacro:if value="${hand_type == 'linkerhand_l6'}">
+            <xacro:include filename="$(find linkerhand_description)/xacro/l6.xacro"/>
+            <xacro:LinkerHandL6 name="left_hand" direction="1" use_flange="true" fixed_joints="false"/>
+            <joint name="left_hand_base_joint" type="fixed">
+                <origin xyz="0 0 0.0045" rpy="0 0 ${PI}"/>
+                <parent link="left_tcp"/>
+                <child link="left_hand_flange"/>
+            </joint>
+            <xacro:LinkerHandL6 name="right_hand" direction="-1" use_flange="true" fixed_joints="false"/>
+            <joint name="right_hand_base_joint" type="fixed">
+                <parent link="right_tcp"/>
+                <child link="right_hand_flange"/>
+                <origin xyz="0 0 0.0045"/>
+            </joint>
+        </xacro:if>
+    </xacro:macro>
 </robot>

File: xacro/ros2_control/robot.xacro (robot description, xacro)
@@ -7,17 +7,4 @@
 	<xacro:include filename="$(find m6_ccs_description)/xacro/ros2_control/interfaces.xacro"/>
 	<xacro:include filename="$(find fiveages_w2_description)/xacro/ros2_control/body.xacro"/>
-	<!-- 宏：创建单个 modbus 灵巧手系统（USB 模式） -->
-	<xacro:macro name="create_modbus_hand_single" params="hand_type system_suffix side serial_port">
-		<ros2_control name="linkerhand_${system_suffix}_${side}_system" type="system">
-			<hardware>
-				<plugin>modbus_ros2_control/DexterousHandHardware</plugin>
-				<param name="serial_port">${serial_port}</param>
-				<param name="hand_type">${hand_type}</param>
-				<param name="hand_side">${side}</param>
-				<param name="max_speed_ratio">1.0</param>
-			</hardware>
-			<xacro:insert_block/>
-		</ros2_control>
-	</xacro:macro>
 	<xacro:if value="${'$(arg ros2_control_hardware_type)' == 'real'}">
 		<!-- 确定传递给 marvin_ros2_control 的 gripper_type 参数 -->
@@ -98,25 +85,53 @@
 			<xacro:body_interfaces/>
 		</ros2_control>
-		<!-- 灵巧手接口：USB 模式（modbus_ros2_control） -->
+		<!-- 灵巧手接口：USB 模式（modbus_ros2_control），直接内联 ros2_control 配置 -->
 		<xacro:if value="${selected_hand_type != '' and hand_control_mode_arg == 'usb'}">
 			<!-- O6/L6: 6-DOF 手 -->
 			<xacro:if value="${selected_hand_type == 'linkerhand_o6' or selected_hand_type == 'linkerhand_l6'}">
 				<xacro:include filename="$(find linkerhand_description)/xacro/ros2_control/o6.xacro"/>
-				<xacro:create_modbus_hand_single hand_type="${selected_hand_type}" system_suffix="6" side="left" serial_port="/dev/ttyUSB1">
+				<ros2_control name="linkerhand_6_left_system" type="system">
+					<hardware>
+						<plugin>modbus_ros2_control/DexterousHandHardware</plugin>
+						<param name="serial_port">/dev/ttyUSB1</param>
+						<param name="hand_type">${selected_hand_type}</param>
+						<param name="hand_side">left</param>
+						<param name="max_speed_ratio">1.0</param>
+					</hardware>
 					<xacro:linkerhand_o6_interfaces name="left_hand"/>
-				</xacro:create_modbus_hand_single>
-				<xacro:create_modbus_hand_single hand_type="${selected_hand_type}" system_suffix="6" side="right" serial_port="/dev/ttyUSB0">
+				</ros2_control>
+				<ros2_control name="linkerhand_6_right_system" type="system">
+					<hardware>
+						<plugin>modbus_ros2_control/DexterousHandHardware</plugin>
+						<param name="serial_port">/dev/ttyUSB0</param>
+						<param name="hand_type">${selected_hand_type}</param>
+						<param name="hand_side">right</param>
+						<param name="max_speed_ratio">1.0</param>
+					</hardware>
 					<xacro:linkerhand_o6_interfaces name="right_hand"/>
-				</xacro:create_modbus_hand_single>
+				</ros2_control>
 			</xacro:if>
 			<!-- O7: 7-DOF 手 -->
 			<xacro:if value="${selected_hand_type == 'linkerhand_o7'}">
 				<xacro:include filename="$(find linkerhand_description)/xacro/ros2_control/o7.xacro"/>
-				<xacro:create_modbus_hand_single hand_type="${selected_hand_type}" system_suffix="7" side="left" serial_port="/dev/ttyUSB1">
+				<ros2_control name="linkerhand_7_left_system" type="system">
+					<hardware>
+						<plugin>modbus_ros2_control/DexterousHandHardware</plugin>
+						<param name="serial_port">/dev/ttyUSB1</param>
+						<param name="hand_type">${selected_hand_type}</param>
+						<param name="hand_side">left</param>
+						<param name="max_speed_ratio">1.0</param>
+					</hardware>
 					<xacro:linkerhand_o7_interfaces name="left_hand"/>
-				</xacro:create_modbus_hand_single>
-				<xacro:create_modbus_hand_single hand_type="${selected_hand_type}" system_suffix="7" side="right" serial_port="/dev/ttyUSB0">
+				</ros2_control>
+				<ros2_control name="linkerhand_7_right_system" type="system">
+					<hardware>
+						<plugin>modbus_ros2_control/DexterousHandHardware</plugin>
+						<param name="serial_port">/dev/ttyUSB0</param>
+						<param name="hand_type">${selected_hand_type}</param>
+						<param name="hand_side">right</param>
+						<param name="max_speed_ratio">1.0</param>
+					</hardware>
 					<xacro:linkerhand_o7_interfaces name="right_hand"/>
-				</xacro:create_modbus_hand_single>
+				</ros2_control>
 			</xacro:if>
 		</xacro:if>
@@ -164,9 +179,4 @@
 				<xacro:linkerhand_o7_interfaces name="right_hand"/>
 			</xacro:if>
-			<xacro:if value="${selected_hand_type == 'linkerhand_o7'}">
-				<xacro:include filename="$(find linkerhand_description)/xacro/ros2_control/o7.xacro"/>
-				<xacro:linkerhand_o7_interfaces name="left_hand"/>
-				<xacro:linkerhand_o7_interfaces name="right_hand"/>
-			</xacro:if>
 		</ros2_control>
 	</xacro:unless>
