Commit message: fix xacro problem

File: xacro/eefs.xacro (robot description, xacro)
@@ -38,13 +38,19 @@
         <xacro:if value="${gripper_type == 'rg75'}">
             <xacro:include filename="$(find jodell_description)/xacro/RG75-300.xacro"/>
-            <xacro:RG75-300 name="left" use_flange="true"/>
-            <xacro:RG75-300 name="right" use_flange="true"/>
+            <xacro:RG75-300 name="left" use_flange="true" pad="${selected_gripper_pad}"/>
+            <xacro:RG75-300 name="right" use_flange="true" pad="${selected_gripper_pad}"/>
             <joint name="left_gripper_base_joint" type="fixed">
                 <parent link="left_tcp"/>
                 <child link="left_flange"/>
+                <xacro:if value="${selected_gripper_pad == 'heavy_carry'}">
+                    <origin rpy="0 0 ${PI/2}"/>
+                </xacro:if>
             </joint>
             <joint name="right_gripper_base_joint" type="fixed">
                 <parent link="right_tcp"/>
                 <child link="right_flange"/>
+                <xacro:if value="${selected_gripper_pad == 'heavy_carry'}">
+                    <origin rpy="0 0 ${PI/2}"/>
+                </xacro:if>
             </joint>
         </xacro:if>

File: xacro/robot.xacro (robot description, xacro)
@@ -1,99 +1,60 @@
 <?xml version="1.0"?>
-<robot xmlns:xacro="http://www.ros.org/wiki/xacro">
-    <xacro:macro name="EndEffectors" params="hand_type:='' gripper_type:=''">
-        <!-- Note:
-             - gripper_type 不为空时表示使用夹爪（保持原有逻辑）
-             - hand_type 只在需要区分灵巧手时使用（如 linkerhand_o6）
-             - 两者都为空时表示无末端执行器配置
-        -->
-        <!-- 无末端执行器配置 -->
-        <xacro:if value="${hand_type == '' and gripper_type == ''}">
-            <link name="left_eef"/>
-            <link name="right_eef"/>
-            <joint name="left_eef_joint" type="fixed">
-                <parent link="left_tcp"/>
-                <child link="left_eef"/>
-            </joint>
-            <joint name="right_eef_joint" type="fixed">
-                <parent link="right_tcp"/>
-                <child link="right_eef"/>
-            </joint>
-        </xacro:if>
-        <!-- 夹爪类型：gripper_type 不为空即表示使用夹爪 -->
-        <xacro:if value="${gripper_type == 'ag2f90_c' or gripper_type == 'ag2f90_d'}">
-            <xacro:include filename="$(find changingtek_description)/xacro/AG2F90-C.xacro"/>
-            <xacro:AG2F90-C name="left" use_flange="true"/>
-            <joint name="left_gripper_fix" type="fixed">
-                <parent link="left_tcp"/>
-                <child link="left_flange"/>
-                <origin xyz="0 0 0.0045"/>
-            </joint>
-            <xacro:AG2F90-C name="right" use_flange="true"/>
-            <joint name="right_gripper_fix" type="fixed">
-                <parent link="right_tcp"/>
-                <child link="right_flange"/>
-                <origin xyz="0 0 0.0045"/>
-            </joint>
-        </xacro:if>
-        <xacro:if value="${gripper_type == 'rg75'}">
-            <xacro:include filename="$(find jodell_description)/xacro/RG75-300.xacro"/>
-            <xacro:RG75-300 name="left" use_flange="true"/>
-            <xacro:RG75-300 name="right" use_flange="true"/>
-            <joint name="left_gripper_base_joint" type="fixed">
-                <parent link="left_tcp"/>
-                <child link="left_flange"/>
-            </joint>
-            <joint name="right_gripper_base_joint" type="fixed">
-                <parent link="right_tcp"/>
-                <child link="right_flange"/>
-            </joint>
-        </xacro:if>
-        <!-- 灵巧手类型 -->
-        <xacro:if value="${hand_type == 'linkerhand_o6'}">
-            <xacro:include filename="$(find linkerhand_description)/xacro/o6.xacro"/>
-            <xacro:LinkerHandO6 name="left_hand" direction="1" use_flange="true" fixed_joints="false"/>
-            <joint name="left_hand_base_joint" type="fixed">
-                <origin xyz="0 0 0.0045" rpy="0 0 ${PI}"/>
-                <parent link="left_tcp"/>
-                <child link="left_hand_flange"/>
-            </joint>
-            <xacro:LinkerHandO6 name="right_hand" direction="-1" use_flange="true" fixed_joints="false"/>
-            <joint name="right_hand_base_joint" type="fixed">
-                <parent link="right_tcp"/>
-                <child link="right_hand_flange"/>
-                <origin xyz="0 0 0.0045"/>
-            </joint>
-        </xacro:if>
-        <xacro:if value="${hand_type == 'linkerhand_o7'}">
-            <xacro:include filename="$(find linkerhand_description)/xacro/o7.xacro"/>
-            <xacro:LinkerHandO7 name="left_hand" direction="1" use_flange="true" fixed_joints="false"/>
-            <joint name="left_hand_base_joint" type="fixed">
-                <origin rpy="0 0 ${PI/2}"/>
-                <parent link="left_tcp"/>
-                <child link="left_hand_flange"/>
-            </joint>
-            <xacro:LinkerHandO7 name="right_hand" direction="-1" use_flange="true" fixed_joints="false"/>
-            <joint name="right_hand_base_joint" type="fixed">
-                <origin rpy="0 0 ${-PI/2}"/>
-                <parent link="right_tcp"/>
-                <child link="right_hand_flange"/>
-            </joint>
-        </xacro:if>
-        <!-- 灵巧手类型 -->
-        <xacro:if value="${hand_type == 'linkerhand_l6'}">
-            <xacro:include filename="$(find linkerhand_description)/xacro/l6.xacro"/>
-            <xacro:LinkerHandL6 name="left_hand" direction="1" use_flange="true" fixed_joints="false"/>
-            <joint name="left_hand_base_joint" type="fixed">
-                <origin xyz="0 0 0.0045" rpy="0 0 ${PI}"/>
-                <parent link="left_tcp"/>
-                <child link="left_hand_flange"/>
-            </joint>
-            <xacro:LinkerHandL6 name="right_hand" direction="-1" use_flange="true" fixed_joints="false"/>
-            <joint name="right_hand_base_joint" type="fixed">
-                <parent link="right_tcp"/>
-                <child link="right_hand_flange"/>
-                <origin xyz="0 0 0.0045"/>
-            </joint>
-        </xacro:if>
-    </xacro:macro>
+<robot name="FiveAges W2" xmlns:xacro="http://www.ros.org/wiki/xacro">
+    <xacro:arg name="collider" default="convex"/>
+    <xacro:arg name="chassis_joints_movable" default="false"/>
+    <!-- 从 type 参数解析出 hand_type 和 gripper_type -->
+    <xacro:arg name="type" default=""/>
+    <xacro:property name="type_arg" value="$(arg type)"/>
+    <!-- 默认值 -->
+    <xacro:property name="selected_hand_type" value=""/>
+    <xacro:property name="selected_gripper_type" value=""/>
+    <xacro:property name="selected_gripper_pad" value="default"/>
+    <!-- 从 type 解析 hand_type 和 gripper_type -->
+    <!-- 夹爪类型：selected_gripper_type 不为空即表示使用夹爪 -->
+    <xacro:if value="${type_arg == 'rg75'}">
+        <xacro:property name="selected_gripper_type" value="rg75"/>
+    </xacro:if>
+    <xacro:if value="${type_arg == 'rg75_heavy'}">
+        <xacro:property name="selected_gripper_type" value="rg75"/>
+        <xacro:property name="selected_gripper_pad" value="heavy_carry"/>
+    </xacro:if>
+    <xacro:if value="${type_arg == 'ag2f90'}">
+        <xacro:property name="selected_gripper_type" value="ag2f90_d"/>
+    </xacro:if>
+    <xacro:if value="${type_arg == 'ag2f90_c'}">
+        <xacro:property name="selected_gripper_type" value="ag2f90_c"/>
+    </xacro:if>
+    <xacro:if value="${type_arg == 'ag2f90_d'}">
+        <xacro:property name="selected_gripper_type" value="ag2f90_d"/>
+    </xacro:if>
+    <!-- 灵巧手类型 -->
+    <xacro:if value="${type_arg == 'linkerhand_o6'}">
+        <xacro:property name="selected_hand_type" value="linkerhand_o6"/>
+    </xacro:if>
+    <xacro:if value="${type_arg == 'linkerhand_l6'}">
+        <xacro:property name="selected_hand_type" value="linkerhand_l6"/>
+    </xacro:if>
+    <xacro:if value="${type_arg == 'linkerhand_o7'}">
+        <xacro:property name="selected_hand_type" value="linkerhand_o7"/>
+    </xacro:if>
+    <xacro:include filename="$(find fiveages_w2_description)/xacro/components/linkhou_s2.xacro"/>
+    <xacro:linkhou_s2 joints_movable="$(arg chassis_joints_movable)"/>
+    <xacro:include filename="$(find fiveages_w2_description)/xacro/components/body.xacro"/>
+    <!-- Left Arm -->
+    <joint name="left_arm_base_joint" type="fixed">
+        <parent link="arm_base"/>
+        <child link="left_base_link"/>
+        <origin rpy="-${PI/2} 0 0" xyz="0.0 0.062 0"/>
+    </joint>
+    <!-- Right Arm -->
+    <joint name="right_arm_base_joint" type="fixed">
+        <parent link="arm_base"/>
+        <child link="right_base_link"/>
+        <origin rpy="${PI/2} 0 0" xyz="0 -0.062 0"/>
+    </joint>
+    <xacro:include filename="$(find m6_ccs_description)/xacro/arm.xacro"/>
+    <xacro:M6_CCS name="left" style="fiveages_w2"/>
+    <xacro:M6_CCS name="right" direction="-1" style="fiveages_w2"/>
+    <xacro:include filename="$(find fiveages_w2_description)/xacro/eefs.xacro"/>
+    <xacro:EndEffectors hand_type="${selected_hand_type}" gripper_type="${selected_gripper_type}"/>
 </robot>

File: xacro/ros2_control/robot.xacro (robot description, xacro)
@@ -2,10 +2,10 @@
 <robot name="fiveages_w2" xmlns:xacro="http://www.ros.org/wiki/xacro">
 	<xacro:arg name="ros2_control_hardware_type" default="mock_components"/>
-	<xacro:arg name="device_ip" default="192.168.1.190"/>
-	<xacro:property name="device_ip_arg" value="$(arg device_ip)"/>
+	<xacro:property name="is_real_hardware" value="${'$(arg ros2_control_hardware_type)' == 'real' or '$(arg ros2_control_hardware_type)' == 'real_usb'}"/>
+	<xacro:property name="ee_drive_type" value="${'usb' if '$(arg ros2_control_hardware_type)' == 'real_usb' else ('marvin' if '$(arg ros2_control_hardware_type)' == 'real' else '')}"/>
 	<xacro:include filename="$(find fiveages_w2_description)/xacro/robot.xacro"/>
 	<xacro:include filename="$(find m6_ccs_description)/xacro/ros2_control/interfaces.xacro"/>
 	<xacro:include filename="$(find fiveages_w2_description)/xacro/ros2_control/body.xacro"/>
-	<xacro:if value="${'$(arg ros2_control_hardware_type)' == 'real' or '$(arg ros2_control_hardware_type)' == 'real_usb'}">
+	<xacro:if value="${is_real_hardware}">
 		<!-- 确定传递给 marvin_ros2_control 的 gripper_type 参数 -->
 		<!--
@@ -26,5 +26,5 @@
 				-->
 				<!-- 485/marvin(real) + hand: pass hand type; otherwise pass gripper type (or empty). -->
-				<param name="gripper_type">${selected_hand_type if (selected_hand_type != '' and '$(arg ros2_control_hardware_type)' == 'real') else selected_gripper_type}</param>
+				<param name="gripper_type">${selected_hand_type if ee_drive_type == 'marvin' else selected_gripper_type}</param>
 				<param name="max_joint_speed">50</param>
 				<param name="max_joint_acceleration">30</param>
@@ -32,5 +32,5 @@
 				<param name="left_dyn_param">0.4,0,0,50.65,0,0,0,0,0,0</param>
 				<param name="right_dyn_param">0.4,0,0,50.85,0,0,0,0,0,0</param>
-				<param name="device_ip">${device_ip_arg}</param>
+				<param name="device_ip">192.168.1.190</param>
 			</hardware>
 			<xacro:m6_interfaces name="left"/>
@@ -52,6 +52,6 @@
 			</xacro:if>
 			<!-- 灵巧手接口：485/marvin（通过 M6_CCS_System） -->
-			<xacro:if value="${selected_hand_type != '' and '$(arg ros2_control_hardware_type)' == 'real'}">
-				<xacro:if value="${selected_hand_type == 'linkerhand_o6' or selected_hand_type == 'linkerhand_l6'}">
+			<xacro:if value="${ee_drive_type == 'marvin'}">
+				<xacro:if value="${selected_hand_type in ['linkerhand_o6', 'linkerhand_l6']}">
 					<xacro:include filename="$(find linkerhand_description)/xacro/ros2_control/o6.xacro"/>
 					<xacro:linkerhand_o6_interfaces name="left_hand"/>
@@ -78,9 +78,14 @@
 		</ros2_control>
 		<!-- 灵巧手接口：USB 模式（hardware=real_usb，modbus_ros2_control），直接内联 ros2_control 配置 -->
-		<xacro:if value="${selected_hand_type != '' and '$(arg ros2_control_hardware_type)' == 'real_usb'}">
-			<!-- O6/L6: 6-DOF 手 -->
-			<xacro:if value="${selected_hand_type == 'linkerhand_o6' or selected_hand_type == 'linkerhand_l6'}">
-				<xacro:include filename="$(find linkerhand_description)/xacro/ros2_control/o6.xacro"/>
-				<ros2_control name="linkerhand_6_left_system" type="system">
+		<xacro:if value="${ee_drive_type == 'usb'}">
+			<xacro:if value="${selected_hand_type in ('linkerhand_o6', 'linkerhand_l6', 'linkerhand_o7')}">
+				<xacro:property name="usb_hand_series" value="${'7' if selected_hand_type == 'linkerhand_o7' else '6'}"/>
+				<xacro:if value="${usb_hand_series == '6'}">
+					<xacro:include filename="$(find linkerhand_description)/xacro/ros2_control/o6.xacro"/>
+				</xacro:if>
+				<xacro:if value="${usb_hand_series == '7'}">
+					<xacro:include filename="$(find linkerhand_description)/xacro/ros2_control/o7.xacro"/>
+				</xacro:if>
+				<ros2_control name="linkerhand_${usb_hand_series}_left_system" type="system">
 					<hardware>
 						<plugin>modbus_ros2_control/DexterousHandHardware</plugin>
@@ -90,7 +95,12 @@
 						<param name="max_speed_ratio">1.0</param>
 					</hardware>
-					<xacro:linkerhand_o6_interfaces name="left_hand"/>
+					<xacro:if value="${usb_hand_series == '6'}">
+						<xacro:linkerhand_o6_interfaces name="left_hand"/>
+					</xacro:if>
+					<xacro:if value="${usb_hand_series == '7'}">
+						<xacro:linkerhand_o7_interfaces name="left_hand"/>
+					</xacro:if>
 				</ros2_control>
-				<ros2_control name="linkerhand_6_right_system" type="system">
+				<ros2_control name="linkerhand_${usb_hand_series}_right_system" type="system">
 					<hardware>
 						<plugin>modbus_ros2_control/DexterousHandHardware</plugin>
@@ -100,34 +110,15 @@
 						<param name="max_speed_ratio">1.0</param>
 					</hardware>
-					<xacro:linkerhand_o6_interfaces name="right_hand"/>
-				</ros2_control>
-			</xacro:if>
-			<!-- O7: 7-DOF 手 -->
-			<xacro:if value="${selected_hand_type == 'linkerhand_o7'}">
-				<xacro:include filename="$(find linkerhand_description)/xacro/ros2_control/o7.xacro"/>
-				<ros2_control name="linkerhand_7_left_system" type="system">
-					<hardware>
-						<plugin>modbus_ros2_control/DexterousHandHardware</plugin>
-						<param name="serial_port">/dev/ttyUSB1</param>
-						<param name="hand_type">${selected_hand_type}</param>
-						<param name="hand_side">left</param>
-						<param name="max_speed_ratio">1.0</param>
-					</hardware>
-					<xacro:linkerhand_o7_interfaces name="left_hand"/>
-				</ros2_control>
-				<ros2_control name="linkerhand_7_right_system" type="system">
-					<hardware>
-						<plugin>modbus_ros2_control/DexterousHandHardware</plugin>
-						<param name="serial_port">/dev/ttyUSB0</param>
-						<param name="hand_type">${selected_hand_type}</param>
-						<param name="hand_side">right</param>
-						<param name="max_speed_ratio">1.0</param>
-					</hardware>
-					<xacro:linkerhand_o7_interfaces name="right_hand"/>
+					<xacro:if value="${usb_hand_series == '6'}">
+						<xacro:linkerhand_o6_interfaces name="right_hand"/>
+					</xacro:if>
+					<xacro:if value="${usb_hand_series == '7'}">
+						<xacro:linkerhand_o7_interfaces name="right_hand"/>
+					</xacro:if>
 				</ros2_control>
 			</xacro:if>
 		</xacro:if>
 	</xacro:if>
-	<xacro:unless value="${'$(arg ros2_control_hardware_type)' == 'real' or '$(arg ros2_control_hardware_type)' == 'real_usb'}">
+	<xacro:unless value="${is_real_hardware}">
 		<ros2_control name="fiveages_w2_system" type="system">
 			<hardware>
@@ -155,5 +146,5 @@
 				<xacro:rg75_interfaces name="right"/>
 			</xacro:if>
-			<xacro:if value="${selected_gripper_type == 'ag2f90_c' or selected_gripper_type == 'ag2f90_d'}">
+			<xacro:if value="${selected_gripper_type in ('ag2f90_c', 'ag2f90_d')}">
 				<xacro:include filename="$(find changingtek_description)/xacro/ros2_control/AG2F90-C.xacro"/>
 				<xacro:ag2f90c_interfaces name="left"/>
@@ -161,5 +152,5 @@
 			</xacro:if>
 			<!-- 灵巧手接口 -->
-			<xacro:if value="${selected_hand_type == 'linkerhand_o6' or selected_hand_type == 'linkerhand_l6'}">
+			<xacro:if value="${selected_hand_type in ['linkerhand_o6', 'linkerhand_l6']}">
 				<xacro:include filename="$(find linkerhand_description)/xacro/ros2_control/o6.xacro"/>
 				<xacro:linkerhand_o6_interfaces name="left_hand"/>

Commit message: 增加90c-soft

File: xacro/eefs.xacro (robot description, xacro)
@@ -24,5 +24,5 @@
         <xacro:if value="${gripper_type == 'ag2f90_c' or gripper_type == 'ag2f90_d'}">
             <xacro:include filename="$(find changingtek_description)/xacro/AG2F90-C.xacro"/>
-            <xacro:AG2F90-C name="left" use_flange="true"/>
+            <xacro:AG2F90-C name="left" use_flange="true" pad="${selected_gripper_pad}"/>
             <joint name="left_gripper_fix" type="fixed">
                 <parent link="left_tcp"/>
@@ -30,5 +30,5 @@
                 <origin xyz="0 0 0.0045"/>
             </joint>
-            <xacro:AG2F90-C name="right" use_flange="true"/>
+            <xacro:AG2F90-C name="right" use_flange="true" pad="${selected_gripper_pad}"/>
             <joint name="right_gripper_fix" type="fixed">
                 <parent link="right_tcp"/>

File: xacro/robot.xacro (robot description, xacro)
@@ -25,4 +25,8 @@
     <xacro:if value="${type_arg == 'ag2f90_c'}">
         <xacro:property name="selected_gripper_type" value="ag2f90_c"/>
+    </xacro:if>
+    <xacro:if value="${type_arg == 'ag2f90_c_soft'}">
+        <xacro:property name="selected_gripper_type" value="ag2f90_c"/>
+        <xacro:property name="selected_gripper_pad" value="soft"/>
     </xacro:if>
     <xacro:if value="${type_arg == 'ag2f90_d'}">

File: xacro/ros2_control/robot.xacro (robot description, xacro)
@@ -151,4 +151,5 @@
 				<xacro:rg75_interfaces name="right"/>
 			</xacro:if>
+			<!-- ag2f90_c_soft 在 robot.xacro 中解析为 selected_gripper_type=ag2f90_c + pad=soft -->
 			<xacro:if value="${selected_gripper_type in ('ag2f90_c', 'ag2f90_d')}">
 				<xacro:include filename="$(find changingtek_description)/xacro/ros2_control/AG2F90-C.xacro"/>
