Commit message: add demo launch for basic joint controller

File: xacro/component.xacro (robot description, xacro)
@@ -9,3 +9,7 @@
 		<xacro:include filename="$(find fiveages_w2_description)/xacro/chassis/linkhou_s2.xacro"/>
 	</xacro:if>
+	<xacro:if value="${'$(arg type)' == 'body'}">
+		<link name="base_link"/>
+		<xacro:include filename="$(find fiveages_w2_description)/xacro/body.xacro"/>
+	</xacro:if>
 </robot>

File: xacro/robot.xacro (robot description, xacro)
@@ -3,224 +3,5 @@
 	<xacro:arg name="collider" default="convex"/>
 	<xacro:include filename="$(find fiveages_w2_description)/xacro/chassis/linkhou_s2.xacro"/>
-	<link name="body_base">
-		<inertial>
-			<origin xyz="-0.000200488559999101 -0.000273639516978452 -0.146062494992026"/>
-			<mass value="8.23744177260185" />
-			<inertia
-					ixx="0.0427044289140212"
-					ixy="0.000110484904723097"
-					ixz="5.20117375313561E-06"
-					iyy="0.0344639116909607"
-					iyz="-1.07902056768718E-05"
-					izz="0.0490685771548297" />
-		</inertial>
-		<visual>
-			<geometry>
-				<mesh filename="file://$(find fiveages_w2_description)/meshes/body/base.obj" />
-			</geometry>
-		</visual>
-		<collision>
-			<geometry>
-				<mesh filename="file://$(find fiveages_w2_description)/meshes/body/base.obj" />
-			</geometry>
-		</collision>
-	</link>
-	<joint name="body_fixed_joint" type="fixed">
-		<origin xyz="0.10525 0 0.2295"/>
-		<parent link="base_link" />
-		<child link="body_base" />
-	</joint>
-	<link name="body_link1">
-		<inertial>
-			<origin xyz="-5.26269080900477E-05 -0.000546927086993554 0.159848926806017"/>
-			<mass value="5.6518910145446" />
-			<inertia
-					ixx="0.129446325951384"
-					ixy="8.587994128406E-06"
-					ixz="9.34570905413505E-06"
-					iyy="0.118974430850637"
-					iyz="0.000463913896532557"
-					izz="0.0161870223281112" />
-		</inertial>
-		<visual>
-			<geometry>
-				<mesh filename="file://$(find fiveages_w2_description)/meshes/body/link1.obj" />
-			</geometry>
-		</visual>
-		<collision>
-			<geometry>
-				<mesh filename="file://$(find fiveages_w2_description)/meshes/body/link1.obj" />
-			</geometry>
-		</collision>
-	</link>
-	<joint name="body_joint1" type="revolute">
-		<parent link="body_base" />
-		<child link="body_link1" />
-		<axis xyz="0 1 0" />
-		<limit lower="-3.14" upper="3.14" effort="100" velocity="1" />
-	</joint>
-	<link name="body_link2">
-		<inertial>
-			<origin xyz="-5.06261699229071E-14 -1.0902390101819E-13 0.172448903272911"/>
-			<mass value="7.6108743790626" />
-			<inertia
-					ixx="0.168898657844891"
-					ixy="-7.65126788334289E-08"
-					ixz="-2.99913165388078E-14"
-					iyy="0.189588222903554"
-					iyz="-2.80537312130624E-15"
-					izz="0.0218547815193579" />
-		</inertial>
-		<visual>
-			<geometry>
-				<mesh filename="file://$(find fiveages_w2_description)/meshes/body/link2.obj" />
-			</geometry>
-		</visual>
-		<collision>
-			<geometry>
-				<mesh filename="file://$(find fiveages_w2_description)/meshes/body/link2.obj" />
-			</geometry>
-		</collision>
-	</link>
-	<joint name="body_joint2" type="revolute">
-		<origin xyz="0 0 0.323"/>
-		<parent link="body_link1" />
-		<child link="body_link2" />
-		<axis xyz="0 -1 0" />
-		<limit lower="-3.14" upper="3.14" effort="100" velocity="1" />
-	</joint>
-	<link name="body_link3">
-		<inertial>
-			<origin xyz="2.24765231915391E-06 -0.017843126813746 0.0199837851518558"/>
-			<mass value="13.7293315804368" />
-			<inertia
-					ixx="0.0380691419113999"
-					ixy="-6.90768437813021E-08"
-					ixz="3.88596630213136E-06"
-					iyy="0.0443960808652778"
-					iyz="8.97911264129812E-06"
-					izz="0.0332593124725221" />
-		</inertial>
-		<visual>
-			<geometry>
-				<mesh filename="file://$(find fiveages_w2_description)/meshes/body/link3.obj" />
-			</geometry>
-		</visual>
-		<collision>
-			<geometry>
-				<mesh filename="file://$(find fiveages_w2_description)/meshes/body/link3.obj" />
-			</geometry>
-		</collision>
-	</link>
-	<joint name="body_joint3" type="revolute">
-		<origin xyz="0 0.0019 0.35294"/>
-		<parent link="body_link2" />
-		<child link="body_link3" />
-		<axis xyz="0 -1 0" />
-		<limit lower="-3.14" upper="3.14" effort="100" velocity="1" />
-	</joint>
-	<link name="body_link4">
-		<inertial>
-			<origin xyz="-0.0249769763515 0.00261378092766984 0.273685327435851"/>
-			<mass value="23.7446873792875" />
-			<inertia
-					ixx="0.32004495936722"
-					ixy="8.27745275816937E-05"
-					ixz="0.0072338104417254"
-					iyy="0.228581680748554"
-					iyz="8.86157129443541E-05"
-					izz="0.136693312472866" />
-		</inertial>
-		<visual>
-			<geometry>
-				<mesh filename="file://$(find fiveages_w2_description)/meshes/body/link4.obj" />
-			</geometry>
-		</visual>
-		<collision>
-			<geometry>
-				<mesh filename="file://$(find fiveages_w2_description)/meshes/body/link4.obj" />
-			</geometry>
-		</collision>
-	</link>
-	<joint name="body_joint4" type="revolute">
-		<origin xyz="0 -0.0019 0.1443"/>
-		<parent link="body_link3" />
-		<child link="body_link4" />
-		<axis xyz="0 0 -1" />
-		<limit lower="-3.14" upper="3.14" effort="100" velocity="1" />
-	</joint>
-	<link name="head_yaw">
-		<inertial>
-			<origin xyz="0.0110684120335558 0.0270955929655894 -0.0849037421704728"/>
-			<mass value="1.76592019732553" />
-			<inertia
-					ixx="0.00540494211688139"
-					ixy="5.45899583655646E-06"
-					ixz="0.000512508898720623"
-					iyy="0.0045794535946287"
-					iyz="5.71011553188605E-05"
-					izz="0.00441063426341843" />
-		</inertial>
-		<visual>
-			<geometry>
-				<mesh filename="file://$(find fiveages_w2_description)/meshes/body/head_yaw.obj" />
-			</geometry>
-		</visual>
-		<collision>
-			<geometry>
-				<mesh filename="file://$(find fiveages_w2_description)/meshes/body/head_yaw.obj" />
-			</geometry>
-		</collision>
-	</link>
-	<joint name="head_joint1" type="revolute">
-		<origin xyz="-0.046314 -0.0272 0.63334"/>
-		<parent link="body_link4" />
-		<child link="head_yaw" />
-		<axis xyz="0.036088 0 -0.99935" />
-		<limit lower="-3.14" upper="3.14" effort="100" velocity="1" />
-	</joint>
-	<link name="head_pitch">
-		<inertial>
-			<origin xyz="0.0106970783153679 -0.00153937526954917 0.0535386876730146"/>
-			<mass value="1.96837023227358" />
-			<inertia
-					ixx="0.00378109514744319"
-					ixy="-1.35306059382265E-05"
-					ixz="-4.33373870574624E-05"
-					iyy="0.0035236676197971"
-					iyz="9.33508804534738E-06"
-					izz="0.00568993406575938" />
-		</inertial>
-		<visual>
-			<geometry>
-				<mesh filename="file://$(find fiveages_w2_description)/meshes/body/head_pitch.obj" />
-			</geometry>
-		</visual>
-		<collision>
-			<geometry>
-				<mesh filename="file://$(find fiveages_w2_description)/meshes/body/head_pitch.obj" />
-			</geometry>
-		</collision>
-	</link>
-	<joint name="head_joint2" type="revolute">
-		<origin xyz="0 0.0315 0"/>
-		<parent link="head_yaw" />
-		<child link="head_pitch" />
-		<axis xyz="0 -1 0" />
-		<limit lower="-3.14" upper="3.14" effort="100" velocity="1" />
-	</joint>
-	<!-- Alias link for compatibility with arms_target_manager (which expects head_link2) -->
-	<link name="head_link2"/>
-	<joint name="head_link2_alias_joint" type="fixed">
-		<parent link="head_pitch"/>
-		<child link="head_link2"/>
-		<origin xyz="0 0 0" rpy="0 0 0"/>
-	</joint>
-	<link name="arm_base"/>
-	<joint name="arm_base_joint" type="fixed">
-		<origin xyz="-0.0164439628111166 0 0.457354971463696"/>
-		<parent link="body_link4" />
-		<child link="arm_base" />
-	</joint>
+	<xacro:include filename="$(find fiveages_w2_description)/xacro/body.xacro"/>
 	<!-- Left Arm -->
 	<joint name="left_arm_base_joint" type="fixed">

File: xacro/ros2_control/robot.xacro (robot description, xacro)
@@ -6,24 +6,24 @@
 	<xacro:include filename="$(find fiveages_w2_description)/xacro/ros2_control/body.xacro"/>
 	<!-- <xacro:include filename="$(find fiveages_w2_description)/xacro/ros2_control/chassis.xacro"/> -->
-    <ros2_control name="fiveages_w2_system" type="system">
-        <hardware>
-            <xacro:if value="${'$(arg ros2_control_hardware_type)' == 'gz'}">
-                <plugin>gz_ros2_control/GazeboSimSystem</plugin>
-            </xacro:if>
-            <xacro:if value="${'$(arg ros2_control_hardware_type)' == 'mock_components'}">
-                <plugin>mock_components/GenericSystem</plugin>
-            </xacro:if>
-            <xacro:if value="${'$(arg ros2_control_hardware_type)' == 'isaac'}">
-                <plugin>topic_based_ros2_control/TopicBasedSystem</plugin>
-                <param name="joint_commands_topic">/isaac/joint_command</param>
-                <param name="joint_states_topic">/isaac/joint_states</param>
-                <param name="sum_wrapped_joint_states">false</param>
-                <param name="initialize_commands_from_state">true</param>
-            </xacro:if>
-        </hardware>
-        <xacro:body_interfaces/>
-        <xacro:m6_interfaces name="left"/>
-        <xacro:m6_interfaces name="right"/>
-    </ros2_control>
+	<ros2_control name="fiveages_w2_system" type="system">
+		<hardware>
+			<xacro:if value="${'$(arg ros2_control_hardware_type)' == 'gz'}">
+				<plugin>gz_ros2_control/GazeboSimSystem</plugin>
+			</xacro:if>
+			<xacro:if value="${'$(arg ros2_control_hardware_type)' == 'mock_components'}">
+				<plugin>mock_components/GenericSystem</plugin>
+			</xacro:if>
+			<xacro:if value="${'$(arg ros2_control_hardware_type)' == 'isaac'}">
+				<plugin>topic_based_ros2_control/TopicBasedSystem</plugin>
+				<param name="joint_commands_topic">/isaac/joint_command</param>
+				<param name="joint_states_topic">/isaac/joint_states</param>
+				<param name="sum_wrapped_joint_states">false</param>
+				<param name="initialize_commands_from_state">true</param>
+			</xacro:if>
+		</hardware>
+		<xacro:body_interfaces/>
+		<xacro:m6_interfaces name="left"/>
+		<xacro:m6_interfaces name="right"/>
+	</ros2_control>
 	<!-- Gazebo plugin configuration -->
 	<xacro:arg name="gazebo" default="false"/>

Commit message: add 90c and 90d

File: xacro/component.xacro (robot description, xacro)
@@ -1,5 +1,5 @@
 <?xml version="1.0" ?>
 <!-- =================================================================================== -->
-<!-- |    Complete Robot Description for Agibot G1                                     | -->
+<!-- |    Complete Robot Description for FiveAges W2                                     | -->
 <!-- |    This file includes the base robot structure and both arms                    | -->
 <!-- =================================================================================== -->

File: xacro/grippers.xacro (robot description, xacro)
@@ -15,5 +15,5 @@
             </joint>
         </xacro:if>
-        <xacro:if value="${type == 'ag2f90'}">
+        <xacro:if value="${type == 'ag2f90_c' or type == 'ag2f90_d'}">
             <xacro:include filename="$(find changingtek_description)/xacro/AG2F90-C.xacro"/>
             <xacro:AG2F90-C name="left" use_flange="true"/>

File: xacro/robot.xacro (robot description, xacro)
@@ -21,6 +21,22 @@
 	<xacro:M6_CCS name="left" collider="$(arg collider)"/>
 	<xacro:M6_CCS name="right" direction="-1" collider="$(arg collider)"/>
+	<!-- 从 type 参数解析出 gripper_type -->
 	<xacro:arg name="type" default=""/>
-	<xacro:property name="selected_gripper_type" value="$(arg type)"/>
+	<xacro:property name="type_arg" value="$(arg type)"/>
+	<!-- 默认值 -->
+	<xacro:property name="selected_gripper_type" value=""/>
+	<!-- 从 type 解析 gripper_type -->
+	<xacro:if value="${type_arg == 'rg75'}">
+		<xacro:property name="selected_gripper_type" value="rg75"/>
+	</xacro:if>
+	<xacro:if value="${type_arg == 'ag2f90'}">
+		<xacro:property name="selected_gripper_type" value="ag2f90_d"/>
+	</xacro:if>
+	<xacro:if value="${type_arg == 'ag2f90_c'}">
+		<xacro:property name="selected_gripper_type" value="ag2f90_c"/>
+	</xacro:if>
+	<xacro:if value="${type_arg == 'ag2f90_d'}">
+		<xacro:property name="selected_gripper_type" value="ag2f90_d"/>
+	</xacro:if>
 	<xacro:include filename="$(find fiveages_w2_description)/xacro/grippers.xacro"/>
 	<xacro:Grippers type="${selected_gripper_type}"/>

File: xacro/ros2_control/robot.xacro (robot description, xacro)
@@ -9,9 +9,13 @@
 			<hardware>
 				<plugin>marvin_ros2_control/MarvinHardware</plugin>
-				<param name="left_right_arm">2</param>
+				<param name="arm_type">dual</param>
+				<param name="ctrl_mode">position</param>
+				<param name="gripper_type">${selected_gripper_type}</param>
+				<param name="max_velocity">40</param>
+				<param name="max_acceleration">10</param>
 			</hardware>
 			<xacro:m6_interfaces name="left"/>
 			<xacro:m6_interfaces name="right"/>
-			<xacro:if value="${'$(arg type)' != ''}">
+			<xacro:if value="${selected_gripper_type != ''}">
 				<joint name="left_gripper_joint">
 					<command_interface name="position"/>
@@ -62,5 +66,5 @@
 			<xacro:m6_interfaces name="right"/>
 			<xacro:if
-					value="${'$(arg type)' == 'rg75' or '$(arg type)' == 'leapmotor'}">
+					value="${selected_gripper_type == 'rg75'}">
 				<xacro:include filename="$(find jodell_description)/xacro/ros2_control/RG75-300.xacro"/>
 				<xacro:rg75_interfaces name="left"/>
@@ -68,5 +72,5 @@
 			</xacro:if>
 			<xacro:if
-					value="${'$(arg type)' == 'ag2f90'}">
+					value="${selected_gripper_type == 'ag2f90_c' or selected_gripper_type == 'ag2f90_d'}">
 				<xacro:include filename="$(find changingtek_description)/xacro/ros2_control/AG2F90-C.xacro"/>
 				<xacro:ag2f90c_interfaces name="left"/>

Commit message: add launch configuration for linkerhand o7

File: xacro/component.xacro (robot description, xacro)
@@ -1,11 +1,8 @@
 <?xml version="1.0" ?>
-<!-- =================================================================================== -->
-<!-- |    Complete Robot Description for FiveAges W2                                     | -->
-<!-- |    This file includes the base robot structure and both arms                    | -->
-<!-- =================================================================================== -->
-<robot name="FiveAges_W2" xmlns:xacro="http://www.ros.org/wiki/xacro">
-	<xacro:arg name="type" default="linkhou_q2"/>
+<robot name="M6 CCS Dual" xmlns:xacro="http://www.ros.org/wiki/xacro">
+	<xacro:property name="PI" value="3.1415926535897931"/>
+	<xacro:arg name="type" default="linkhou_s2"/>
 	<xacro:arg name="chassis_joints_movable" default="true"/>
-	<xacro:if value="${'$(arg type)' == 'linkhou_q2'}">
+	<xacro:if value="${'$(arg type)' == 'linkhou_s2'}">
 		<xacro:include filename="$(find fiveages_w2_description)/xacro/components/linkhou_s2.xacro"/>
 		<xacro:linkhou_s2 joints_movable="$(arg chassis_joints_movable)"/>
@@ -15,3 +12,19 @@
 		<xacro:include filename="$(find fiveages_w2_description)/xacro/components/body.xacro"/>
 	</xacro:if>
+	<xacro:if value="${'$(arg type)' == 'arms'}">
+		<link name="arm_base"/>
+		<joint name="left_arm_base_joint" type="fixed">
+			<parent link="arm_base"/>
+			<child link="left_base_link"/>
+			<origin rpy="-${PI/2} 0 0" xyz="0.0 0.062 0"/>
+		</joint>
+		<joint name="right_arm_base_joint" type="fixed">
+			<parent link="arm_base"/>
+			<child link="right_base_link"/>
+			<origin rpy="${PI/2} 0 0" xyz="0 -0.062 0"/>
+		</joint>
+		<xacro:include filename="$(find m6_ccs_description)/xacro/arm.xacro"/>
+		<xacro:M6_CCS name="left" style="fiveages_w2"/>
+		<xacro:M6_CCS name="right" direction="-1" style="fiveages_w2"/>
+	</xacro:if>
 </robot>

Commit message: add rg75 heavy config

File: xacro/component.xacro (robot description, xacro)
@@ -1,4 +1,4 @@
 <?xml version="1.0" ?>
-<robot name="M6 CCS Dual" xmlns:xacro="http://www.ros.org/wiki/xacro">
+<robot name="FiveAges W2" xmlns:xacro="http://www.ros.org/wiki/xacro">
 	<xacro:property name="PI" value="3.1415926535897931"/>
 	<xacro:arg name="type" default="linkhou_s2"/>

File: xacro/eefs.xacro (robot description, xacro)
@@ -38,13 +38,19 @@
         <xacro:if value="${gripper_type == 'rg75'}">
             <xacro:include filename="$(find jodell_description)/xacro/RG75-300.xacro"/>
-            <xacro:RG75-300 name="left" use_flange="true"/>
-            <xacro:RG75-300 name="right" use_flange="true"/>
+            <xacro:RG75-300 name="left" use_flange="true" pad="${selected_gripper_pad}"/>
+            <xacro:RG75-300 name="right" use_flange="true" pad="${selected_gripper_pad}"/>
             <joint name="left_gripper_base_joint" type="fixed">
                 <parent link="left_tcp"/>
                 <child link="left_flange"/>
+                <xacro:if value="${selected_gripper_pad == 'heavy_carry'}">
+                    <origin rpy="0 0 ${PI/2}"/>
+                </xacro:if>
             </joint>
             <joint name="right_gripper_base_joint" type="fixed">
                 <parent link="right_tcp"/>
                 <child link="right_flange"/>
+                <xacro:if value="${selected_gripper_pad == 'heavy_carry'}">
+                    <origin rpy="0 0 ${PI/2}"/>
+                </xacro:if>
             </joint>
         </xacro:if>

File: xacro/robot.xacro (robot description, xacro)
@@ -9,8 +9,13 @@
 	<xacro:property name="selected_hand_type" value=""/>
 	<xacro:property name="selected_gripper_type" value=""/>
+	<xacro:property name="selected_gripper_pad" value="default"/>
 	<!-- 从 type 解析 hand_type 和 gripper_type -->
 	<!-- 夹爪类型：selected_gripper_type 不为空即表示使用夹爪 -->
 	<xacro:if value="${type_arg == 'rg75'}">
 		<xacro:property name="selected_gripper_type" value="rg75"/>
+	</xacro:if>
+	<xacro:if value="${type_arg == 'rg75_heavy'}">
+		<xacro:property name="selected_gripper_type" value="rg75"/>
+		<xacro:property name="selected_gripper_pad" value="heavy_carry"/>
 	</xacro:if>
 	<xacro:if value="${type_arg == 'ag2f90'}">

Commit message: ocs2 wbc config

File: xacro/component.xacro (robot description, xacro)
@@ -28,3 +28,8 @@
 		<xacro:M6_CCS name="right" direction="-1" style="fiveages_w2"/>
 	</xacro:if>
+	<xacro:if value="${'$(arg type)' == 'lp02_336_camera'}">
+		<link name="base_link"/>
+		<xacro:include filename="$(find fiveages_w2_description)/xacro/components/lp02_336_camera.xacro"/>
+		<xacro:lp02_336_camera prefix="" parent_link="base_link"/>
+	</xacro:if>
 </robot>

File: xacro/eefs.xacro (robot description, xacro)
@@ -1,4 +1,5 @@
 <?xml version="1.0"?>
 <robot xmlns:xacro="http://www.ros.org/wiki/xacro">
+    <xacro:include filename="$(find fiveages_w2_description)/xacro/components/lp02_336_camera.xacro"/>
     <xacro:macro name="EndEffectors" params="hand_type:='' gripper_type:=''">
         <!-- Note:
@@ -47,4 +48,6 @@
                 </xacro:if>
             </joint>
+            <xacro:lp02_336_camera prefix="left_" parent_link="left_flange"/>
+            <xacro:lp02_336_camera prefix="right_" parent_link="right_flange"/>
             <joint name="right_gripper_base_joint" type="fixed">
                 <parent link="right_tcp"/>

Commit message: Remove body (#9)
* Add common controller defaults and update robot.xacro for configuration

* 默认不开启外部底盘topic监听

* 身体升降和旋转使用不同的配置参数

* update

* update yaml using common.yaml

* Refactor ROS2 control configuration files

- Cleaned up the `linkerhand_o7.yaml` by removing commented-out parameters and organizing controller configurations.
- Simplified `rg75.yaml` and `rg75_heavy.yaml` by removing unnecessary comments and retaining only essential parameters.
- Updated `ros2_controllers.yaml` to streamline controller definitions and remove redundant comments, focusing on active configurations.
- Consolidated home position definitions and removed deprecated parameters across all configuration files for clarity and maintainability.

* update 左右手hand controller in common.yaml

* Refactor YAML configuration files by removing unused hand controllers and cleaning up parameters

* update

* remove linkhou

* update body param

---------

Co-authored-by: ldh9299 <929908985@qq.com>
Co-authored-by: Zinan <zacharyx359@gmail.com>

File: xacro/component.xacro (robot description, xacro)
@@ -2,14 +2,5 @@
 <robot name="FiveAges W2" xmlns:xacro="http://www.ros.org/wiki/xacro">
 	<xacro:property name="PI" value="3.1415926535897931"/>
-	<xacro:arg name="type" default="linkhou_s2"/>
-	<xacro:arg name="chassis_joints_movable" default="true"/>
-	<xacro:if value="${'$(arg type)' == 'linkhou_s2'}">
-		<xacro:include filename="$(find fiveages_w2_description)/xacro/components/linkhou_s2.xacro"/>
-		<xacro:linkhou_s2 joints_movable="$(arg chassis_joints_movable)"/>
-	</xacro:if>
-	<xacro:if value="${'$(arg type)' == 'body'}">
-		<link name="base_link"/>
-		<xacro:include filename="$(find fiveages_w2_description)/xacro/components/body.xacro"/>
-	</xacro:if>
+	<xacro:arg name="type" default="arms"/>
 	<xacro:if value="${'$(arg type)' == 'arms'}">
 		<link name="arm_base"/>

File: xacro/robot.xacro (robot description, xacro)
@@ -1,6 +1,7 @@
 <?xml version="1.0"?>
 <robot name="FiveAges W2" xmlns:xacro="http://www.ros.org/wiki/xacro">
-    <xacro:arg name="collider" default="convex"/>
+    <xacro:arg name="collider" default="simple"/>
     <xacro:arg name="chassis_joints_movable" default="false"/>
+    <xacro:arg name="variant" default=""/>
     <!-- 从 type 参数解析出 hand_type 和 gripper_type -->
     <xacro:arg name="type" default=""/>
@@ -38,7 +39,10 @@
         <xacro:property name="selected_hand_type" value="linkerhand_o7"/>
     </xacro:if>
-    <xacro:include filename="$(find fiveages_w2_description)/xacro/components/linkhou_s2.xacro"/>
-    <xacro:linkhou_s2 joints_movable="$(arg chassis_joints_movable)"/>
-    <xacro:include filename="$(find fiveages_w2_description)/xacro/components/body.xacro"/>
+    <xacro:include filename="$(find fiveages_w2_common_description)/xacro/components/linkhou_s2.xacro"/>
+    <xacro:linkhou_s2 joints_movable="$(arg chassis_joints_movable)" variant="$(arg variant)"/>
+    <xacro:include filename="$(find fiveages_w2_common_description)/xacro/components/body.xacro"/>
+    <xacro:body variant="$(arg variant)"/>
+    <xacro:include filename="$(find fiveages_w2_common_description)/xacro/components/head.xacro"/>
+    <xacro:head variant="$(arg variant)"/>
     <!-- Left Arm -->
     <joint name="left_arm_base_joint" type="fixed">

File: xacro/ros2_control/robot.xacro (robot description, xacro)
@@ -6,5 +6,5 @@
 	<xacro:include filename="$(find fiveages_w2_description)/xacro/robot.xacro"/>
 	<xacro:include filename="$(find m6_ccs_description)/xacro/ros2_control/interfaces.xacro"/>
-	<xacro:include filename="$(find fiveages_w2_description)/xacro/ros2_control/body.xacro"/>
+	<xacro:include filename="$(find fiveages_w2_common_description)/xacro/ros2_control/body.xacro"/>
 	<xacro:if value="${is_real_hardware}">
 		<!-- 确定传递给 marvin_ros2_control 的 gripper_type 参数 -->
