Commit message: feat(robot): platform_variant and m6 skin for arm visuals; drop meshes/arm
Co-authored-by: Cursor <cursoragent@cursor.com>

File: xacro/component.xacro (robot description, xacro)
@@ -2,10 +2,11 @@
 <robot name="FiveAges W2" xmlns:xacro="http://www.ros.org/wiki/xacro">
 	<xacro:arg name="type" default="arms"/>
+	<xacro:arg name="variant" default=""/>
 	<xacro:if value="${'$(arg type)' == 'arms'}">
 		<xacro:include filename="$(find m6_ccs_description)/xacro/arm_mount.xacro"/>
 		<xacro:DualArmBase/>
 		<xacro:include filename="$(find m6_ccs_description)/xacro/arm.xacro"/>
-		<xacro:M6_CCS name="left" style="fiveages_w2"/>
-		<xacro:M6_CCS name="right" direction="-1" style="fiveages_w2"/>
+		<xacro:M6_CCS name="left" skin="fiveages_w2" variant="$(arg variant)"/>
+		<xacro:M6_CCS name="right" direction="-1" skin="fiveages_w2" variant="$(arg variant)"/>
 	</xacro:if>
 </robot>

File: xacro/robot.xacro (robot description, xacro)
@@ -21,25 +21,26 @@
     <xacro:set_side_eef_types side="right" type_key="${effective_right_type}"/>
     <xacro:property name="chassis_arg" value="$(arg chassis)"/>
-    <xacro:property name="chassis_variant" value="$(arg variant)"/>
+    <!-- platform-wide OEM visual variant (launch/profile: variant); not the chassis model selector -->
+    <xacro:property name="platform_variant" value="$(arg variant)"/>
     <xacro:if value="${chassis_arg == 'linkhou_s2_sinopec'}">
-        <xacro:property name="chassis_variant" value="sinopec"/>
+        <xacro:property name="platform_variant" value="sinopec"/>
     </xacro:if>
     <xacro:if value="${chassis_arg == 'linkhou_s2' or chassis_arg == 'linkhou_s2_sinopec'}">
         <xacro:include filename="$(find fiveages_w2_common_description)/xacro/components/linkhou_s2.xacro"/>
-        <xacro:linkhou_s2 joints_movable="$(arg chassis_joints_movable)" variant="${chassis_variant}"/>
+        <xacro:linkhou_s2 joints_movable="$(arg chassis_joints_movable)" variant="${platform_variant}"/>
     </xacro:if>
     <xacro:if value="${chassis_arg == 'linkhou_s2_v2'}">
         <xacro:include filename="$(find fiveages_w2_common_description)/xacro/components/linkhou_s2_v2.xacro"/>
-        <xacro:linkhou_s2 joints_movable="$(arg chassis_joints_movable)" variant="${chassis_variant}"/>
+        <xacro:linkhou_s2 joints_movable="$(arg chassis_joints_movable)" variant="${platform_variant}"/>
     </xacro:if>
     <xacro:include filename="$(find fiveages_w2_common_description)/xacro/components/body.xacro"/>
-    <xacro:body variant="${chassis_variant}"/>
+    <xacro:body variant="${platform_variant}"/>
     <xacro:include filename="$(find fiveages_w2_common_description)/xacro/components/head.xacro"/>
-    <xacro:head variant="${chassis_variant}"/>
+    <xacro:head variant="${platform_variant}"/>
     <xacro:include filename="$(find m6_ccs_description)/xacro/arm_mount.xacro"/>
     <xacro:DualArmMount parent="arm_base"/>
     <xacro:include filename="$(find m6_ccs_description)/xacro/arm.xacro"/>
-    <xacro:M6_CCS name="left" style="fiveages_w2"/>
-    <xacro:M6_CCS name="right" direction="-1" style="fiveages_w2"/>
+    <xacro:M6_CCS name="left" skin="fiveages_w2" variant="${platform_variant}"/>
+    <xacro:M6_CCS name="right" direction="-1" skin="fiveages_w2" variant="${platform_variant}"/>
     <xacro:include filename="$(find m6_ccs_description)/xacro/eefs.xacro"/>
     <xacro:EndEffectors
