Commit message: add white skin

File: xacro/component.xacro (robot description, xacro)
@@ -8,6 +8,7 @@
 		<xacro:DualArmBase/>
 		<xacro:include filename="$(find m6_ccs_description)/xacro/arm.xacro"/>
-		<xacro:M6_CCS name="left" skin="fiveages_w2" variant="$(arg variant)"/>
-		<xacro:M6_CCS name="right" direction="-1" skin="fiveages_w2" variant="$(arg variant)"/>
+		<xacro:property name="arm_skin" value="${'default' if '$(arg variant)' == 'white' else 'fiveages_w2'}"/>
+		<xacro:M6_CCS name="left" skin="${arm_skin}" variant="$(arg variant)"/>
+		<xacro:M6_CCS name="right" direction="-1" skin="${arm_skin}" variant="$(arg variant)"/>
 	</xacro:if>
 </robot>

File: xacro/robot.xacro (robot description, xacro)
@@ -45,8 +45,10 @@
     <xacro:DualArmMount parent="arm_base"/>
     <xacro:include filename="$(find m6_ccs_description)/xacro/arm.xacro"/>
-    <xacro:M6_CCS name="left" skin="fiveages_w2" variant="${platform_variant}"
+    <!-- white platform: M6-CCS factory (default) visuals; otherwise W2 repaint -->
+    <xacro:property name="arm_skin" value="${'default' if platform_variant == 'white' else 'fiveages_w2'}"/>
+    <xacro:M6_CCS name="left" skin="${arm_skin}" variant="${platform_variant}"
         tcp_offset_xyz="$(arg left_tcp_offset_xyz)"
         tcp_offset_rpy="$(arg left_tcp_offset_rpy)"/>
-    <xacro:M6_CCS name="right" direction="-1" skin="fiveages_w2" variant="${platform_variant}"
+    <xacro:M6_CCS name="right" direction="-1" skin="${arm_skin}" variant="${platform_variant}"
         tcp_offset_xyz="$(arg right_tcp_offset_xyz)"
         tcp_offset_rpy="$(arg right_tcp_offset_rpy)"/>
