Commit message: update collision for gripper

File: urdf/fiveages_w2_ag2f90.urdf (robot description, URDF)
Before this commit: robot FiveAges W2, 69 links, 68 joints
Links:
- link left_link7: geometry collision cylinder length=0.038392 radius=0.041707; collision cylinder length=0.08 radius=0.021707
- link right_link7: geometry collision cylinder length=0.038392 radius=0.041707; collision cylinder length=0.08 radius=0.021707

File: urdf/fiveages_w2_rg75.urdf (robot description, URDF)
Before this commit: robot FiveAges W2, 57 links, 56 joints
Links:
- link left_link7: geometry collision cylinder length=0.038392 radius=0.041707; collision cylinder length=0.08 radius=0.021707
- link right_link7: geometry collision cylinder length=0.038392 radius=0.041707; collision cylinder length=0.08 radius=0.021707

File: xacro/components/arm.xacro (robot description, xacro)
@@ -1,6 +1,8 @@
 <?xml version="1.0"?>
 <robot xmlns:xacro="http://www.ros.org/wiki/xacro">
+	<xacro:arg name="collider" default="convex"/>
 	<xacro:property name="PI" value="3.1415926535897931"/>
-	<xacro:macro name="M6_CCS" params="name:='' direction:=1 collider:=convex">
+	<xacro:property name="collider_type" value="$(arg collider)"/>
+	<xacro:macro name="M6_CCS" params="name:='' direction:=1">
 		<xacro:property name="prefix" value="${name + '_' if name else ''}"/>
 		<!-- Base Link -->
@@ -18,5 +20,5 @@
 				</geometry>
 			</visual>
-			<xacro:if value="${collider == 'convex'}">
+			<xacro:if value="${collider_type == 'convex'}">
 				<collision>
 					<geometry>
@@ -25,5 +27,5 @@
 				</collision>
 			</xacro:if>
-			<xacro:if value="${collider == 'simple'}">
+			<xacro:if value="${collider_type == 'simple'}">
 				<collision>
 					<origin xyz="0 0 0.041832"/>
@@ -48,5 +50,5 @@
 				</geometry>
 			</visual>
-			<xacro:if value="${collider == 'convex'}">
+			<xacro:if value="${collider_type == 'convex'}">
 				<collision>
 					<geometry>
@@ -55,5 +57,5 @@
 				</collision>
 			</xacro:if>
-			<xacro:if value="${collider == 'simple'}">
+			<xacro:if value="${collider_type == 'simple'}">
 				<collision>
 					<origin rpy="${PI/2} 0 0"/>
@@ -86,12 +88,12 @@
 				</geometry>
 			</visual>
-			<xacro:if value="${collider == 'convex'}">
-				<collision>
-					<geometry>
-						<mesh filename="file://$(find m6_ccs_description)/meshes/link2.glb" scale="1 1 ${direction}"/>
-					</geometry>
-				</collision>
-			</xacro:if>
-			<xacro:if value="${collider == 'simple'}">
+			<xacro:if value="${collider_type == 'convex'}">
+				<collision>
+					<geometry>
+						<mesh filename="file://$(find m6_ccs_description)/meshes/link2.glb"/>
+					</geometry>
+				</collision>
+			</xacro:if>
+			<xacro:if value="${collider_type == 'simple'}">
 				<collision>
 					<origin xyz="0 0.099087 0" rpy="${PI/2} 0 0"/>
@@ -124,5 +126,5 @@
 				</geometry>
 			</visual>
-			<xacro:if value="${collider == 'convex'}">
+			<xacro:if value="${collider_type == 'convex'}">
 				<collision>
 					<geometry>
@@ -131,5 +133,5 @@
 				</collision>
 			</xacro:if>
-			<xacro:if value="${collider == 'simple'}">
+			<xacro:if value="${collider_type == 'simple'}">
 				<collision>
 					<origin xyz="0 0 -0.098932"/>
@@ -168,5 +170,5 @@
 				</geometry>
 			</visual>
-			<xacro:if value="${collider == 'convex'}">
+			<xacro:if value="${collider_type == 'convex'}">
 				<collision>
 					<geometry>
@@ -175,5 +177,5 @@
 				</collision>
 			</xacro:if>
-			<xacro:if value="${collider == 'simple'}">
+			<xacro:if value="${collider_type == 'simple'}">
 				<collision>
 					<origin xyz="0.017721 -0.079733 0" rpy="${PI/2} 0 0"/>
@@ -206,12 +208,12 @@
 				</geometry>
 			</visual>
-			<xacro:if value="${collider == 'convex'}">
-				<collision>
-					<geometry>
-						<mesh filename="file://$(find m6_ccs_description)/meshes/link5.glb" scale="1 ${direction} 1"/>
-					</geometry>
-				</collision>
-			</xacro:if>
-			<xacro:if value="${collider == 'simple'}">
+			<xacro:if value="${collider_type == 'convex'}">
+				<collision>
+					<geometry>
+						<mesh filename="file://$(find m6_ccs_description)/meshes/link5.glb"/>
+					</geometry>
+				</collision>
+			</xacro:if>
+			<xacro:if value="${collider_type == 'simple'}">
 				<collision>
 					<origin xyz="0 0 -0.117153"/>
@@ -244,5 +246,5 @@
 				</geometry>
 			</visual>
-			<xacro:if value="${collider == 'convex'}">
+			<xacro:if value="${collider_type == 'convex'}">
 				<collision>
 					<geometry>
@@ -251,7 +253,7 @@
 				</collision>
 			</xacro:if>
-			<xacro:if value="${collider == 'simple'}">
-				<collision>
-					<origin xyz="0 0 0" rpy="${PI/2} 0 0"/>
+			<xacro:if value="${collider_type == 'simple'}">
+				<collision>
+					<origin rpy="${PI/2} 0 0"/>
 					<geometry>
 						<cylinder length="0.108046" radius="0.038348"/>
@@ -287,5 +289,5 @@
 				</geometry>
 			</visual>
-			<xacro:if value="${collider == 'convex'}">
+			<xacro:if value="${collider_type == 'convex'}">
 				<collision>
 					<geometry>
@@ -294,5 +296,5 @@
 				</collision>
 			</xacro:if>
-			<xacro:if value="${collider == 'simple'}">
+			<xacro:if value="${collider_type == 'simple'}">
 				<collision>
 					<origin xyz="0 -0.075732 0" rpy="${PI/2} 0 0"/>
@@ -305,5 +307,11 @@
 						<origin xyz="0 -0.175732 0" rpy="${PI/2} 0 0"/>
 						<geometry>
-							<cylinder length="0.138392" radius="0.041707"/>
+							<cylinder length="0.138392" radius="0.05"/>
+						</geometry>
+					</collision>
+					<collision>
+						<origin xyz="0 -0.28 0" rpy="${PI/2} 0 0"/>
+						<geometry>
+							<cylinder length="0.08" radius="0.021707"/>
 						</geometry>
 					</collision>
@@ -316,4 +324,10 @@
 						</geometry>
 					</collision>
+					<collision>
+						<origin xyz="0 -0.28 0" rpy="${PI/2} 0 0"/>
+						<geometry>
+							<cylinder length="0.08" radius="0.021707"/>
+						</geometry>
+					</collision>
 				</xacro:if>
 			</xacro:if>

File: xacro/robot.xacro (robot description, xacro)
@@ -49,6 +49,6 @@
 	</joint>
 	<xacro:include filename="$(find fiveages_w2_description)/xacro/components/arm.xacro"/>
-	<xacro:M6_CCS name="left" collider="$(arg collider)"/>
-	<xacro:M6_CCS name="right" direction="-1" collider="$(arg collider)"/>
+	<xacro:M6_CCS name="left"/>
+	<xacro:M6_CCS name="right" direction="-1"/>
 	<xacro:include filename="$(find fiveages_w2_description)/xacro/eefs.xacro"/>
 	<xacro:EndEffectors hand_type="${selected_hand_type}" gripper_type="${selected_gripper_type}"/>
