Commit message: 修复命名问题以及路径问题

File: urdf/fiveages_w2_rg75.urdf (robot description, URDF)
Before this commit: robot FiveAges W2, 56 links, 55 joints
Links:
- link left_flange: geometry collision mesh filename=package://jodell_description/meshes/RG75/flange.obj; visual mesh filename=package://jodell_description/meshes/RG75/flange.obj
- link left_gripper_base: geometry collision mesh filename=package://jodell_description/meshes/RG75/base.obj; visual mesh filename=package://jodell_description/meshes/RG75/base.obj
- link left_left_finger: geometry collision mesh filename=package://jodell_description/meshes/RG75/finger.obj; visual mesh filename=package://jodell_description/meshes/RG75/finger.obj
- link left_left_finger_pad: geometry collision mesh filename=package://jodell_description/meshes/RG75/pad_fiveages.obj; visual mesh filename=package://jodell_description/meshes/RG75/pad_fiveages.obj
- link left_right_finger: geometry collision mesh filename=package://jodell_description/meshes/RG75/finger.obj scale=-1 -1 1; visual mesh filename=package://jodell_description/meshes/RG75/finger.obj scale=-1 -1 1
- link left_right_finger_pad: geometry collision mesh filename=package://jodell_description/meshes/RG75/pad_fiveages.obj scale=1 -1 1; visual mesh filename=package://jodell_description/meshes/RG75/pad_fiveages.obj scale=1 -1 1
- link right_flange: geometry collision mesh filename=package://jodell_description/meshes/RG75/flange.obj; visual mesh filename=package://jodell_description/meshes/RG75/flange.obj
- link right_gripper_base: geometry collision mesh filename=package://jodell_description/meshes/RG75/base.obj; visual mesh filename=package://jodell_description/meshes/RG75/base.obj
- link right_left_finger: geometry collision mesh filename=package://jodell_description/meshes/RG75/finger.obj; visual mesh filename=package://jodell_description/meshes/RG75/finger.obj
- link right_left_finger_pad: geometry collision mesh filename=package://jodell_description/meshes/RG75/pad_fiveages.obj; visual mesh filename=package://jodell_description/meshes/RG75/pad_fiveages.obj
- link right_right_finger: geometry collision mesh filename=package://jodell_description/meshes/RG75/finger.obj scale=-1 -1 1; visual mesh filename=package://jodell_description/meshes/RG75/finger.obj scale=-1 -1 1
- link right_right_finger_pad: geometry collision mesh filename=package://jodell_description/meshes/RG75/pad_fiveages.obj scale=1 -1 1; visual mesh filename=package://jodell_description/meshes/RG75/pad_fiveages.obj scale=1 -1 1

Commit message: change w2 urdf

File: urdf/fiveages_w2_rg75.urdf (robot description, URDF)
Before this commit: robot FiveAges W2, 57 links, 56 joints
Joints:
- joint left_joint6: limit lower=-1.0122909661567112 upper=1.0122909661567112 effort=18 velocity=3.141592653589793 -> lower=-0.8 upper=0.8 effort=18 velocity=3.141592653589793
- joint right_joint6: limit lower=-1.0122909661567112 upper=1.0122909661567112 effort=18 velocity=3.141592653589793 -> lower=-0.8 upper=0.8 effort=18 velocity=3.141592653589793
