Commit message: 修改碰撞体 配置split body control

File: urdf/fiveages_w2.urdf (robot description, URDF)
Before this commit: robot FiveAges W2, 40 links, 39 joints
Links:
- removed link head_pitch
- removed link head_yaw
- added link head_link1, mass 1.76592019732553; collision mesh filename=file:///home/fiveages/ros2_ws/install/fiveages_w2_descripti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; visual mesh filename=file:///home/fiveages/ros2_ws/install/fiveages_w2_descripti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
- link body_link4: mass 23.7446873792875 -> 23.7446394325596
- link head_link2: mass None -> 1.96836671464479; geometry collision mesh filename=file:///home/fiveages/ros2_ws/install/fiveages_w2_descripti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; visual mesh filename=file:///home/fiveages/ros2_ws/install/fiveages_w2_descripti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
Joints:
- removed joint head_link2_alias_joint
- joint arm_base_joint: origin xyz=-0.0164439628111166 0 0.457354971463696 -> xyz=7.1612E-05 0 0.45765
- joint body_joint1: limit lower=-3.14 upper=3.14 effort=100 velocity=1 -> lower=-1.352633 upper=0.567 effort=100 velocity=1
- joint body_joint2: limit lower=-3.14 upper=3.14 effort=100 velocity=1 -> lower=-2.66 upper=1.605 effort=100 velocity=1
- joint body_joint3: axis 0 -1 0 -> 0 1 0; limit lower=-3.14 upper=3.14 effort=100 velocity=1 -> lower=-1.745 upper=1.745 effort=100 velocity=1
- joint body_joint4: origin xyz=0 -0.0019 0.1443 -> xyz=-7.1612E-05 -0.0019 0.14441
- joint head_joint1: axis 0.036088 0 -0.99935 -> 0 0 1; child head_yaw -> head_link1; origin xyz=-0.046314 -0.0272 0.63334 -> xyz=-0.023428 0 0.48475
- joint head_joint2: child head_pitch -> head_link2; origin xyz=0 0.0315 0 -> xyz=0 0.0042 0.15 rpy=3.1416 0 3.1416; parent head_yaw -> head_link1

File: xacro/ros2_control/body.xacro (robot description, xacro)
@@ -27,5 +27,5 @@
       <!-- <state_interface name="effort"/> -->
     </joint>
-    <!-- <joint name="head_joint1">
+    <joint name="head_joint1">
       <command_interface name="position"/>
       <state_interface name="position"/>
@@ -38,5 +38,5 @@
       <state_interface name="velocity"/>
       <state_interface name="effort"/>
-    </joint> -->
+    </joint>
   </xacro:macro>
 </robot>

Commit message: add isaac config

File: urdf/fiveages_w2.urdf (robot description, URDF)
Before this commit: robot FiveAges W2, 39 links, 38 joints
Links:
- added link base_footprint
- added link body_camera; visual mesh filename=file:///home/fiveages/ros2_ws/install/sensor_models/share/s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
- added link head_camera; visual mesh filename=file:///home/fiveages/ros2_ws/install/sensor_models/share/s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
- link body_base: geometry collision mesh filename=package://fiveages_w2_description/meshes/body/base.obj; visual mesh filename=package://fiveages_w2_description/meshes/body/base.obj
- link body_link1: geometry collision mesh filename=package://fiveages_w2_description/meshes/body/link1.obj; visual mesh filename=package://fiveages_w2_description/meshes/body/link1.obj
- link body_link2: geometry collision mesh filename=package://fiveages_w2_description/meshes/body/link2.obj; visual mesh filename=package://fiveages_w2_description/meshes/body/link2.obj
- link body_link3: geometry collision mesh filename=package://fiveages_w2_description/meshes/body/link3.obj; visual mesh filename=package://fiveages_w2_description/meshes/body/link3.obj
- link body_link4: geometry collision mesh filename=package://fiveages_w2_description/meshes/body/link4.obj; visual mesh filename=package://fiveages_w2_description/meshes/body/link4.obj
- link chassis_base: geometry collision box size=0.5 0.3 0.2; visual mesh filename=package://fiveages_w2_description/meshes/linkhou_s2/base_li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
- link chassis_camera: geometry collision mesh filename=package://fiveages_w2_description/meshes/linkhou_s2/camera.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; visual mesh filename=package://fiveages_w2_description/meshes/linkhou_s2/camera.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
- link fl_lidar: geometry collision mesh filename=package://fiveages_w2_description/meshes/linkhou_s2/lidar.o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; visual mesh filename=package://fiveages_w2_description/meshes/linkhou_s2/lidar.o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
- link fl_steer: geometry visual mesh filename=package://fiveages_w2_description/meshes/linkhou_s2/steer_l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
- link fl_wheel: geometry collision cylinder length=0.046 radius=0.07; visual mesh filename=package://fiveages_w2_description/meshes/linkhou_s2/wheel.o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
- link fr_steer: geometry visual mesh filename=package://fiveages_w2_description/meshes/linkhou_s2/steer_l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 scale=1 -1 1
- link fr_wheel: geometry collision cylinder length=0.046 radius=0.07; visual mesh filename=package://fiveages_w2_description/meshes/linkhou_s2/wheel.o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 scale=1 -1 1
- link head_link1: geometry collision mesh filename=package://fiveages_w2_description/meshes/body/head_yaw.obj; visual mesh filename=package://fiveages_w2_description/meshes/body/head_yaw.obj
- link head_link2: geometry collision mesh filename=package://fiveages_w2_description/meshes/body/head_pitch.obj; visual mesh filename=package://fiveages_w2_description/meshes/body/head_pitch.obj
- link left_base_link: geometry collision cylinder length=0.083664 radius=0.051277; visual mesh filename=package://m6_ccs_description/meshes/base.obj
- link left_link1: geometry collision cylinder length=0.125958 radius=0.057588; visual mesh filename=package://m6_ccs_description/meshes/link1.obj
- link left_link2: geometry collision cylinder length=0.078386 radius=0.046717; visual mesh filename=package://m6_ccs_description/meshes/link2.obj
- link left_link3: geometry collision cylinder length=0.089056 radius=0.046717; collision cylinder length=0.117016 radius=0.049964
- link left_link4: geometry collision cylinder length=0.080203 radius=0.041759; visual mesh filename=package://m6_ccs_description/meshes/link4.obj
- link left_link5: geometry collision cylinder length=0.14268 radius=0.056747; visual mesh filename=package://m6_ccs_description/meshes/link5.obj scale=1 1 1
- link left_link6: geometry collision cylinder length=0.108046 radius=0.038348; visual mesh filename=package://m6_ccs_description/meshes/link6.obj
- link left_link7: geometry collision cylinder length=0.038392 radius=0.041707; visual mesh filename=package://m6_ccs_description/meshes/link7.obj
- link right_base_link: geometry collision cylinder length=0.083664 radius=0.051277; visual mesh filename=package://m6_ccs_description/meshes/base.obj
- link right_link1: geometry collision cylinder length=0.125958 radius=0.057588; visual mesh filename=package://m6_ccs_description/meshes/link1.obj
- link right_link2: geometry collision cylinder length=0.078386 radius=0.046717; visual mesh filename=package://m6_ccs_description/meshes/link2.obj
- link right_link3: geometry collision cylinder length=0.089056 radius=0.046717; collision cylinder length=0.117016 radius=0.049964
- link right_link4: geometry collision cylinder length=0.080203 radius=0.041759; visual mesh filename=package://m6_ccs_description/meshes/link4.obj
- link right_link5: geometry collision cylinder length=0.14268 radius=0.056747; visual mesh filename=package://m6_ccs_description/meshes/link5.obj scale=1 -1 1
- link right_link6: geometry collision cylinder length=0.108046 radius=0.038348; visual mesh filename=package://m6_ccs_description/meshes/link6.obj
- link right_link7: geometry collision cylinder length=0.038392 radius=0.041707; visual mesh filename=package://m6_ccs_description/meshes/link7_r.obj
- link rl_steer: geometry visual mesh filename=package://fiveages_w2_description/meshes/linkhou_s2/steer_l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
- link rl_wheel: geometry collision cylinder length=0.046 radius=0.07; visual mesh filename=package://fiveages_w2_description/meshes/linkhou_s2/wheel.o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
- link rr_lidar: geometry collision mesh filename=package://fiveages_w2_description/meshes/linkhou_s2/lidar.o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; visual mesh filename=package://fiveages_w2_description/meshes/linkhou_s2/lidar.o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
- link rr_steer: geometry visual mesh filename=package://fiveages_w2_description/meshes/linkhou_s2/steer_l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 scale=1 -1 1
- link rr_wheel: geometry collision cylinder length=0.046 radius=0.07; visual mesh filename=package://fiveages_w2_description/meshes/linkhou_s2/wheel.o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 scale=1 -1 1
Joints:
- added joint base_footprint_joint: type fixed, parent base_footprint, child base_link, origin xyz=0 0 0.04
- added joint body_camera_joint: type fixed, parent body_link4, child body_camera, origin xyz=0.10065 0.024257 0.28812 rpy=3.141592653589793 0.378684973 0
- added joint head_camera_joint: type fixed, parent head_link2, child head_camera, origin xyz=-0.097847  0.046703 -0.12364 rpy=0 -0.64460396 3.141592653589793
- joint base_link_mount: origin rpy=0 0 3.1415926535 -> rpy=0 0 3.141592653589793
- joint body_joint2: origin xyz=0 0 0.323 -> xyz=0 0 0.322
- joint body_joint3: origin xyz=0 0.0019 0.35294 -> xyz=0 0.0019 0.355
- joint body_joint4: limit lower=-3.14 upper=3.14 effort=100 velocity=1 -> lower=-3.141592653589793 upper=3.141592653589793 effort=100 velocity=1; origin xyz=-7.1612E-05 -0.0019 0.14441 -> xyz=-7.1612E-05 -0.0019 0.14331
- joint chassis_camera_joint: origin xyz=-0.3438 -0.00032028 0.159 rpy=0 0 3.1416 -> xyz=-0.3438 -0.00032028 0.159 rpy=0 0 3.141592653589793
- joint fl_lidar_joint: origin xyz=-0.21412 -0.19406 0.32957 rpy=1.5708 -1.309 3.1416 -> xyz=-0.21412 -0.19406 0.32957 rpy=1.5707963267948966 -1.309 3.1416
- joint fl_steer_joint: limit lower=-2.97 upper=2.97 effort=0 velocity=6.28 -> lower=-3.141592653589793 upper=3.141592653589793 effort=5 velocity=6.28
- joint fl_wheel_joint: limit effort=0 velocity=6.28 -> (none)
- joint fr_steer_joint: limit lower=-2.97 upper=2.97 effort=0 velocity=6.28 -> lower=-3.141592653589793 upper=3.141592653589793 effort=5 velocity=6.28
- joint fr_wheel_joint: axis 0 -1 0 -> 0 1 0; limit lower=-2.97 upper=2.97 effort=0 velocity=6.28 -> (none); type revolute -> continuous
- joint head_joint2: origin xyz=0 0.0042 0.15 rpy=3.1416 0 3.1416 -> xyz=0 0.0042 0.15 rpy=3.141592653589793 0 3.141592653589793
- joint left_arm_base_joint: origin xyz=0.0 0.062 0 rpy=-1.5708 0 0 -> xyz=0.0 0.062 0 rpy=-1.5707963267948966 0 0
- joint left_joint1: limit lower=-3.1067 upper=3.1067 effort=108 velocity=3.1416 -> lower=-3.1067 upper=3.1067 effort=108 velocity=3.141592653589793
- joint left_joint2: limit lower=-2.0944 upper=2.0944 effort=108 velocity=3.1416 -> lower=-2.0944 upper=2.0944 effort=108 velocity=3.141592653589793; origin rpy=1.5708 0 0 -> rpy=1.5707963267948966 0 0
- joint left_joint3: limit lower=-3.1067 upper=3.1067 effort=66 velocity=3.1416 -> lower=-3.1067 upper=3.1067 effort=66 velocity=3.141592653589793; origin xyz=0 0.287 0 rpy=-1.5708 0 0 -> xyz=0 0.287 0 rpy=-1.5707963267948966 0 0
- joint left_joint4: limit lower=-2.5307 upper=1.0472 effort=66 velocity=3.1416 -> lower=-2.5307 upper=1.0472 effort=66 velocity=3.141592653589793; origin xyz=0.018 0 0 rpy=-1.5708 0 3.1416 -> xyz=0.018 0 0 rpy=-1.5707963267948966 0 3.141592653589793
- joint left_joint5: limit lower=-3.1067 upper=3.1067 effort=18 velocity=3.1416 -> lower=-3.1067 upper=3.1067 effort=18 velocity=3.141592653589793; origin xyz=0.018 -0.314 0 rpy=-1.5708 0 3.1416 -> xyz=0.018 -0.314 0 rpy=-1.5707963267948966 0 3.141592653589793
- joint left_joint6: limit lower=-1.0472 upper=1.0472 effort=18 velocity=3.1416 -> lower=-1.0472 upper=1.0472 effort=18 velocity=3.141592653589793; origin rpy=1.5708 -1.5708 0 -> rpy=1.5707963267948966 -1.5707963267948966 0
- joint left_joint7: limit lower=-1.5708 upper=1.5708 effort=18 velocity=3.1416 -> lower=-1.5707963267948966 upper=1.5707963267948966 effort=18 velocity=3.141592653589793; origin rpy=1.5708 -1.5708 0 -> rpy=1.5707963267948966 -1.5707963267948966 0
- joint right_arm_base_joint: origin xyz=0 -0.062 0 rpy=1.5708 0 0 -> xyz=0 -0.062 0 rpy=1.5707963267948966 0 0
- joint right_joint1: limit lower=-3.1067 upper=3.1067 effort=108 velocity=3.1416 -> lower=-3.1067 upper=3.1067 effort=108 velocity=3.141592653589793
- joint right_joint2: limit lower=-2.0944 upper=2.0944 effort=108 velocity=3.1416 -> lower=-2.0944 upper=2.0944 effort=108 velocity=3.141592653589793; origin rpy=1.5708 0 0 -> rpy=1.5707963267948966 0 0
- joint right_joint3: limit lower=-3.1067 upper=3.1067 effort=66 velocity=3.1416 -> lower=-3.1067 upper=3.1067 effort=66 velocity=3.141592653589793; origin xyz=0 0.287 0 rpy=-1.5708 0 0 -> xyz=0 0.287 0 rpy=-1.5707963267948966 0 0
- joint right_joint4: limit lower=-2.5307 upper=1.0472 effort=66 velocity=3.1416 -> lower=-2.5307 upper=1.0472 effort=66 velocity=3.141592653589793; origin xyz=0.018 0 0 rpy=-1.5708 0 3.1416 -> xyz=0.018 0 0 rpy=-1.5707963267948966 0 3.141592653589793
- joint right_joint5: limit lower=-3.1067 upper=3.1067 effort=18 velocity=3.1416 -> lower=-3.1067 upper=3.1067 effort=18 velocity=3.141592653589793; origin xyz=0.018 -0.314 0 rpy=-1.5708 0 3.1416 -> xyz=0.018 -0.314 0 rpy=-1.5707963267948966 0 3.141592653589793
- joint right_joint6: limit lower=-1.0472 upper=1.0472 effort=18 velocity=3.1416 -> lower=-1.0472 upper=1.0472 effort=18 velocity=3.141592653589793; origin rpy=1.5708 -1.5708 0 -> rpy=1.5707963267948966 -1.5707963267948966 0
- joint right_joint7: limit lower=-1.5708 upper=1.5708 effort=18 velocity=3.1416 -> lower=-1.5707963267948966 upper=1.5707963267948966 effort=18 velocity=3.141592653589793; origin rpy=1.5708 -1.5708 0 -> rpy=1.5707963267948966 -1.5707963267948966 0
- joint rl_steer_joint: limit lower=-2.97 upper=2.97 effort=0 velocity=6.28 -> lower=-3.141592653589793 upper=3.141592653589793 effort=5 velocity=6.28
- joint rl_wheel_joint: limit effort=0 velocity=6.28 -> (none)
- joint rr_lidar_joint: origin xyz=0.21412 0.19406 0.32957 rpy=1.5708 -1.309 0 -> xyz=0.21412 0.19406 0.32957 rpy=1.5707963267948966 -1.309 0
- joint rr_steer_joint: limit lower=-2.97 upper=2.97 effort=0 velocity=6.28 -> lower=-3.141592653589793 upper=3.141592653589793 effort=5 velocity=6.28
- joint rr_wheel_joint: axis 0 -1 0 -> 0 1 0; limit lower=-2.97 upper=2.97 effort=0 velocity=6.28 -> (none); type revolute -> continuous

File: xacro/body.xacro (robot description, xacro)
@@ -83,5 +83,5 @@
 	</link>
 	<joint name="body_joint2" type="revolute">
-		<origin xyz="0 0 0.323"/>
+		<origin xyz="0 0 0.322"/>
 		<parent link="body_link1"/>
 		<child link="body_link2"/>
@@ -113,5 +113,5 @@
 	</link>
 	<joint name="body_joint3" type="revolute">
-		<origin xyz="0 0.0019 0.35294"/>
+		<origin xyz="0 0.0019 0.355"/>
 		<parent link="body_link2"/>
 		<child link="body_link3"/>
@@ -143,9 +143,21 @@
 	</link>
 	<joint name="body_joint4" type="revolute">
-		<origin xyz="-7.1612E-05 -0.0019 0.14441"/>
+		<origin xyz="-7.1612E-05 -0.0019 0.14331"/>
 		<parent link="body_link3"/>
 		<child link="body_link4"/>
 		<axis xyz="0 0 -1"/>
 		<limit lower="-${PI}" upper="${PI}" effort="100" velocity="1"/>
+	</joint>
+	<link name="body_camera">
+<!--		<visual>-->
+<!--			<geometry>-->
+<!--				<mesh filename="file://$(find sensor_models)/meshes/orbbec/336.obj"/>-->
+<!--			</geometry>-->
+<!--		</visual>-->
+	</link>
+	<joint name="body_camera_joint" type="fixed">
+		<origin xyz="0.10065 0.024257 0.28812" rpy="${PI} 0.378684973 0"/>
+		<parent link="body_link4"/>
+		<child link="body_camera"/>
 	</joint>
 	<link name="head_link1">
@@ -209,4 +221,16 @@
 		<limit lower="-3.14" upper="3.14" effort="100" velocity="1"/>
 	</joint>
+	<link name="head_camera">
+<!--		<visual>-->
+<!--			<geometry>-->
+<!--				<mesh filename="file://$(find sensor_models)/meshes/orbbec/336L.obj"/>-->
+<!--			</geometry>-->
+<!--		</visual>-->
+	</link>
+	<joint name="head_camera_joint" type="fixed">
+		<origin xyz="-0.097847  0.046703 -0.12364" rpy="0 -0.64460396 ${PI}"/>
+		<parent link="head_link2"/>
+		<child link="head_camera"/>
+	</joint>
 	<link name="arm_base"/>
 	<joint name="arm_base_joint" type="fixed">

Commit message: add gripper config

File: urdf/fiveages_w2.urdf (robot description, URDF)
Before this commit: robot FiveAges W2, 42 links, 41 joints
Links:
- added link left_tcp
- added link right_tcp
- link body_camera: geometry visual mesh filename=package://sensor_models/meshes/orbbec/336.obj
- link body_link4: geometry collision box size=0.2000 0.32 0.5029; visual mesh filename=package://fiveages_w2_description/meshes/body/link4.obj
- link head_camera: geometry visual mesh filename=package://sensor_models/meshes/orbbec/336L.obj
Joints:
- added joint left_tcp_joint: type fixed, parent left_link7, child left_tcp, origin xyz=0 -0.095296 0 rpy=0 0 0
- added joint right_tcp_joint: type fixed, parent right_link7, child right_tcp, origin xyz=0 -0.095296 0 rpy=0 0 0
- joint head_joint1: limit lower=-3.14 upper=3.14 effort=100 velocity=1 -> lower=-0.436 upper=0.436 effort=100 velocity=1
- joint head_joint2: limit lower=-3.14 upper=3.14 effort=100 velocity=1 -> lower=-0.26 upper=0.26 effort=100 velocity=1
- joint left_eef_joint: origin xyz=0 -0.095296 0 rpy=0 0 0 -> rpy=1.5707963267948966 0 0; parent left_link7 -> left_tcp
- joint right_eef_joint: origin xyz=0 -0.095296 0 rpy=0 0 0 -> rpy=1.5707963267948966 0 0; parent right_link7 -> right_tcp

File: xacro/body.xacro (robot description, xacro)
@@ -137,6 +137,7 @@
 		</visual>
 		<collision>
-			<geometry>
-				<mesh filename="file://$(find fiveages_w2_description)/meshes/body/link4.obj"/>
+			<origin xyz="0.0091 0 0.25765"/>
+			<geometry>
+				<box size="0.2000 0.32 0.5029"/>
 			</geometry>
 		</collision>
@@ -150,9 +151,9 @@
 	</joint>
 	<link name="body_camera">
-<!--		<visual>-->
-<!--			<geometry>-->
-<!--				<mesh filename="file://$(find sensor_models)/meshes/orbbec/336.obj"/>-->
-<!--			</geometry>-->
-<!--		</visual>-->
+		<visual>
+			<geometry>
+				<mesh filename="file://$(find sensor_models)/meshes/orbbec/336.obj"/>
+			</geometry>
+		</visual>
 	</link>
 	<joint name="body_camera_joint" type="fixed">
@@ -189,5 +190,5 @@
 		<child link="head_link1"/>
 		<axis xyz="0 0 1"/>
-		<limit lower="-3.14" upper="3.14" effort="100" velocity="1"/>
+		<limit lower="-0.436" upper="0.436" effort="100" velocity="1"/>
 	</joint>
 	<link name="head_link2">
@@ -219,12 +220,12 @@
 		<child link="head_link2"/>
 		<axis xyz="0 -1 0"/>
-		<limit lower="-3.14" upper="3.14" effort="100" velocity="1"/>
+		<limit lower="-0.26" upper="0.26" effort="100" velocity="1"/>
 	</joint>
 	<link name="head_camera">
-<!--		<visual>-->
-<!--			<geometry>-->
-<!--				<mesh filename="file://$(find sensor_models)/meshes/orbbec/336L.obj"/>-->
-<!--			</geometry>-->
-<!--		</visual>-->
+		<visual>
+			<geometry>
+				<mesh filename="file://$(find sensor_models)/meshes/orbbec/336L.obj"/>
+			</geometry>
+		</visual>
 	</link>
 	<joint name="head_camera_joint" type="fixed">

File: xacro/grippers.xacro (robot description, xacro)
@@ -3,4 +3,18 @@
     <xacro:macro name="Grippers" params="type:=''">
         <!-- Note: type parameter is now passed as macro parameter -->
+        <xacro:if value="${type == ''}">
+            <link name="left_eef"/>
+            <link name="right_eef"/>
+            <joint name="left_eef_joint" type="fixed">
+                <parent link="left_tcp"/>
+                <child link="left_eef"/>
+                <origin rpy=" ${PI/2} 0 0"/>
+            </joint>
+            <joint name="right_eef_joint" type="fixed">
+                <parent link="right_tcp"/>
+                <child link="right_eef"/>
+                <origin rpy=" ${PI/2} 0 0"/>
+            </joint>
+        </xacro:if>
         <xacro:if value="${type == 'ag2f90'}">
             <xacro:include filename="$(find changingtek_description)/xacro/AG2F90-C.xacro"/>
