Commit message: fix m6 ccs urdf param

File: urdf/fiveages_w2.urdf (robot description, URDF)
Before this commit: robot FiveAges W2, 44 links, 43 joints
Joints:
- joint left_eef_joint: origin rpy=1.5707963267948966 0 0 -> (none)
- joint left_tcp_joint: origin xyz=0 -0.095296 0 rpy=0 0 0 -> xyz=0 -0.095 0 rpy=1.5707963267948966 -1.5707963267948966 0
- joint right_eef_joint: origin rpy=1.5707963267948966 0 0 -> (none)
- joint right_tcp_joint: origin xyz=0 -0.095296 0 rpy=0 0 0 -> xyz=0 -0.095 0 rpy=1.5707963267948966 -1.5707963267948966 0

File: urdf/fiveages_w2_ag2f90.urdf (robot description, URDF)
Before this commit: robot FiveAges W2, 68 links, 67 joints
Joints:
- joint left_gripper_fix: origin xyz=0 -0.0995 0 rpy= 1.5707963267948966 0 0 -> xyz=0 0 0.0045; parent left_link7 -> left_tcp
- joint left_tcp_joint: origin xyz=0 -0.095296 0 rpy=0 0 0 -> xyz=0 -0.095 0 rpy=1.5707963267948966 -1.5707963267948966 0
- joint right_gripper_fix: origin xyz=0 -0.0995 0 rpy= 1.5707963267948966 0 0 -> xyz=0 0 0.0045; parent right_link7 -> right_tcp
- joint right_tcp_joint: origin xyz=0 -0.095296 0 rpy=0 0 0 -> xyz=0 -0.095 0 rpy=1.5707963267948966 -1.5707963267948966 0

File: urdf/fiveages_w2_rg75.urdf (robot description, URDF)
Before this commit: robot FiveAges W2, 56 links, 55 joints
Links:
- link body_camera: geometry visual mesh filename=package://sensor_models/meshes/orbbec/336.obj
- link head_camera: geometry visual mesh filename=package://sensor_models/meshes/orbbec/336L.obj
- link left_flange: geometry collision mesh filename=file:///home/fa/ros2_ws/install/jodell_description/share/jo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; visual mesh filename=file:///home/fa/ros2_ws/install/jodell_description/share/jo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
- link left_gripper_base: geometry collision mesh filename=file:///home/fa/ros2_ws/install/jodell_description/share/jo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; visual mesh filename=file:///home/fa/ros2_ws/install/jodell_description/share/jo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
- link left_left_finger: geometry collision mesh filename=file:///home/fa/ros2_ws/install/jodell_description/share/jo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; visual mesh filename=file:///home/fa/ros2_ws/install/jodell_description/share/jo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
- link left_left_finger_pad: geometry collision mesh filename=file:///home/fa/ros2_ws/install/jodell_description/share/jo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; visual mesh filename=file:///home/fa/ros2_ws/install/jodell_description/share/jo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
- link left_right_finger: geometry collision mesh filename=file:///home/fa/ros2_ws/install/jodell_description/share/jo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 scale=-1 -1 1; visual mesh filename=file:///home/fa/ros2_ws/install/jodell_description/share/jo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 scale=-1 -1 1
- link left_right_finger_pad: geometry collision mesh filename=file:///home/fa/ros2_ws/install/jodell_description/share/jo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 scale=1 -1 1; visual mesh filename=file:///home/fa/ros2_ws/install/jodell_description/share/jo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 scale=1 -1 1
- link right_flange: geometry collision mesh filename=file:///home/fa/ros2_ws/install/jodell_description/share/jo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; visual mesh filename=file:///home/fa/ros2_ws/install/jodell_description/share/jo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
- link right_gripper_base: geometry collision mesh filename=file:///home/fa/ros2_ws/install/jodell_description/share/jo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; visual mesh filename=file:///home/fa/ros2_ws/install/jodell_description/share/jo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
- link right_left_finger: geometry collision mesh filename=file:///home/fa/ros2_ws/install/jodell_description/share/jo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; visual mesh filename=file:///home/fa/ros2_ws/install/jodell_description/share/jo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
- link right_left_finger_pad: geometry collision mesh filename=file:///home/fa/ros2_ws/install/jodell_description/share/jo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; visual mesh filename=file:///home/fa/ros2_ws/install/jodell_description/share/jo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
- link right_right_finger: geometry collision mesh filename=file:///home/fa/ros2_ws/install/jodell_description/share/jo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 scale=-1 -1 1; visual mesh filename=file:///home/fa/ros2_ws/install/jodell_description/share/jo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 scale=-1 -1 1
- link right_right_finger_pad: geometry collision mesh filename=file:///home/fa/ros2_ws/install/jodell_description/share/jo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 scale=1 -1 1; visual mesh filename=file:///home/fa/ros2_ws/install/jodell_description/share/jo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 scale=1 -1 1
Joints:
- joint left_gripper_base_joint: origin rpy=-1.5707963267948966 0 3.141592653589793 -> (none)
- joint left_tcp_joint: origin xyz=0 -0.095296 0 rpy=0 0 0 -> xyz=0 -0.095 0 rpy=1.5707963267948966 -1.5707963267948966 0
- joint right_gripper_base_joint: origin rpy=1.5707963267948966 0 0 -> (none)
- joint right_tcp_joint: origin xyz=0 -0.095296 0 rpy=0 0 0 -> xyz=0 -0.095 0 rpy=1.5707963267948966 -1.5707963267948966 0

File: xacro/grippers.xacro (robot description, xacro)
@@ -9,10 +9,8 @@
                 <parent link="left_tcp"/>
                 <child link="left_eef"/>
-                <origin rpy=" ${PI/2} 0 0"/>
             </joint>
             <joint name="right_eef_joint" type="fixed">
                 <parent link="right_tcp"/>
                 <child link="right_eef"/>
-                <origin rpy=" ${PI/2} 0 0"/>
             </joint>
         </xacro:if>
@@ -21,13 +19,13 @@
             <xacro:AG2F90-C name="left" use_flange="true"/>
             <joint name="left_gripper_fix" type="fixed">
-                <parent link="left_link7"/>
+                <parent link="left_tcp"/>
                 <child link="left_flange"/>
-                <origin xyz="0 -0.0995 0" rpy=" ${PI/2} 0 0"/>
+                <origin xyz="0 0 0.0045"/>
             </joint>
             <xacro:AG2F90-C name="right" use_flange="true"/>
             <joint name="right_gripper_fix" type="fixed">
-                <parent link="right_link7"/>
+                <parent link="right_tcp"/>
                 <child link="right_flange"/>
-                <origin xyz="0 -0.0995 0" rpy=" ${PI/2} 0 0"/>
+                <origin xyz="0 0 0.0045"/>
             </joint>
         </xacro:if>
@@ -37,10 +35,8 @@
             <xacro:RG75-300 name="right" use_flange="true"/>
             <joint name="left_gripper_base_joint" type="fixed">
-                <origin rpy="${-PI/2} 0 ${PI}"/>
                 <parent link="left_tcp"/>
                 <child link="left_flange"/>
             </joint>
             <joint name="right_gripper_base_joint" type="fixed">
-                <origin rpy="${PI/2} 0 0"/>
                 <parent link="right_tcp"/>
                 <child link="right_flange"/>

File: xacro/ros2_control/body.xacro (robot description, xacro)
@@ -7,5 +7,5 @@
       <state_interface name="position"/>
       <state_interface name="velocity"/>
-      <!-- <state_interface name="effort"/> -->
+       <state_interface name="effort"/>
     </joint>
     <joint name="body_joint2">
@@ -13,5 +13,5 @@
       <state_interface name="position"/>
       <state_interface name="velocity"/>
-      <!-- <state_interface name="effort"/> -->
+       <state_interface name="effort"/>
     </joint>
     <joint name="body_joint3">
@@ -19,5 +19,5 @@
       <state_interface name="position"/>
       <state_interface name="velocity"/>
-      <!-- <state_interface name="effort"/> -->
+       <state_interface name="effort"/>
     </joint>
     <joint name="body_joint4">
@@ -25,5 +25,5 @@
       <state_interface name="position"/>
       <state_interface name="velocity"/>
-      <!-- <state_interface name="effort"/> -->
+       <state_interface name="effort"/>
     </joint>
     <joint name="head_joint1">

File: xacro/ros2_control/robot.xacro (robot description, xacro)
@@ -5,5 +5,4 @@
 	<xacro:include filename="$(find m6_ccs_description)/xacro/ros2_control/interfaces.xacro"/>
 	<xacro:include filename="$(find fiveages_w2_description)/xacro/ros2_control/body.xacro"/>
-	<!-- <xacro:include filename="$(find fiveages_w2_description)/xacro/ros2_control/chassis.xacro"/> -->
 	<xacro:if value="${'$(arg ros2_control_hardware_type)' == 'real'}">
 		<ros2_control name="M6_CCS_System" type="system">

Commit message: fix head joint

File: urdf/fiveages_w2.urdf (robot description, URDF)
Before this commit: robot FiveAges W2, 44 links, 43 joints
Joints:
- joint head_camera_joint: origin xyz=-0.097847  0.046703 -0.12364 rpy=0 -0.64460396 3.141592653589793 -> xyz=0.097847  0.046703 0.12364 rpy=3.141592653589793 0.64460396 0
- joint head_joint2: origin xyz=0 0.0042 0.15 rpy=3.141592653589793 0 3.141592653589793 -> xyz=0 0.0042 0.15

File: urdf/fiveages_w2_ag2f90.urdf (robot description, URDF)
Before this commit: robot FiveAges W2, 68 links, 67 joints
Joints:
- joint head_camera_joint: origin xyz=-0.097847  0.046703 -0.12364 rpy=0 -0.64460396 3.141592653589793 -> xyz=0.097847  0.046703 0.12364 rpy=3.141592653589793 0.64460396 0
- joint head_joint2: origin xyz=0 0.0042 0.15 rpy=3.141592653589793 0 3.141592653589793 -> xyz=0 0.0042 0.15

File: urdf/fiveages_w2_rg75.urdf (robot description, URDF)
Before this commit: robot FiveAges W2, 56 links, 55 joints
Joints:
- joint head_camera_joint: origin xyz=-0.097847  0.046703 -0.12364 rpy=0 -0.64460396 3.141592653589793 -> xyz=0.097847  0.046703 0.12364 rpy=3.141592653589793 0.64460396 0
- joint head_joint2: origin xyz=0 0.0042 0.15 rpy=3.141592653589793 0 3.141592653589793 -> xyz=0 0.0042 0.15

Commit message: update joint limits

File: urdf/fiveages_w2.urdf (robot description, URDF)
Before this commit: robot FiveAges W2, 44 links, 43 joints
Links:
- added link head_top_camera
- link left_link1: geometry collision cylinder length=0.125958 radius=0.057588; visual mesh filename=package://fiveages_w2_description/meshes/arm/link1.obj
- link left_link2: geometry collision cylinder length=0.078386 radius=0.046717; visual mesh filename=package://fiveages_w2_description/meshes/arm/link2.obj scale=1 1 1
- link left_link3: geometry collision cylinder length=0.089056 radius=0.046717; collision cylinder length=0.117016 radius=0.049964
- link left_link4: geometry collision cylinder length=0.080203 radius=0.041759; visual mesh filename=package://fiveages_w2_description/meshes/arm/link4.obj
- link left_link5: geometry collision cylinder length=0.14268 radius=0.056747; visual mesh filename=package://fiveages_w2_description/meshes/arm/link5.obj scale=1 1 1
- link right_link1: geometry collision cylinder length=0.125958 radius=0.057588; visual mesh filename=package://fiveages_w2_description/meshes/arm/link1.obj
- link right_link2: geometry collision cylinder length=0.078386 radius=0.046717; visual mesh filename=package://fiveages_w2_description/meshes/arm/link2.obj scale=1 1 -1
- link right_link3: geometry collision cylinder length=0.089056 radius=0.046717; collision cylinder length=0.117016 radius=0.049964
- link right_link4: geometry collision cylinder length=0.080203 radius=0.041759; visual mesh filename=package://fiveages_w2_description/meshes/arm/link4.obj
- link right_link5: geometry collision cylinder length=0.14268 radius=0.056747; visual mesh filename=package://fiveages_w2_description/meshes/arm/link5.obj scale=1 -1 1
Joints:
- added joint head_top_camera_joint: type fixed, parent head_link2, child head_top_camera, origin xyz=0.0877736 0.0245687 0.107989 rpy=-2.100227811211368 0.0016038446958035316 -1.583610269343787
- joint body_joint1: limit lower=-1.352633 upper=0.567 effort=100 velocity=1 -> lower=-1.2217304763960306 upper=0.5235987755982988 effort=100 velocity=1
- joint body_joint2: limit lower=-2.66 upper=1.605 effort=100 velocity=1 -> lower=-2.0943951023931953 upper=1.5707963267948966 effort=100 velocity=1
- joint body_joint3: limit lower=-1.745 upper=1.745 effort=100 velocity=1 -> lower=-0.8726646259971648 upper=1.2217304763960306 effort=100 velocity=1
- joint head_joint1: limit lower=-0.436 upper=0.436 effort=100 velocity=1 -> lower=-0.4363323129985824 upper=0.4363323129985824 effort=100 velocity=1
- joint head_joint2: limit lower=-0.26 upper=0.26 effort=100 velocity=1 -> lower=-0.2617993877991494 upper=0.2617993877991494 effort=100 velocity=1; origin xyz=0 0.0042 0.15 -> xyz=0 0.0 0.15

File: urdf/fiveages_w2_ag2f90.urdf (robot description, URDF)
Before this commit: robot FiveAges W2, 68 links, 67 joints
Links:
- added link head_top_camera
- link left_link1: geometry collision cylinder length=0.125958 radius=0.057588; visual mesh filename=package://fiveages_w2_description/meshes/arm/link1.obj
- link left_link2: geometry collision cylinder length=0.078386 radius=0.046717; visual mesh filename=package://fiveages_w2_description/meshes/arm/link2.obj scale=1 1 1
- link left_link3: geometry collision cylinder length=0.089056 radius=0.046717; collision cylinder length=0.117016 radius=0.049964
- link left_link4: geometry collision cylinder length=0.080203 radius=0.041759; visual mesh filename=package://fiveages_w2_description/meshes/arm/link4.obj
- link left_link5: geometry collision cylinder length=0.14268 radius=0.056747; visual mesh filename=package://fiveages_w2_description/meshes/arm/link5.obj scale=1 1 1
- link right_link1: geometry collision cylinder length=0.125958 radius=0.057588; visual mesh filename=package://fiveages_w2_description/meshes/arm/link1.obj
- link right_link2: geometry collision cylinder length=0.078386 radius=0.046717; visual mesh filename=package://fiveages_w2_description/meshes/arm/link2.obj scale=1 1 -1
- link right_link3: geometry collision cylinder length=0.089056 radius=0.046717; collision cylinder length=0.117016 radius=0.049964
- link right_link4: geometry collision cylinder length=0.080203 radius=0.041759; visual mesh filename=package://fiveages_w2_description/meshes/arm/link4.obj
- link right_link5: geometry collision cylinder length=0.14268 radius=0.056747; visual mesh filename=package://fiveages_w2_description/meshes/arm/link5.obj scale=1 -1 1
Joints:
- added joint head_top_camera_joint: type fixed, parent head_link2, child head_top_camera, origin xyz=0.0877736 0.0245687 0.107989 rpy=-2.100227811211368 0.0016038446958035316 -1.583610269343787
- joint body_joint1: limit lower=-1.352633 upper=0.567 effort=100 velocity=1 -> lower=-1.2217304763960306 upper=0.5235987755982988 effort=100 velocity=1
- joint body_joint2: limit lower=-2.66 upper=1.605 effort=100 velocity=1 -> lower=-2.0943951023931953 upper=1.5707963267948966 effort=100 velocity=1
- joint body_joint3: limit lower=-1.745 upper=1.745 effort=100 velocity=1 -> lower=-0.8726646259971648 upper=1.2217304763960306 effort=100 velocity=1
- joint head_joint1: limit lower=-0.436 upper=0.436 effort=100 velocity=1 -> lower=-0.4363323129985824 upper=0.4363323129985824 effort=100 velocity=1
- joint head_joint2: limit lower=-0.26 upper=0.26 effort=100 velocity=1 -> lower=-0.2617993877991494 upper=0.2617993877991494 effort=100 velocity=1; origin xyz=0 0.0042 0.15 -> xyz=0 0.0 0.15

File: urdf/fiveages_w2_rg75.urdf (robot description, URDF)
Before this commit: robot FiveAges W2, 56 links, 55 joints
Links:
- added link head_top_camera
- link left_flange: geometry collision mesh filename=package://jodell_description/meshes/RG75/flange.obj; visual mesh filename=package://jodell_description/meshes/RG75/flange.obj
- link left_gripper_base: geometry collision mesh filename=package://jodell_description/meshes/RG75/base.obj; visual mesh filename=package://jodell_description/meshes/RG75/base.obj
- link left_left_finger: geometry collision mesh filename=package://jodell_description/meshes/RG75/finger.obj; visual mesh filename=package://jodell_description/meshes/RG75/finger.obj
- link left_left_finger_pad: geometry collision mesh filename=package://jodell_description/meshes/RG75/pad_fiveages.obj; visual mesh filename=package://jodell_description/meshes/RG75/pad_fiveages.obj
- link left_link1: geometry collision cylinder length=0.125958 radius=0.057588; visual mesh filename=package://fiveages_w2_description/meshes/arm/link1.obj
- link left_link2: geometry collision cylinder length=0.078386 radius=0.046717; visual mesh filename=package://fiveages_w2_description/meshes/arm/link2.obj scale=1 1 1
- link left_link3: geometry collision cylinder length=0.089056 radius=0.046717; collision cylinder length=0.117016 radius=0.049964
- link left_link4: geometry collision cylinder length=0.080203 radius=0.041759; visual mesh filename=package://fiveages_w2_description/meshes/arm/link4.obj
- link left_link5: geometry collision cylinder length=0.14268 radius=0.056747; visual mesh filename=package://fiveages_w2_description/meshes/arm/link5.obj scale=1 1 1
- link left_right_finger: geometry collision mesh filename=package://jodell_description/meshes/RG75/finger.obj scale=-1 -1 1; visual mesh filename=package://jodell_description/meshes/RG75/finger.obj scale=-1 -1 1
- link left_right_finger_pad: geometry collision mesh filename=package://jodell_description/meshes/RG75/pad_fiveages.obj scale=1 -1 1; visual mesh filename=package://jodell_description/meshes/RG75/pad_fiveages.obj scale=1 -1 1
- link right_flange: geometry collision mesh filename=package://jodell_description/meshes/RG75/flange.obj; visual mesh filename=package://jodell_description/meshes/RG75/flange.obj
- link right_gripper_base: geometry collision mesh filename=package://jodell_description/meshes/RG75/base.obj; visual mesh filename=package://jodell_description/meshes/RG75/base.obj
- link right_left_finger: geometry collision mesh filename=package://jodell_description/meshes/RG75/finger.obj; visual mesh filename=package://jodell_description/meshes/RG75/finger.obj
- link right_left_finger_pad: geometry collision mesh filename=package://jodell_description/meshes/RG75/pad_fiveages.obj; visual mesh filename=package://jodell_description/meshes/RG75/pad_fiveages.obj
- link right_link1: geometry collision cylinder length=0.125958 radius=0.057588; visual mesh filename=package://fiveages_w2_description/meshes/arm/link1.obj
- link right_link2: geometry collision cylinder length=0.078386 radius=0.046717; visual mesh filename=package://fiveages_w2_description/meshes/arm/link2.obj scale=1 1 -1
- link right_link3: geometry collision cylinder length=0.089056 radius=0.046717; collision cylinder length=0.117016 radius=0.049964
- link right_link4: geometry collision cylinder length=0.080203 radius=0.041759; visual mesh filename=package://fiveages_w2_description/meshes/arm/link4.obj
- link right_link5: geometry collision cylinder length=0.14268 radius=0.056747; visual mesh filename=package://fiveages_w2_description/meshes/arm/link5.obj scale=1 -1 1
- link right_right_finger: geometry collision mesh filename=package://jodell_description/meshes/RG75/finger.obj scale=-1 -1 1; visual mesh filename=package://jodell_description/meshes/RG75/finger.obj scale=-1 -1 1
- link right_right_finger_pad: geometry collision mesh filename=package://jodell_description/meshes/RG75/pad_fiveages.obj scale=1 -1 1; visual mesh filename=package://jodell_description/meshes/RG75/pad_fiveages.obj scale=1 -1 1
Joints:
- added joint head_top_camera_joint: type fixed, parent head_link2, child head_top_camera, origin xyz=0.0877736 0.0245687 0.107989 rpy=-2.100227811211368 0.0016038446958035316 -1.583610269343787
- joint body_joint1: limit lower=-1.352633 upper=0.567 effort=100 velocity=1 -> lower=-1.2217304763960306 upper=0.5235987755982988 effort=100 velocity=1
- joint body_joint2: limit lower=-2.66 upper=1.605 effort=100 velocity=1 -> lower=-2.0943951023931953 upper=1.5707963267948966 effort=100 velocity=1
- joint body_joint3: limit lower=-1.745 upper=1.745 effort=100 velocity=1 -> lower=-0.8726646259971648 upper=1.2217304763960306 effort=100 velocity=1
- joint head_joint1: limit lower=-0.436 upper=0.436 effort=100 velocity=1 -> lower=-0.4363323129985824 upper=0.4363323129985824 effort=100 velocity=1
- joint head_joint2: limit lower=-0.26 upper=0.26 effort=100 velocity=1 -> lower=-0.2617993877991494 upper=0.2617993877991494 effort=100 velocity=1; origin xyz=0 0.0042 0.15 -> xyz=0 0.0 0.15

File: xacro/body.xacro (robot description, xacro)
@@ -57,5 +57,5 @@
 		<child link="body_link1"/>
 		<axis xyz="0 1 0"/>
-		<limit lower="-1.352633" upper="0.567" effort="100" velocity="1"/>
+		<limit lower="-${PI*70/180}" upper="${PI*30/180}" effort="100" velocity="1"/>
 	</joint>
 	<link name="body_link2">
@@ -87,5 +87,5 @@
 		<child link="body_link2"/>
 		<axis xyz="0 -1 0"/>
-		<limit lower="-2.66" upper="1.605" effort="100" velocity="1"/>
+		<limit lower="-${PI*120/180}" upper="${PI*90/180}" effort="100" velocity="1"/>
 	</joint>
 	<link name="body_link3">
@@ -117,5 +117,5 @@
 		<child link="body_link3"/>
 		<axis xyz="0 1 0"/>
-		<limit lower="-1.745" upper="1.745" effort="100" velocity="1"/>
+		<limit lower="-${PI*50/180}" upper="${PI*70/180}" effort="100" velocity="1"/>
 	</joint>
 	<link name="body_link4">
@@ -190,5 +190,5 @@
 		<child link="head_link1"/>
 		<axis xyz="0 0 1"/>
-		<limit lower="-0.436" upper="0.436" effort="100" velocity="1"/>
+		<limit lower="-${PI*25/180}" upper="${PI*25/180}" effort="100" velocity="1"/>
 	</joint>
 	<link name="head_link2">
@@ -220,5 +220,5 @@
 		<child link="head_link2"/>
 		<axis xyz="0 1 0"/>
-		<limit lower="-0.26" upper="0.26" effort="100" velocity="1"/>
+		<limit lower="-${PI*15/180}" upper="${PI*15/180}" effort="100" velocity="1"/>
 	</joint>
 	<link name="head_camera">

File: xacro/grippers.xacro (robot description, xacro)
@@ -32,6 +32,6 @@
         <xacro:if value="${type == 'rg75'}">
             <xacro:include filename="$(find jodell_description)/xacro/RG75-300.xacro"/>
-            <xacro:RG75-300 name="left" use_flange="true" pad="leapmotor"/>
-            <xacro:RG75-300 name="right" use_flange="true" pad="leapmotor"/>
+            <xacro:RG75-300 name="left" use_flange="true"/>
+            <xacro:RG75-300 name="right" use_flange="true"/>
             <joint name="left_gripper_base_joint" type="fixed">
                 <parent link="left_tcp"/>
