Commit message: update joint limit

File: urdf/fiveages_w2.urdf (robot description, URDF)
Before this commit: robot FiveAges W2, 44 links, 43 joints
Joints:
- joint left_joint1: limit lower=-3.1067 upper=3.1067 effort=108 velocity=3.141592653589793 -> lower=-3.106686068549907 upper=3.106686068549907 effort=108 velocity=3.141592653589793
- joint left_joint2: limit lower=-2.0944 upper=2.0944 effort=108 velocity=3.141592653589793 -> lower=-2.0594885173533086 upper=2.0594885173533086 effort=108 velocity=3.141592653589793
- joint left_joint3: limit lower=-3.1067 upper=3.1067 effort=66 velocity=3.141592653589793 -> lower=-2.9321531433504737 upper=2.9321531433504737 effort=66 velocity=3.141592653589793
- joint left_joint4: limit lower=-2.5307 upper=1.0472 effort=66 velocity=3.141592653589793 -> lower=-2.4958208303518914 upper=1.0122909661567112 effort=66 velocity=3.141592653589793
- joint left_joint5: limit lower=-3.1067 upper=3.1067 effort=18 velocity=3.141592653589793 -> lower=-2.9321531433504737 upper=2.9321531433504737 effort=18 velocity=3.141592653589793
- joint left_joint6: limit lower=-1.0472 upper=1.0472 effort=18 velocity=3.141592653589793 -> lower=-1.0122909661567112 upper=1.0122909661567112 effort=18 velocity=3.141592653589793
- joint left_joint7: limit lower=-1.5707963267948966 upper=1.5707963267948966 effort=18 velocity=3.141592653589793 -> lower=-1.361356816555577 upper=1.361356816555577 effort=18 velocity=3.141592653589793
- joint right_joint1: limit lower=-3.1067 upper=3.1067 effort=108 velocity=3.141592653589793 -> lower=-3.106686068549907 upper=3.106686068549907 effort=108 velocity=3.141592653589793
- joint right_joint2: limit lower=-2.0944 upper=2.0944 effort=108 velocity=3.141592653589793 -> lower=-2.0594885173533086 upper=2.0594885173533086 effort=108 velocity=3.141592653589793
- joint right_joint3: limit lower=-3.1067 upper=3.1067 effort=66 velocity=3.141592653589793 -> lower=-2.9321531433504737 upper=2.9321531433504737 effort=66 velocity=3.141592653589793
- joint right_joint4: limit lower=-2.5307 upper=1.0472 effort=66 velocity=3.141592653589793 -> lower=-2.4958208303518914 upper=1.0122909661567112 effort=66 velocity=3.141592653589793
- joint right_joint5: limit lower=-3.1067 upper=3.1067 effort=18 velocity=3.141592653589793 -> lower=-2.9321531433504737 upper=2.9321531433504737 effort=18 velocity=3.141592653589793
- joint right_joint6: limit lower=-1.0472 upper=1.0472 effort=18 velocity=3.141592653589793 -> lower=-1.0122909661567112 upper=1.0122909661567112 effort=18 velocity=3.141592653589793
- joint right_joint7: limit lower=-1.5707963267948966 upper=1.5707963267948966 effort=18 velocity=3.141592653589793 -> lower=-1.361356816555577 upper=1.361356816555577 effort=18 velocity=3.141592653589793

File: urdf/fiveages_w2_ag2f90.urdf (robot description, URDF)
Before this commit: robot FiveAges W2, 68 links, 67 joints
Joints:
- joint left_joint1: limit lower=-3.1067 upper=3.1067 effort=108 velocity=3.141592653589793 -> lower=-3.106686068549907 upper=3.106686068549907 effort=108 velocity=3.141592653589793
- joint left_joint2: limit lower=-2.0944 upper=2.0944 effort=108 velocity=3.141592653589793 -> lower=-2.0594885173533086 upper=2.0594885173533086 effort=108 velocity=3.141592653589793
- joint left_joint3: limit lower=-3.1067 upper=3.1067 effort=66 velocity=3.141592653589793 -> lower=-2.9321531433504737 upper=2.9321531433504737 effort=66 velocity=3.141592653589793
- joint left_joint4: limit lower=-2.5307 upper=1.0472 effort=66 velocity=3.141592653589793 -> lower=-2.4958208303518914 upper=1.0122909661567112 effort=66 velocity=3.141592653589793
- joint left_joint5: limit lower=-3.1067 upper=3.1067 effort=18 velocity=3.141592653589793 -> lower=-2.9321531433504737 upper=2.9321531433504737 effort=18 velocity=3.141592653589793
- joint left_joint6: limit lower=-1.0472 upper=1.0472 effort=18 velocity=3.141592653589793 -> lower=-1.0122909661567112 upper=1.0122909661567112 effort=18 velocity=3.141592653589793
- joint left_joint7: limit lower=-1.5707963267948966 upper=1.5707963267948966 effort=18 velocity=3.141592653589793 -> lower=-1.361356816555577 upper=1.361356816555577 effort=18 velocity=3.141592653589793
- joint right_joint1: limit lower=-3.1067 upper=3.1067 effort=108 velocity=3.141592653589793 -> lower=-3.106686068549907 upper=3.106686068549907 effort=108 velocity=3.141592653589793
- joint right_joint2: limit lower=-2.0944 upper=2.0944 effort=108 velocity=3.141592653589793 -> lower=-2.0594885173533086 upper=2.0594885173533086 effort=108 velocity=3.141592653589793
- joint right_joint3: limit lower=-3.1067 upper=3.1067 effort=66 velocity=3.141592653589793 -> lower=-2.9321531433504737 upper=2.9321531433504737 effort=66 velocity=3.141592653589793
- joint right_joint4: limit lower=-2.5307 upper=1.0472 effort=66 velocity=3.141592653589793 -> lower=-2.4958208303518914 upper=1.0122909661567112 effort=66 velocity=3.141592653589793
- joint right_joint5: limit lower=-3.1067 upper=3.1067 effort=18 velocity=3.141592653589793 -> lower=-2.9321531433504737 upper=2.9321531433504737 effort=18 velocity=3.141592653589793
- joint right_joint6: limit lower=-1.0472 upper=1.0472 effort=18 velocity=3.141592653589793 -> lower=-1.0122909661567112 upper=1.0122909661567112 effort=18 velocity=3.141592653589793
- joint right_joint7: limit lower=-1.5707963267948966 upper=1.5707963267948966 effort=18 velocity=3.141592653589793 -> lower=-1.361356816555577 upper=1.361356816555577 effort=18 velocity=3.141592653589793

File: urdf/fiveages_w2_rg75.urdf (robot description, URDF)
Before this commit: robot FiveAges W2, 56 links, 55 joints
Joints:
- joint left_joint1: limit lower=-3.1067 upper=3.1067 effort=108 velocity=3.141592653589793 -> lower=-3.106686068549907 upper=3.106686068549907 effort=108 velocity=3.141592653589793
- joint left_joint2: limit lower=-2.0944 upper=2.0944 effort=108 velocity=3.141592653589793 -> lower=-2.0594885173533086 upper=2.0594885173533086 effort=108 velocity=3.141592653589793
- joint left_joint3: limit lower=-3.1067 upper=3.1067 effort=66 velocity=3.141592653589793 -> lower=-2.9321531433504737 upper=2.9321531433504737 effort=66 velocity=3.141592653589793
- joint left_joint4: limit lower=-2.5307 upper=1.0472 effort=66 velocity=3.141592653589793 -> lower=-2.4958208303518914 upper=1.0122909661567112 effort=66 velocity=3.141592653589793
- joint left_joint5: limit lower=-3.1067 upper=3.1067 effort=18 velocity=3.141592653589793 -> lower=-2.9321531433504737 upper=2.9321531433504737 effort=18 velocity=3.141592653589793
- joint left_joint6: limit lower=-1.0472 upper=1.0472 effort=18 velocity=3.141592653589793 -> lower=-1.0122909661567112 upper=1.0122909661567112 effort=18 velocity=3.141592653589793
- joint left_joint7: limit lower=-1.5707963267948966 upper=1.5707963267948966 effort=18 velocity=3.141592653589793 -> lower=-1.361356816555577 upper=1.361356816555577 effort=18 velocity=3.141592653589793
- joint right_joint1: limit lower=-3.1067 upper=3.1067 effort=108 velocity=3.141592653589793 -> lower=-3.106686068549907 upper=3.106686068549907 effort=108 velocity=3.141592653589793
- joint right_joint2: limit lower=-2.0944 upper=2.0944 effort=108 velocity=3.141592653589793 -> lower=-2.0594885173533086 upper=2.0594885173533086 effort=108 velocity=3.141592653589793
- joint right_joint3: limit lower=-3.1067 upper=3.1067 effort=66 velocity=3.141592653589793 -> lower=-2.9321531433504737 upper=2.9321531433504737 effort=66 velocity=3.141592653589793
- joint right_joint4: limit lower=-2.5307 upper=1.0472 effort=66 velocity=3.141592653589793 -> lower=-2.4958208303518914 upper=1.0122909661567112 effort=66 velocity=3.141592653589793
- joint right_joint5: limit lower=-3.1067 upper=3.1067 effort=18 velocity=3.141592653589793 -> lower=-2.9321531433504737 upper=2.9321531433504737 effort=18 velocity=3.141592653589793
- joint right_joint6: limit lower=-1.0472 upper=1.0472 effort=18 velocity=3.141592653589793 -> lower=-1.0122909661567112 upper=1.0122909661567112 effort=18 velocity=3.141592653589793
- joint right_joint7: limit lower=-1.5707963267948966 upper=1.5707963267948966 effort=18 velocity=3.141592653589793 -> lower=-1.361356816555577 upper=1.361356816555577 effort=18 velocity=3.141592653589793

File: xacro/components/arm.xacro (robot description, xacro)
@@ -70,5 +70,5 @@
 			<child link="${prefix}link1"/>
 			<axis xyz="0 0 1"/>
-			<limit lower="-3.1067" upper="3.1067" effort="108" velocity="${PI}"/>
+			<limit lower="-${PI*178/180}" upper="${PI*178/180}" effort="108" velocity="${PI}"/>
 		</joint>
 		<!-- Link 2 -->
@@ -108,5 +108,5 @@
 			<child link="${prefix}link2"/>
 			<axis xyz="0 0 1"/>
-			<limit lower="-2.0944" upper="2.0944" effort="108" velocity="${PI}"/>
+			<limit lower="-${PI*118/180}" upper="${PI*118/180}" effort="108" velocity="${PI}"/>
 		</joint>
 		<!-- Link 3 -->
@@ -152,5 +152,5 @@
 			<child link="${prefix}link3"/>
 			<axis xyz="0 0 1"/>
-			<limit lower="-3.1067" upper="3.1067" effort="66" velocity="${PI}"/>
+			<limit lower="-${PI*168/180}" upper="${PI*168/180}" effort="66" velocity="${PI}"/>
 		</joint>
 		<!-- Link 4 -->
@@ -190,5 +190,5 @@
 			<child link="${prefix}link4"/>
 			<axis xyz="0 0 1"/>
-			<limit lower="-2.5307" upper="1.0472" effort="66" velocity="${PI}"/>
+			<limit lower="-${PI*143/180}" upper="${PI*58/180}" effort="66" velocity="${PI}"/>
 		</joint>
 		<!-- Link 5 - Mirrored COM and partial inertia -->
@@ -228,5 +228,5 @@
 			<child link="${prefix}link5"/>
 			<axis xyz="0 0 1"/>
-			<limit lower="-3.1067" upper="3.1067" effort="18" velocity="${PI}"/>
+			<limit lower="-${PI*168/180}" upper="${PI*168/180}" effort="18" velocity="${PI}"/>
 		</joint>
 		<!-- Link 6 - Partially mirrored COM and inertia -->
@@ -266,5 +266,5 @@
 			<child link="${prefix}link6"/>
 			<axis xyz="0 0 1"/>
-			<limit lower="-1.0472" upper="1.0472" effort="18" velocity="${PI}"/>
+			<limit lower="-${PI*58/180}" upper="${PI*58/180}" effort="18" velocity="${PI}"/>
 		</joint>
 		<!-- Link 7 -->
@@ -309,5 +309,5 @@
 			<child link="${prefix}link7"/>
 			<axis xyz="0 0 1"/>
-			<limit lower="-${PI/2}" upper="${PI/2}" effort="18" velocity="${PI}"/>
+			<limit lower="-${PI*78/180}" upper="${PI*78/180}" effort="18" velocity="${PI}"/>
 		</joint>
 		<link name="${prefix}tcp"/>
