Commit message: migrate to glb mesh

File: urdf/fiveages_w2.urdf (robot description, URDF)
Before this commit: robot FiveAges W2, 44 links, 43 joints
Links:
- link body_base: geometry collision mesh filename=package://fiveages_w2_description/meshes/body/base.glb; visual mesh filename=package://fiveages_w2_description/meshes/body/base.glb
- link body_camera: geometry visual mesh filename=package://sensor_models/meshes/orbbec/336.glb
- link body_link1: geometry collision mesh filename=package://fiveages_w2_description/meshes/body/link1.glb; visual mesh filename=package://fiveages_w2_description/meshes/body/link1.glb
- link body_link2: geometry collision mesh filename=package://fiveages_w2_description/meshes/body/link2.glb; visual mesh filename=package://fiveages_w2_description/meshes/body/link2.glb
- link body_link3: geometry collision mesh filename=package://fiveages_w2_description/meshes/body/link3.glb; visual mesh filename=package://fiveages_w2_description/meshes/body/link3.glb
- link body_link4: geometry collision box size=0.2000 0.32 0.5029; visual mesh filename=package://fiveages_w2_description/meshes/body/link4.glb
- link fl_lidar: geometry collision mesh filename=package://fiveages_w2_description/meshes/linkhou_s2/lidar.g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; visual mesh filename=package://fiveages_w2_description/meshes/linkhou_s2/lidar.g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
- link fl_wheel: geometry collision cylinder length=0.046 radius=0.07; visual mesh filename=package://fiveages_w2_description/meshes/linkhou_s2/wheel.g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
- link fr_wheel: geometry collision cylinder length=0.046 radius=0.07; visual mesh filename=package://fiveages_w2_description/meshes/linkhou_s2/wheel.g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 scale=1 -1 1
- link head_camera: geometry visual mesh filename=package://sensor_models/meshes/orbbec/336L.glb
- link head_link1: geometry collision mesh filename=package://fiveages_w2_description/meshes/body/head_yaw.glb; visual mesh filename=package://fiveages_w2_description/meshes/body/head_yaw.glb
- link head_link2: geometry collision mesh filename=package://fiveages_w2_description/meshes/body/head_pitch.glb; visual mesh filename=package://fiveages_w2_description/meshes/body/head_pitch.glb
- link left_base_link: geometry collision cylinder length=0.083664 radius=0.051277; visual mesh filename=package://m6_ccs_description/meshes/base.glb
- link left_link1: geometry collision cylinder length=0.125958 radius=0.057588; visual mesh filename=package://m6_ccs_description/meshes/link1.glb
- link left_link2: geometry collision cylinder length=0.078386 radius=0.046717; visual mesh filename=package://m6_ccs_description/meshes/link2.glb
- link left_link3: geometry collision cylinder length=0.089056 radius=0.046717; collision cylinder length=0.117016 radius=0.049964
- link left_link4: geometry collision cylinder length=0.080203 radius=0.041759; visual mesh filename=package://m6_ccs_description/meshes/link4.glb
- link left_link5: geometry collision cylinder length=0.14268 radius=0.056747; visual mesh filename=package://m6_ccs_description/meshes/link5.glb scale=1 1 1
- link left_link6: geometry collision cylinder length=0.108046 radius=0.038348; visual mesh filename=package://m6_ccs_description/meshes/link6.glb
- link left_link7: geometry collision cylinder length=0.038392 radius=0.041707; visual mesh filename=package://m6_ccs_description/meshes/link7.glb
- link right_base_link: geometry collision cylinder length=0.083664 radius=0.051277; visual mesh filename=package://m6_ccs_description/meshes/base.glb
- link right_link1: geometry collision cylinder length=0.125958 radius=0.057588; visual mesh filename=package://m6_ccs_description/meshes/link1.glb
- link right_link2: geometry collision cylinder length=0.078386 radius=0.046717; visual mesh filename=package://m6_ccs_description/meshes/link2.glb
- link right_link3: geometry collision cylinder length=0.089056 radius=0.046717; collision cylinder length=0.117016 radius=0.049964
- link right_link4: geometry collision cylinder length=0.080203 radius=0.041759; visual mesh filename=package://m6_ccs_description/meshes/link4.glb
- link right_link5: geometry collision cylinder length=0.14268 radius=0.056747; visual mesh filename=package://m6_ccs_description/meshes/link5.glb scale=1 -1 1
- link right_link6: geometry collision cylinder length=0.108046 radius=0.038348; visual mesh filename=package://m6_ccs_description/meshes/link6.glb
- link right_link7: geometry collision cylinder length=0.038392 radius=0.041707; visual mesh filename=package://m6_ccs_description/meshes/link7_r.glb
- link rl_wheel: geometry collision cylinder length=0.046 radius=0.07; visual mesh filename=package://fiveages_w2_description/meshes/linkhou_s2/wheel.g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
- link rr_lidar: geometry collision mesh filename=package://fiveages_w2_description/meshes/linkhou_s2/lidar.g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; visual mesh filename=package://fiveages_w2_description/meshes/linkhou_s2/lidar.g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
- link rr_wheel: geometry collision cylinder length=0.046 radius=0.07; visual mesh filename=package://fiveages_w2_description/meshes/linkhou_s2/wheel.g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 scale=1 -1 1

File: urdf/fiveages_w2_ag2f90.urdf (robot description, URDF)
Before this commit: robot FiveAges W2, 68 links, 67 joints
Links:
- link body_base: geometry collision mesh filename=package://fiveages_w2_description/meshes/body/base.glb; visual mesh filename=package://fiveages_w2_description/meshes/body/base.glb
- link body_camera: geometry visual mesh filename=package://sensor_models/meshes/orbbec/336.glb
- link body_link1: geometry collision mesh filename=package://fiveages_w2_description/meshes/body/link1.glb; visual mesh filename=package://fiveages_w2_description/meshes/body/link1.glb
- link body_link2: geometry collision mesh filename=package://fiveages_w2_description/meshes/body/link2.glb; visual mesh filename=package://fiveages_w2_description/meshes/body/link2.glb
- link body_link3: geometry collision mesh filename=package://fiveages_w2_description/meshes/body/link3.glb; visual mesh filename=package://fiveages_w2_description/meshes/body/link3.glb
- link body_link4: geometry collision box size=0.2000 0.32 0.5029; visual mesh filename=package://fiveages_w2_description/meshes/body/link4.glb
- link fl_lidar: geometry collision mesh filename=package://fiveages_w2_description/meshes/linkhou_s2/lidar.g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; visual mesh filename=package://fiveages_w2_description/meshes/linkhou_s2/lidar.g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
- link fl_wheel: geometry collision cylinder length=0.046 radius=0.07; visual mesh filename=package://fiveages_w2_description/meshes/linkhou_s2/wheel.g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
- link fr_wheel: geometry collision cylinder length=0.046 radius=0.07; visual mesh filename=package://fiveages_w2_description/meshes/linkhou_s2/wheel.g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 scale=1 -1 1
- link head_camera: geometry visual mesh filename=package://sensor_models/meshes/orbbec/336L.glb
- link head_link1: geometry collision mesh filename=package://fiveages_w2_description/meshes/body/head_yaw.glb; visual mesh filename=package://fiveages_w2_description/meshes/body/head_yaw.glb
- link head_link2: geometry collision mesh filename=package://fiveages_w2_description/meshes/body/head_pitch.glb; visual mesh filename=package://fiveages_w2_description/meshes/body/head_pitch.glb
- link left_base_link: geometry collision cylinder length=0.083664 radius=0.051277; visual mesh filename=package://m6_ccs_description/meshes/base.glb
- link left_link1: geometry collision cylinder length=0.125958 radius=0.057588; visual mesh filename=package://m6_ccs_description/meshes/link1.glb
- link left_link2: geometry collision cylinder length=0.078386 radius=0.046717; visual mesh filename=package://m6_ccs_description/meshes/link2.glb
- link left_link3: geometry collision cylinder length=0.089056 radius=0.046717; collision cylinder length=0.117016 radius=0.049964
- link left_link4: geometry collision cylinder length=0.080203 radius=0.041759; visual mesh filename=package://m6_ccs_description/meshes/link4.glb
- link left_link5: geometry collision cylinder length=0.14268 radius=0.056747; visual mesh filename=package://m6_ccs_description/meshes/link5.glb scale=1 1 1
- link left_link6: geometry collision cylinder length=0.108046 radius=0.038348; visual mesh filename=package://m6_ccs_description/meshes/link6.glb
- link left_link7: geometry collision cylinder length=0.038392 radius=0.041707; visual mesh filename=package://m6_ccs_description/meshes/link7.glb
- link right_base_link: geometry collision cylinder length=0.083664 radius=0.051277; visual mesh filename=package://m6_ccs_description/meshes/base.glb
- link right_link1: geometry collision cylinder length=0.125958 radius=0.057588; visual mesh filename=package://m6_ccs_description/meshes/link1.glb
- link right_link2: geometry collision cylinder length=0.078386 radius=0.046717; visual mesh filename=package://m6_ccs_description/meshes/link2.glb
- link right_link3: geometry collision cylinder length=0.089056 radius=0.046717; collision cylinder length=0.117016 radius=0.049964
- link right_link4: geometry collision cylinder length=0.080203 radius=0.041759; visual mesh filename=package://m6_ccs_description/meshes/link4.glb
- link right_link5: geometry collision cylinder length=0.14268 radius=0.056747; visual mesh filename=package://m6_ccs_description/meshes/link5.glb scale=1 -1 1
- link right_link6: geometry collision cylinder length=0.108046 radius=0.038348; visual mesh filename=package://m6_ccs_description/meshes/link6.glb
- link right_link7: geometry collision cylinder length=0.038392 radius=0.041707; visual mesh filename=package://m6_ccs_description/meshes/link7_r.glb
- link rl_wheel: geometry collision cylinder length=0.046 radius=0.07; visual mesh filename=package://fiveages_w2_description/meshes/linkhou_s2/wheel.g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
- link rr_lidar: geometry collision mesh filename=package://fiveages_w2_description/meshes/linkhou_s2/lidar.g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; visual mesh filename=package://fiveages_w2_description/meshes/linkhou_s2/lidar.g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
- link rr_wheel: geometry collision cylinder length=0.046 radius=0.07; visual mesh filename=package://fiveages_w2_description/meshes/linkhou_s2/wheel.g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 scale=1 -1 1

File: urdf/fiveages_w2_rg75.urdf (robot description, URDF)
Before this commit: robot FiveAges W2, 56 links, 55 joints
Links:
- link body_base: geometry collision mesh filename=package://fiveages_w2_description/meshes/body/base.glb; visual mesh filename=package://fiveages_w2_description/meshes/body/base.glb
- link body_camera: geometry visual mesh filename=package://sensor_models/meshes/orbbec/336.glb
- link body_link1: geometry collision mesh filename=package://fiveages_w2_description/meshes/body/link1.glb; visual mesh filename=package://fiveages_w2_description/meshes/body/link1.glb
- link body_link2: geometry collision mesh filename=package://fiveages_w2_description/meshes/body/link2.glb; visual mesh filename=package://fiveages_w2_description/meshes/body/link2.glb
- link body_link3: geometry collision mesh filename=package://fiveages_w2_description/meshes/body/link3.glb; visual mesh filename=package://fiveages_w2_description/meshes/body/link3.glb
- link body_link4: geometry collision box size=0.2000 0.32 0.5029; visual mesh filename=package://fiveages_w2_description/meshes/body/link4.glb
- link fl_lidar: geometry collision mesh filename=package://fiveages_w2_description/meshes/linkhou_s2/lidar.g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; visual mesh filename=package://fiveages_w2_description/meshes/linkhou_s2/lidar.g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
- link fl_wheel: geometry collision cylinder length=0.046 radius=0.07; visual mesh filename=package://fiveages_w2_description/meshes/linkhou_s2/wheel.g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
- link fr_wheel: geometry collision cylinder length=0.046 radius=0.07; visual mesh filename=package://fiveages_w2_description/meshes/linkhou_s2/wheel.g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 scale=1 -1 1
- link head_camera: geometry visual mesh filename=package://sensor_models/meshes/orbbec/336L.glb
- link head_link1: geometry collision mesh filename=package://fiveages_w2_description/meshes/body/head_yaw.glb; visual mesh filename=package://fiveages_w2_description/meshes/body/head_yaw.glb
- link head_link2: geometry collision mesh filename=package://fiveages_w2_description/meshes/body/head_pitch.glb; visual mesh filename=package://fiveages_w2_description/meshes/body/head_pitch.glb
- link left_base_link: geometry collision cylinder length=0.083664 radius=0.051277; visual mesh filename=package://m6_ccs_description/meshes/base.glb
- link left_flange: geometry collision mesh filename=package://jodell_description/meshes/RG75/flange.glb; visual mesh filename=package://jodell_description/meshes/RG75/flange.glb
- link left_gripper_base: geometry collision mesh filename=package://jodell_description/meshes/RG75/base.glb; visual mesh filename=package://jodell_description/meshes/RG75/base.glb
- link left_left_finger: geometry collision mesh filename=package://jodell_description/meshes/RG75/finger.glb; visual mesh filename=package://jodell_description/meshes/RG75/finger.glb
- link left_left_finger_pad: geometry collision mesh filename=package://jodell_description/meshes/RG75/pad_fiveages.glb; visual mesh filename=package://jodell_description/meshes/RG75/pad_fiveages.glb
- link left_link1: geometry collision cylinder length=0.125958 radius=0.057588; visual mesh filename=package://m6_ccs_description/meshes/link1.glb
- link left_link2: geometry collision cylinder length=0.078386 radius=0.046717; visual mesh filename=package://m6_ccs_description/meshes/link2.glb
- link left_link3: geometry collision cylinder length=0.089056 radius=0.046717; collision cylinder length=0.117016 radius=0.049964
- link left_link4: geometry collision cylinder length=0.080203 radius=0.041759; visual mesh filename=package://m6_ccs_description/meshes/link4.glb
- link left_link5: geometry collision cylinder length=0.14268 radius=0.056747; visual mesh filename=package://m6_ccs_description/meshes/link5.glb scale=1 1 1
- link left_link6: geometry collision cylinder length=0.108046 radius=0.038348; visual mesh filename=package://m6_ccs_description/meshes/link6.glb
- link left_link7: geometry collision cylinder length=0.038392 radius=0.041707; visual mesh filename=package://m6_ccs_description/meshes/link7.glb
- link left_right_finger: geometry collision mesh filename=package://jodell_description/meshes/RG75/finger.glb scale=-1 -1 1; visual mesh filename=package://jodell_description/meshes/RG75/finger.glb scale=-1 -1 1
- link left_right_finger_pad: geometry collision mesh filename=package://jodell_description/meshes/RG75/pad_fiveages.glb scale=1 -1 1; visual mesh filename=package://jodell_description/meshes/RG75/pad_fiveages.glb scale=1 -1 1
- link right_base_link: geometry collision cylinder length=0.083664 radius=0.051277; visual mesh filename=package://m6_ccs_description/meshes/base.glb
- link right_flange: geometry collision mesh filename=package://jodell_description/meshes/RG75/flange.glb; visual mesh filename=package://jodell_description/meshes/RG75/flange.glb
- link right_gripper_base: geometry collision mesh filename=package://jodell_description/meshes/RG75/base.glb; visual mesh filename=package://jodell_description/meshes/RG75/base.glb
- link right_left_finger: geometry collision mesh filename=package://jodell_description/meshes/RG75/finger.glb; visual mesh filename=package://jodell_description/meshes/RG75/finger.glb
- link right_left_finger_pad: geometry collision mesh filename=package://jodell_description/meshes/RG75/pad_fiveages.glb; visual mesh filename=package://jodell_description/meshes/RG75/pad_fiveages.glb
- link right_link1: geometry collision cylinder length=0.125958 radius=0.057588; visual mesh filename=package://m6_ccs_description/meshes/link1.glb
- link right_link2: geometry collision cylinder length=0.078386 radius=0.046717; visual mesh filename=package://m6_ccs_description/meshes/link2.glb
- link right_link3: geometry collision cylinder length=0.089056 radius=0.046717; collision cylinder length=0.117016 radius=0.049964
- link right_link4: geometry collision cylinder length=0.080203 radius=0.041759; visual mesh filename=package://m6_ccs_description/meshes/link4.glb
- link right_link5: geometry collision cylinder length=0.14268 radius=0.056747; visual mesh filename=package://m6_ccs_description/meshes/link5.glb scale=1 -1 1
- link right_link6: geometry collision cylinder length=0.108046 radius=0.038348; visual mesh filename=package://m6_ccs_description/meshes/link6.glb
- link right_link7: geometry collision cylinder length=0.038392 radius=0.041707; visual mesh filename=package://m6_ccs_description/meshes/link7_r.glb
- link right_right_finger: geometry collision mesh filename=package://jodell_description/meshes/RG75/finger.glb scale=-1 -1 1; visual mesh filename=package://jodell_description/meshes/RG75/finger.glb scale=-1 -1 1
- link right_right_finger_pad: geometry collision mesh filename=package://jodell_description/meshes/RG75/pad_fiveages.glb scale=1 -1 1; visual mesh filename=package://jodell_description/meshes/RG75/pad_fiveages.glb scale=1 -1 1
- link rl_wheel: geometry collision cylinder length=0.046 radius=0.07; visual mesh filename=package://fiveages_w2_description/meshes/linkhou_s2/wheel.g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
- link rr_lidar: geometry collision mesh filename=package://fiveages_w2_description/meshes/linkhou_s2/lidar.g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; visual mesh filename=package://fiveages_w2_description/meshes/linkhou_s2/lidar.g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
- link rr_wheel: geometry collision cylinder length=0.046 radius=0.07; visual mesh filename=package://fiveages_w2_description/meshes/linkhou_s2/wheel.g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 scale=1 -1 1

File: xacro/body.xacro (robot description, xacro)
@@ -16,10 +16,10 @@
 		<visual>
 			<geometry>
-				<mesh filename="file://$(find fiveages_w2_description)/meshes/body/base.obj"/>
-			</geometry>
-		</visual>
-		<collision>
-			<geometry>
-				<mesh filename="file://$(find fiveages_w2_description)/meshes/body/base.obj"/>
+				<mesh filename="file://$(find fiveages_w2_description)/meshes/body/base.glb"/>
+			</geometry>
+		</visual>
+		<collision>
+			<geometry>
+				<mesh filename="file://$(find fiveages_w2_description)/meshes/body/base.glb"/>
 			</geometry>
 		</collision>
@@ -44,10 +44,10 @@
 		<visual>
 			<geometry>
-				<mesh filename="file://$(find fiveages_w2_description)/meshes/body/link1.obj"/>
-			</geometry>
-		</visual>
-		<collision>
-			<geometry>
-				<mesh filename="file://$(find fiveages_w2_description)/meshes/body/link1.obj"/>
+				<mesh filename="file://$(find fiveages_w2_description)/meshes/body/link1.glb"/>
+			</geometry>
+		</visual>
+		<collision>
+			<geometry>
+				<mesh filename="file://$(find fiveages_w2_description)/meshes/body/link1.glb"/>
 			</geometry>
 		</collision>
@@ -57,5 +57,5 @@
 		<child link="body_link1"/>
 		<axis xyz="0 1 0"/>
-		<limit lower="-1.352633" upper="0.567" effort="100" velocity="1"/>
+		<limit lower="-1.352633" upper="0.567" effort="500" velocity="1"/>
 	</joint>
 	<link name="body_link2">
@@ -73,10 +73,10 @@
 		<visual>
 			<geometry>
-				<mesh filename="file://$(find fiveages_w2_description)/meshes/body/link2.obj"/>
-			</geometry>
-		</visual>
-		<collision>
-			<geometry>
-				<mesh filename="file://$(find fiveages_w2_description)/meshes/body/link2.obj"/>
+				<mesh filename="file://$(find fiveages_w2_description)/meshes/body/link2.glb"/>
+			</geometry>
+		</visual>
+		<collision>
+			<geometry>
+				<mesh filename="file://$(find fiveages_w2_description)/meshes/body/link2.glb"/>
 			</geometry>
 		</collision>
@@ -87,5 +87,5 @@
 		<child link="body_link2"/>
 		<axis xyz="0 -1 0"/>
-		<limit lower="-2.66" upper="1.605" effort="100" velocity="1"/>
+		<limit lower="-2.66" upper="1.605" effort="500" velocity="1"/>
 	</joint>
 	<link name="body_link3">
@@ -103,10 +103,10 @@
 		<visual>
 			<geometry>
-				<mesh filename="file://$(find fiveages_w2_description)/meshes/body/link3.obj"/>
-			</geometry>
-		</visual>
-		<collision>
-			<geometry>
-				<mesh filename="file://$(find fiveages_w2_description)/meshes/body/link3.obj"/>
+				<mesh filename="file://$(find fiveages_w2_description)/meshes/body/link3.glb"/>
+			</geometry>
+		</visual>
+		<collision>
+			<geometry>
+				<mesh filename="file://$(find fiveages_w2_description)/meshes/body/link3.glb"/>
 			</geometry>
 		</collision>
@@ -117,5 +117,5 @@
 		<child link="body_link3"/>
 		<axis xyz="0 1 0"/>
-		<limit lower="-1.745" upper="1.745" effort="100" velocity="1"/>
+		<limit lower="-1.745" upper="1.745" effort="500" velocity="1"/>
 	</joint>
 	<link name="body_link4">
@@ -133,5 +133,5 @@
 		<visual>
 			<geometry>
-				<mesh filename="file://$(find fiveages_w2_description)/meshes/body/link4.obj"/>
+				<mesh filename="file://$(find fiveages_w2_description)/meshes/body/link4.glb"/>
 			</geometry>
 		</visual>
@@ -148,10 +148,10 @@
 		<child link="body_link4"/>
 		<axis xyz="0 0 -1"/>
-		<limit lower="-${PI}" upper="${PI}" effort="100" velocity="1"/>
+		<limit lower="-${PI}" upper="${PI}" effort="500" velocity="1"/>
 	</joint>
 	<link name="body_camera">
 		<visual>
 			<geometry>
-				<mesh filename="file://$(find sensor_models)/meshes/orbbec/336.obj"/>
+				<mesh filename="file://$(find sensor_models)/meshes/orbbec/336.glb"/>
 			</geometry>
 		</visual>
@@ -176,10 +176,10 @@
 		<visual>
 			<geometry>
-				<mesh filename="file://$(find fiveages_w2_description)/meshes/body/head_yaw.obj"/>
-			</geometry>
-		</visual>
-		<collision>
-			<geometry>
-				<mesh filename="file://$(find fiveages_w2_description)/meshes/body/head_yaw.obj"/>
+				<mesh filename="file://$(find fiveages_w2_description)/meshes/body/head_yaw.glb"/>
+			</geometry>
+		</visual>
+		<collision>
+			<geometry>
+				<mesh filename="file://$(find fiveages_w2_description)/meshes/body/head_yaw.glb"/>
 			</geometry>
 		</collision>
@@ -190,5 +190,5 @@
 		<child link="head_link1"/>
 		<axis xyz="0 0 1"/>
-		<limit lower="-0.436" upper="0.436" effort="100" velocity="1"/>
+		<limit lower="-0.436" upper="0.436" effort="500" velocity="1"/>
 	</joint>
 	<link name="head_link2">
@@ -206,10 +206,10 @@
 		<visual>
 			<geometry>
-				<mesh filename="file://$(find fiveages_w2_description)/meshes/body/head_pitch.obj"/>
-			</geometry>
-		</visual>
-		<collision>
-			<geometry>
-				<mesh filename="file://$(find fiveages_w2_description)/meshes/body/head_pitch.obj"/>
+				<mesh filename="file://$(find fiveages_w2_description)/meshes/body/head_pitch.glb"/>
+			</geometry>
+		</visual>
+		<collision>
+			<geometry>
+				<mesh filename="file://$(find fiveages_w2_description)/meshes/body/head_pitch.glb"/>
 			</geometry>
 		</collision>
@@ -220,10 +220,10 @@
 		<child link="head_link2"/>
 		<axis xyz="0 1 0"/>
-		<limit lower="-0.26" upper="0.26" effort="100" velocity="1"/>
+		<limit lower="-0.26" upper="0.26" effort="500" velocity="1"/>
 	</joint>
 	<link name="head_camera">
 		<visual>
 			<geometry>
-				<mesh filename="file://$(find sensor_models)/meshes/orbbec/336L.obj"/>
+				<mesh filename="file://$(find sensor_models)/meshes/orbbec/336L.glb"/>
 			</geometry>
 		</visual>
