Commit message: migrate to glb mesh

File: xacro/components/arm.xacro (robot description, xacro)
@@ -15,11 +15,11 @@
 			<visual>
 				<geometry>
-					<mesh filename="file://$(find m6_ccs_description)/meshes/base.obj"/>
-				</geometry>
-			</visual>
-			<xacro:if value="${collider == 'convex'}">
-				<collision>
-					<geometry>
-						<mesh filename="file://$(find m6_ccs_description)/meshes/base.obj"/>
+					<mesh filename="file://$(find m6_ccs_description)/meshes/base.glb"/>
+				</geometry>
+			</visual>
+			<xacro:if value="${collider == 'convex'}">
+				<collision>
+					<geometry>
+						<mesh filename="file://$(find m6_ccs_description)/meshes/base.glb"/>
 					</geometry>
 				</collision>
@@ -45,11 +45,11 @@
 			<visual>
 				<geometry>
-					<mesh filename="file://$(find fiveages_w2_description)/meshes/arm/link1.obj"/>
-				</geometry>
-			</visual>
-			<xacro:if value="${collider == 'convex'}">
-				<collision>
-					<geometry>
-						<mesh filename="file://$(find m6_ccs_description)/meshes/link1.obj"/>
+					<mesh filename="file://$(find fiveages_w2_description)/meshes/arm/link1.glb"/>
+				</geometry>
+			</visual>
+			<xacro:if value="${collider == 'convex'}">
+				<collision>
+					<geometry>
+						<mesh filename="file://$(find m6_ccs_description)/meshes/link1.glb"/>
 					</geometry>
 				</collision>
@@ -83,11 +83,11 @@
 			<visual>
 				<geometry>
-					<mesh filename="file://$(find fiveages_w2_description)/meshes/arm/link2.obj" scale="1 1 ${direction}"/>
-				</geometry>
-			</visual>
-			<xacro:if value="${collider == 'convex'}">
-				<collision>
-					<geometry>
-						<mesh filename="file://$(find m6_ccs_description)/meshes/link2.obj" scale="1 1 ${direction}"/>
+					<mesh filename="file://$(find fiveages_w2_description)/meshes/arm/link2.glb" scale="1 1 ${direction}"/>
+				</geometry>
+			</visual>
+			<xacro:if value="${collider == 'convex'}">
+				<collision>
+					<geometry>
+						<mesh filename="file://$(find m6_ccs_description)/meshes/link2.glb" scale="1 1 ${direction}"/>
 					</geometry>
 				</collision>
@@ -121,11 +121,11 @@
 			<visual>
 				<geometry>
-					<mesh filename="file://$(find fiveages_w2_description)/meshes/arm/link3.obj"/>
-				</geometry>
-			</visual>
-			<xacro:if value="${collider == 'convex'}">
-				<collision>
-					<geometry>
-						<mesh filename="file://$(find m6_ccs_description)/meshes/link3.obj"/>
+					<mesh filename="file://$(find fiveages_w2_description)/meshes/arm/link3.glb"/>
+				</geometry>
+			</visual>
+			<xacro:if value="${collider == 'convex'}">
+				<collision>
+					<geometry>
+						<mesh filename="file://$(find m6_ccs_description)/meshes/link3.glb"/>
 					</geometry>
 				</collision>
@@ -165,11 +165,11 @@
 			<visual>
 				<geometry>
-					<mesh filename="file://$(find fiveages_w2_description)/meshes/arm/link4.obj"/>
-				</geometry>
-			</visual>
-			<xacro:if value="${collider == 'convex'}">
-				<collision>
-					<geometry>
-						<mesh filename="file://$(find m6_ccs_description)/meshes/link4.obj"/>
+					<mesh filename="file://$(find fiveages_w2_description)/meshes/arm/link4.glb"/>
+				</geometry>
+			</visual>
+			<xacro:if value="${collider == 'convex'}">
+				<collision>
+					<geometry>
+						<mesh filename="file://$(find m6_ccs_description)/meshes/link4.glb"/>
 					</geometry>
 				</collision>
@@ -203,11 +203,11 @@
 			<visual>
 				<geometry>
-					<mesh filename="file://$(find fiveages_w2_description)/meshes/arm/link5.obj" scale="1 ${direction} 1"/>
-				</geometry>
-			</visual>
-			<xacro:if value="${collider == 'convex'}">
-				<collision>
-					<geometry>
-						<mesh filename="file://$(find m6_ccs_description)/meshes/link5.obj" scale="1 ${direction} 1"/>
+					<mesh filename="file://$(find fiveages_w2_description)/meshes/arm/link5.glb" scale="1 ${direction} 1"/>
+				</geometry>
+			</visual>
+			<xacro:if value="${collider == 'convex'}">
+				<collision>
+					<geometry>
+						<mesh filename="file://$(find m6_ccs_description)/meshes/link5.glb" scale="1 ${direction} 1"/>
 					</geometry>
 				</collision>
@@ -241,11 +241,11 @@
 			<visual>
 				<geometry>
-					<mesh filename="file://$(find fiveages_w2_description)/meshes/arm/link6.obj"/>
-				</geometry>
-			</visual>
-			<xacro:if value="${collider == 'convex'}">
-				<collision>
-					<geometry>
-						<mesh filename="file://$(find m6_ccs_description)/meshes/link6.obj"/>
+					<mesh filename="file://$(find fiveages_w2_description)/meshes/arm/link6.glb"/>
+				</geometry>
+			</visual>
+			<xacro:if value="${collider == 'convex'}">
+				<collision>
+					<geometry>
+						<mesh filename="file://$(find m6_ccs_description)/meshes/link6.glb"/>
 					</geometry>
 				</collision>
@@ -280,8 +280,8 @@
 				<geometry>
 					<xacro:if value="${direction == 1}">
-						<mesh filename="file://$(find fiveages_w2_description)/meshes/arm/link7.obj"/>
+						<mesh filename="file://$(find fiveages_w2_description)/meshes/arm/link7.glb"/>
 					</xacro:if>
 					<xacro:if value="${direction == -1}">
-						<mesh filename="file://$(find fiveages_w2_description)/meshes/arm/link7_r.obj"/>
+						<mesh filename="file://$(find fiveages_w2_description)/meshes/arm/link7_r.glb"/>
 					</xacro:if>
 				</geometry>
@@ -290,5 +290,5 @@
 				<collision>
 					<geometry>
-						<mesh filename="file://$(find m6_ccs_description)/meshes/link7.obj"/>
+						<mesh filename="file://$(find m6_ccs_description)/meshes/link7.glb"/>
 					</geometry>
 				</collision>

File: xacro/components/linkhou_s2.xacro (robot description, xacro)
@@ -38,5 +38,5 @@
 			<visual>
 				<geometry>
-					<mesh filename="file://$(find fiveages_w2_description)/meshes/linkhou_s2/base_link.obj"/>
+					<mesh filename="file://$(find fiveages_w2_description)/meshes/linkhou_s2/base_link.glb"/>
 				</geometry>
 			</visual>
@@ -62,5 +62,5 @@
 			<visual>
 				<geometry>
-					<mesh filename="file://$(find fiveages_w2_description)/meshes/linkhou_s2/steer_link.obj" scale="1 -1 1"/>
+					<mesh filename="file://$(find fiveages_w2_description)/meshes/linkhou_s2/steer_link.glb" scale="1 -1 1"/>
 				</geometry>
 			</visual>
@@ -89,5 +89,5 @@
 			<visual>
 				<geometry>
-					<mesh filename="file://$(find fiveages_w2_description)/meshes/linkhou_s2/wheel.obj" scale="1 -1 1"/>
+					<mesh filename="file://$(find fiveages_w2_description)/meshes/linkhou_s2/wheel.glb" scale="1 -1 1"/>
 				</geometry>
 			</visual>
@@ -121,5 +121,5 @@
 			<visual>
 				<geometry>
-					<mesh filename="file://$(find fiveages_w2_description)/meshes/linkhou_s2/steer_link.obj"/>
+					<mesh filename="file://$(find fiveages_w2_description)/meshes/linkhou_s2/steer_link.glb"/>
 				</geometry>
 			</visual>
@@ -148,5 +148,5 @@
 			<visual>
 				<geometry>
-					<mesh filename="file://$(find fiveages_w2_description)/meshes/linkhou_s2/wheel.obj"/>
+					<mesh filename="file://$(find fiveages_w2_description)/meshes/linkhou_s2/wheel.glb"/>
 				</geometry>
 			</visual>
@@ -180,5 +180,5 @@
 			<visual>
 				<geometry>
-					<mesh filename="file://$(find fiveages_w2_description)/meshes/linkhou_s2/steer_link.obj" scale="1 -1 1"/>
+					<mesh filename="file://$(find fiveages_w2_description)/meshes/linkhou_s2/steer_link.glb" scale="1 -1 1"/>
 				</geometry>
 			</visual>
@@ -207,5 +207,5 @@
 			<visual>
 				<geometry>
-					<mesh filename="file://$(find fiveages_w2_description)/meshes/linkhou_s2/wheel.obj" scale="1 -1 1"/>
+					<mesh filename="file://$(find fiveages_w2_description)/meshes/linkhou_s2/wheel.glb" scale="1 -1 1"/>
 				</geometry>
 			</visual>
@@ -239,5 +239,5 @@
 			<visual>
 				<geometry>
-					<mesh filename="file://$(find fiveages_w2_description)/meshes/linkhou_s2/steer_link.obj"/>
+					<mesh filename="file://$(find fiveages_w2_description)/meshes/linkhou_s2/steer_link.glb"/>
 				</geometry>
 			</visual>
@@ -266,5 +266,5 @@
 			<visual>
 				<geometry>
-					<mesh filename="file://$(find fiveages_w2_description)/meshes/linkhou_s2/wheel.obj"/>
+					<mesh filename="file://$(find fiveages_w2_description)/meshes/linkhou_s2/wheel.glb"/>
 				</geometry>
 			</visual>
@@ -298,10 +298,10 @@
 			<visual>
 				<geometry>
-					<mesh filename="file://$(find fiveages_w2_description)/meshes/linkhou_s2/lidar.obj"/>
-				</geometry>
-			</visual>
-			<collision>
-				<geometry>
-					<mesh filename="file://$(find fiveages_w2_description)/meshes/linkhou_s2/lidar.obj"/>
+					<mesh filename="file://$(find fiveages_w2_description)/meshes/linkhou_s2/lidar.glb"/>
+				</geometry>
+			</visual>
+			<collision>
+				<geometry>
+					<mesh filename="file://$(find fiveages_w2_description)/meshes/linkhou_s2/lidar.glb"/>
 				</geometry>
 			</collision>
@@ -326,10 +326,10 @@
 			<visual>
 				<geometry>
-					<mesh filename="file://$(find fiveages_w2_description)/meshes/linkhou_s2/lidar.obj"/>
-				</geometry>
-			</visual>
-			<collision>
-				<geometry>
-					<mesh filename="file://$(find fiveages_w2_description)/meshes/linkhou_s2/lidar.obj"/>
+					<mesh filename="file://$(find fiveages_w2_description)/meshes/linkhou_s2/lidar.glb"/>
+				</geometry>
+			</visual>
+			<collision>
+				<geometry>
+					<mesh filename="file://$(find fiveages_w2_description)/meshes/linkhou_s2/lidar.glb"/>
 				</geometry>
 			</collision>
@@ -343,10 +343,10 @@
 			<visual>
 				<geometry>
-					<mesh filename="file://$(find fiveages_w2_description)/meshes/linkhou_s2/camera.obj"/>
-				</geometry>
-			</visual>
-			<collision>
-				<geometry>
-					<mesh filename="file://$(find fiveages_w2_description)/meshes/linkhou_s2/camera.obj"/>
+					<mesh filename="file://$(find fiveages_w2_description)/meshes/linkhou_s2/camera.glb"/>
+				</geometry>
+			</visual>
+			<collision>
+				<geometry>
+					<mesh filename="file://$(find fiveages_w2_description)/meshes/linkhou_s2/camera.glb"/>
 				</geometry>
 			</collision>

File: xacro/robot.xacro (robot description, xacro)
@@ -48,4 +48,7 @@
 		<xacro:property name="selected_hand_type" value="linkerhand_l6"/>
 	</xacro:if>
+	<xacro:if value="${type_arg == 'linkerhand_o7'}">
+		<xacro:property name="selected_hand_type" value="linkerhand_o7"/>
+	</xacro:if>
 	<xacro:include filename="$(find fiveages_w2_description)/xacro/eefs.xacro"/>
 	<xacro:EndEffectors hand_type="${selected_hand_type}" gripper_type="${selected_gripper_type}"/>

File: xacro/ros2_control/robot.xacro (robot description, xacro)
@@ -110,4 +110,9 @@
 				<xacro:linkerhand_o6_interfaces name="right_hand"/>
 			</xacro:if>
+			<xacro:if value="${selected_hand_type == 'linkerhand_o7'}">
+				<xacro:include filename="$(find linkerhand_description)/xacro/ros2_control/o7.xacro"/>
+				<xacro:linkerhand_o7_interfaces name="left_hand"/>
+				<xacro:linkerhand_o7_interfaces name="right_hand"/>
+			</xacro:if>
 		</ros2_control>
 	</xacro:unless>
