Commit message: update collision for gripper

File: urdf/fiveages_w2.urdf (robot description, URDF)
Before this commit: robot FiveAges W2, 44 links, 43 joints
Links:
- added link head_top_camera
- link body_base: geometry visual mesh filename=package://fiveages_w2_description/meshes/body/base.glb
- link body_link1: geometry collision box size=0.15 0.145 0.48; visual mesh filename=package://fiveages_w2_description/meshes/body/link1.glb
- link body_link2: geometry collision box size=0.16 0.2 0.5; visual mesh filename=package://fiveages_w2_description/meshes/body/link2.glb
- link body_link3: geometry collision box size=0.13 0.13 0.22; visual mesh filename=package://fiveages_w2_description/meshes/body/link3.glb
- link chassis_base: geometry collision box size=0.5 0.3 0.2; collision box size=0.66 0.16 0.3
- link chassis_camera: geometry visual mesh filename=package://fiveages_w2_description/meshes/linkhou_s2/camera.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
- link fl_lidar: geometry visual mesh filename=package://fiveages_w2_description/meshes/linkhou_s2/lidar.g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
- link head_link1: geometry visual mesh filename=package://fiveages_w2_description/meshes/body/head_yaw.glb
- link head_link2: geometry collision box size=0.15 0.16 0.24; visual mesh filename=package://fiveages_w2_description/meshes/body/head_pitch.glb
- link left_link1: geometry collision cylinder length=0.125958 radius=0.057588; visual mesh filename=package://fiveages_w2_description/meshes/arm/link1.glb
- link left_link2: geometry collision cylinder length=0.078386 radius=0.046717; visual mesh filename=package://fiveages_w2_description/meshes/arm/link2.glb scale=1 1 1
- link left_link3: geometry collision cylinder length=0.089056 radius=0.046717; collision cylinder length=0.117016 radius=0.049964
- link left_link4: geometry collision cylinder length=0.080203 radius=0.041759; visual mesh filename=package://fiveages_w2_description/meshes/arm/link4.glb
- link left_link5: geometry collision cylinder length=0.14268 radius=0.056747; visual mesh filename=package://fiveages_w2_description/meshes/arm/link5.glb scale=1 1 1
- link left_link6: geometry collision cylinder length=0.108046 radius=0.038348; visual mesh filename=package://fiveages_w2_description/meshes/arm/link6.glb
- link left_link7: geometry collision cylinder length=0.038392 radius=0.041707; visual mesh filename=package://fiveages_w2_description/meshes/arm/link7.glb
- link right_link1: geometry collision cylinder length=0.125958 radius=0.057588; visual mesh filename=package://fiveages_w2_description/meshes/arm/link1.glb
- link right_link2: geometry collision cylinder length=0.078386 radius=0.046717; visual mesh filename=package://fiveages_w2_description/meshes/arm/link2.glb scale=1 1 -1
- link right_link3: geometry collision cylinder length=0.089056 radius=0.046717; collision cylinder length=0.117016 radius=0.049964
- link right_link4: geometry collision cylinder length=0.080203 radius=0.041759; visual mesh filename=package://fiveages_w2_description/meshes/arm/link4.glb
- link right_link5: geometry collision cylinder length=0.14268 radius=0.056747; visual mesh filename=package://fiveages_w2_description/meshes/arm/link5.glb scale=1 -1 1
- link right_link6: geometry collision cylinder length=0.108046 radius=0.038348; visual mesh filename=package://fiveages_w2_description/meshes/arm/link6.glb
- link right_link7: geometry collision cylinder length=0.038392 radius=0.041707; visual mesh filename=package://fiveages_w2_description/meshes/arm/link7_r.glb
- link rr_lidar: geometry visual mesh filename=package://fiveages_w2_description/meshes/linkhou_s2/lidar.g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
Joints:
- added joint head_top_camera_joint: type fixed, parent head_link2, child head_top_camera, origin xyz=0.0877736 0.0245687 0.107989 rpy=-2.100227811211368 0.0016038446958035316 -1.583610269343787
- joint body_joint1: limit lower=-1.352633 upper=0.567 effort=100 velocity=1 -> lower=-1.352633 upper=0.567 effort=500 velocity=1
- joint body_joint2: limit lower=-2.66 upper=1.605 effort=100 velocity=1 -> lower=-2.66 upper=1.605 effort=500 velocity=1
- joint body_joint3: limit lower=-1.745 upper=1.745 effort=100 velocity=1 -> lower=-1.745 upper=1.745 effort=500 velocity=1
- joint body_joint4: limit lower=-3.141592653589793 upper=3.141592653589793 effort=100 velocity=1 -> lower=-3.141592653589793 upper=3.141592653589793 effort=500 velocity=1
- joint head_joint1: limit lower=-0.436 upper=0.436 effort=100 velocity=1 -> lower=-0.436 upper=0.436 effort=500 velocity=1
- joint head_joint2: limit lower=-0.26 upper=0.26 effort=100 velocity=1 -> lower=-0.26 upper=0.26 effort=500 velocity=1; origin xyz=0 0.0042 0.15 -> xyz=0 0.0 0.15

File: urdf/fiveages_w2_ag2f90.urdf (robot description, URDF)
Before this commit: robot FiveAges W2, 68 links, 67 joints
Links:
- added link head_top_camera
- link body_base: geometry visual mesh filename=package://fiveages_w2_description/meshes/body/base.glb
- link body_link1: geometry collision box size=0.15 0.145 0.48; visual mesh filename=package://fiveages_w2_description/meshes/body/link1.glb
- link body_link2: geometry collision box size=0.16 0.2 0.5; visual mesh filename=package://fiveages_w2_description/meshes/body/link2.glb
- link body_link3: geometry collision box size=0.13 0.13 0.22; visual mesh filename=package://fiveages_w2_description/meshes/body/link3.glb
- link chassis_base: geometry collision box size=0.5 0.3 0.2; collision box size=0.66 0.16 0.3
- link chassis_camera: geometry visual mesh filename=package://fiveages_w2_description/meshes/linkhou_s2/camera.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
- link fl_lidar: geometry visual mesh filename=package://fiveages_w2_description/meshes/linkhou_s2/lidar.g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
- link head_link1: geometry visual mesh filename=package://fiveages_w2_description/meshes/body/head_yaw.glb
- link head_link2: geometry collision box size=0.15 0.16 0.24; visual mesh filename=package://fiveages_w2_description/meshes/body/head_pitch.glb
- link left_gripper_base: geometry visual mesh filename=package://changingtek_description/meshes/AG2F90-C/visual/gr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
- link left_left_1_link: geometry visual mesh filename=package://changingtek_description/meshes/AG2F90-C/visual/li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
- link left_left_2_link: geometry visual mesh filename=package://changingtek_description/meshes/AG2F90-C/visual/li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
- link left_left_Pad_link: geometry visual mesh filename=package://changingtek_description/meshes/AG2F90-C/visual/pa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
- link left_left_in_link: geometry visual mesh filename=package://changingtek_description/meshes/AG2F90-C/visual/in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
- link left_left_up_link: geometry visual mesh filename=package://changingtek_description/meshes/AG2F90-C/visual/up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
- link left_link1: geometry collision cylinder length=0.125958 radius=0.057588; visual mesh filename=package://fiveages_w2_description/meshes/arm/link1.glb
- link left_link2: geometry collision cylinder length=0.078386 radius=0.046717; visual mesh filename=package://fiveages_w2_description/meshes/arm/link2.glb scale=1 1 1
- link left_link3: geometry collision cylinder length=0.089056 radius=0.046717; collision cylinder length=0.117016 radius=0.049964
- link left_link4: geometry collision cylinder length=0.080203 radius=0.041759; visual mesh filename=package://fiveages_w2_description/meshes/arm/link4.glb
- link left_link5: geometry collision cylinder length=0.14268 radius=0.056747; visual mesh filename=package://fiveages_w2_description/meshes/arm/link5.glb scale=1 1 1
- link left_link6: geometry collision cylinder length=0.108046 radius=0.038348; visual mesh filename=package://fiveages_w2_description/meshes/arm/link6.glb
- link left_link7: geometry collision cylinder length=0.038392 radius=0.041707; collision cylinder length=0.138392 radius=0.041707
- link left_right_1_link: geometry visual mesh filename=package://changingtek_description/meshes/AG2F90-C/visual/li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
- link left_right_2_link: geometry visual mesh filename=package://changingtek_description/meshes/AG2F90-C/visual/li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
- link left_right_Pad_link: geometry visual mesh filename=package://changingtek_description/meshes/AG2F90-C/visual/pa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
- link left_right_in_link: geometry visual mesh filename=package://changingtek_description/meshes/AG2F90-C/visual/in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
- link left_right_up_link: geometry visual mesh filename=package://changingtek_description/meshes/AG2F90-C/visual/up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
- link right_gripper_base: geometry visual mesh filename=package://changingtek_description/meshes/AG2F90-C/visual/gr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
- link right_left_1_link: geometry visual mesh filename=package://changingtek_description/meshes/AG2F90-C/visual/li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
- link right_left_2_link: geometry visual mesh filename=package://changingtek_description/meshes/AG2F90-C/visual/li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
- link right_left_Pad_link: geometry visual mesh filename=package://changingtek_description/meshes/AG2F90-C/visual/pa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
- link right_left_in_link: geometry visual mesh filename=package://changingtek_description/meshes/AG2F90-C/visual/in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
- link right_left_up_link: geometry visual mesh filename=package://changingtek_description/meshes/AG2F90-C/visual/up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
- link right_link1: geometry collision cylinder length=0.125958 radius=0.057588; visual mesh filename=package://fiveages_w2_description/meshes/arm/link1.glb
- link right_link2: geometry collision cylinder length=0.078386 radius=0.046717; visual mesh filename=package://fiveages_w2_description/meshes/arm/link2.glb scale=1 1 -1
- link right_link3: geometry collision cylinder length=0.089056 radius=0.046717; collision cylinder length=0.117016 radius=0.049964
- link right_link4: geometry collision cylinder length=0.080203 radius=0.041759; visual mesh filename=package://fiveages_w2_description/meshes/arm/link4.glb
- link right_link5: geometry collision cylinder length=0.14268 radius=0.056747; visual mesh filename=package://fiveages_w2_description/meshes/arm/link5.glb scale=1 -1 1
- link right_link6: geometry collision cylinder length=0.108046 radius=0.038348; visual mesh filename=package://fiveages_w2_description/meshes/arm/link6.glb
- link right_link7: geometry collision cylinder length=0.038392 radius=0.041707; collision cylinder length=0.138392 radius=0.041707
- link right_right_1_link: geometry visual mesh filename=package://changingtek_description/meshes/AG2F90-C/visual/li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
- link right_right_2_link: geometry visual mesh filename=package://changingtek_description/meshes/AG2F90-C/visual/li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
- link right_right_Pad_link: geometry visual mesh filename=package://changingtek_description/meshes/AG2F90-C/visual/pa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
- link right_right_in_link: geometry visual mesh filename=package://changingtek_description/meshes/AG2F90-C/visual/in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
- link right_right_up_link: geometry visual mesh filename=package://changingtek_description/meshes/AG2F90-C/visual/up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
- link rr_lidar: geometry visual mesh filename=package://fiveages_w2_description/meshes/linkhou_s2/lidar.g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
Joints:
- added joint head_top_camera_joint: type fixed, parent head_link2, child head_top_camera, origin xyz=0.0877736 0.0245687 0.107989 rpy=-2.100227811211368 0.0016038446958035316 -1.583610269343787
- joint body_joint1: limit lower=-1.352633 upper=0.567 effort=100 velocity=1 -> lower=-1.352633 upper=0.567 effort=500 velocity=1
- joint body_joint2: limit lower=-2.66 upper=1.605 effort=100 velocity=1 -> lower=-2.66 upper=1.605 effort=500 velocity=1
- joint body_joint3: limit lower=-1.745 upper=1.745 effort=100 velocity=1 -> lower=-1.745 upper=1.745 effort=500 velocity=1
- joint body_joint4: limit lower=-3.141592653589793 upper=3.141592653589793 effort=100 velocity=1 -> lower=-3.141592653589793 upper=3.141592653589793 effort=500 velocity=1
- joint head_joint1: limit lower=-0.436 upper=0.436 effort=100 velocity=1 -> lower=-0.436 upper=0.436 effort=500 velocity=1
- joint head_joint2: limit lower=-0.26 upper=0.26 effort=100 velocity=1 -> lower=-0.26 upper=0.26 effort=500 velocity=1; origin xyz=0 0.0042 0.15 -> xyz=0 0.0 0.15
- joint left_right_2_Joint: mimic joint=left_left_2_Joint -> joint=left_gripper_joint
- joint left_right_in_Joint: mimic joint=left_right_1_Joint multiplier=0.1 offset=0 -> joint=left_gripper_joint multiplier=0.1 offset=0
- joint left_right_up_Joint: mimic joint=left_right_1_Joint -> joint=left_gripper_joint
- joint right_right_2_Joint: mimic joint=right_left_2_Joint -> joint=right_gripper_joint
- joint right_right_in_Joint: mimic joint=right_right_1_Joint multiplier=0.1 offset=0 -> joint=right_gripper_joint multiplier=0.1 offset=0
- joint right_right_up_Joint: mimic joint=right_right_1_Joint -> joint=right_gripper_joint

File: urdf/fiveages_w2_rg75.urdf (robot description, URDF)
Before this commit: robot FiveAges W2, 56 links, 55 joints
Links:
- added link head_top_camera
- link body_base: geometry visual mesh filename=package://fiveages_w2_description/meshes/body/base.glb
- link body_link1: geometry collision box size=0.15 0.145 0.48; visual mesh filename=package://fiveages_w2_description/meshes/body/link1.glb
- link body_link2: geometry collision box size=0.16 0.2 0.5; visual mesh filename=package://fiveages_w2_description/meshes/body/link2.glb
- link body_link3: geometry collision box size=0.13 0.13 0.22; visual mesh filename=package://fiveages_w2_description/meshes/body/link3.glb
- link chassis_base: geometry collision box size=0.5 0.3 0.2; collision box size=0.66 0.16 0.3
- link chassis_camera: geometry visual mesh filename=package://fiveages_w2_description/meshes/linkhou_s2/camera.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
- link fl_lidar: geometry visual mesh filename=package://fiveages_w2_description/meshes/linkhou_s2/lidar.g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
- link head_link1: geometry visual mesh filename=package://fiveages_w2_description/meshes/body/head_yaw.glb
- link head_link2: geometry collision box size=0.15 0.16 0.24; visual mesh filename=package://fiveages_w2_description/meshes/body/head_pitch.glb
- link left_flange: geometry visual mesh filename=package://jodell_description/meshes/RG75/flange.glb
- link left_gripper_base: geometry visual mesh filename=package://jodell_description/meshes/RG75/base.glb
- link left_left_finger: geometry visual mesh filename=package://jodell_description/meshes/RG75/finger.glb
- link left_left_finger_pad: geometry visual mesh filename=package://jodell_description/meshes/RG75/pad_fiveages.glb
- link left_link1: geometry collision cylinder length=0.125958 radius=0.057588; visual mesh filename=package://fiveages_w2_description/meshes/arm/link1.glb
- link left_link2: geometry collision cylinder length=0.078386 radius=0.046717; visual mesh filename=package://fiveages_w2_description/meshes/arm/link2.glb scale=1 1 1
- link left_link3: geometry collision cylinder length=0.089056 radius=0.046717; collision cylinder length=0.117016 radius=0.049964
- link left_link4: geometry collision cylinder length=0.080203 radius=0.041759; visual mesh filename=package://fiveages_w2_description/meshes/arm/link4.glb
- link left_link5: geometry collision cylinder length=0.14268 radius=0.056747; visual mesh filename=package://fiveages_w2_description/meshes/arm/link5.glb scale=1 1 1
- link left_link6: geometry collision cylinder length=0.108046 radius=0.038348; visual mesh filename=package://fiveages_w2_description/meshes/arm/link6.glb
- link left_link7: geometry collision cylinder length=0.038392 radius=0.041707; collision cylinder length=0.138392 radius=0.041707
- link left_right_finger: geometry visual mesh filename=package://jodell_description/meshes/RG75/finger.glb scale=-1 -1 1
- link left_right_finger_pad: geometry visual mesh filename=package://jodell_description/meshes/RG75/pad_fiveages.glb scale=1 -1 1
- link right_flange: geometry visual mesh filename=package://jodell_description/meshes/RG75/flange.glb
- link right_gripper_base: geometry visual mesh filename=package://jodell_description/meshes/RG75/base.glb
- link right_left_finger: geometry visual mesh filename=package://jodell_description/meshes/RG75/finger.glb
- link right_left_finger_pad: geometry visual mesh filename=package://jodell_description/meshes/RG75/pad_fiveages.glb
- link right_link1: geometry collision cylinder length=0.125958 radius=0.057588; visual mesh filename=package://fiveages_w2_description/meshes/arm/link1.glb
- link right_link2: geometry collision cylinder length=0.078386 radius=0.046717; visual mesh filename=package://fiveages_w2_description/meshes/arm/link2.glb scale=1 1 -1
- link right_link3: geometry collision cylinder length=0.089056 radius=0.046717; collision cylinder length=0.117016 radius=0.049964
- link right_link4: geometry collision cylinder length=0.080203 radius=0.041759; visual mesh filename=package://fiveages_w2_description/meshes/arm/link4.glb
- link right_link5: geometry collision cylinder length=0.14268 radius=0.056747; visual mesh filename=package://fiveages_w2_description/meshes/arm/link5.glb scale=1 -1 1
- link right_link6: geometry collision cylinder length=0.108046 radius=0.038348; visual mesh filename=package://fiveages_w2_description/meshes/arm/link6.glb
- link right_link7: geometry collision cylinder length=0.038392 radius=0.041707; collision cylinder length=0.138392 radius=0.041707
- link right_right_finger: geometry visual mesh filename=package://jodell_description/meshes/RG75/finger.glb scale=-1 -1 1
- link right_right_finger_pad: geometry visual mesh filename=package://jodell_description/meshes/RG75/pad_fiveages.glb scale=1 -1 1
- link rr_lidar: geometry visual mesh filename=package://fiveages_w2_description/meshes/linkhou_s2/lidar.g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
Joints:
- added joint head_top_camera_joint: type fixed, parent head_link2, child head_top_camera, origin xyz=0.0877736 0.0245687 0.107989 rpy=-2.100227811211368 0.0016038446958035316 -1.583610269343787
- joint body_joint1: limit lower=-1.352633 upper=0.567 effort=100 velocity=1 -> lower=-1.352633 upper=0.567 effort=500 velocity=1
- joint body_joint2: limit lower=-2.66 upper=1.605 effort=100 velocity=1 -> lower=-2.66 upper=1.605 effort=500 velocity=1
- joint body_joint3: limit lower=-1.745 upper=1.745 effort=100 velocity=1 -> lower=-1.745 upper=1.745 effort=500 velocity=1
- joint body_joint4: limit lower=-3.141592653589793 upper=3.141592653589793 effort=100 velocity=1 -> lower=-3.141592653589793 upper=3.141592653589793 effort=500 velocity=1
- joint head_joint1: limit lower=-0.436 upper=0.436 effort=100 velocity=1 -> lower=-0.436 upper=0.436 effort=500 velocity=1
- joint head_joint2: limit lower=-0.26 upper=0.26 effort=100 velocity=1 -> lower=-0.26 upper=0.26 effort=500 velocity=1; origin xyz=0 0.0042 0.15 -> xyz=0 0.0 0.15

File: xacro/body.xacro (robot description, xacro)
@@ -19,9 +19,4 @@
 			</geometry>
 		</visual>
-		<collision>
-			<geometry>
-				<mesh filename="file://$(find fiveages_w2_description)/meshes/body/base.glb"/>
-			</geometry>
-		</collision>
 	</link>
 	<joint name="body_fixed_joint" type="fixed">
@@ -48,6 +43,7 @@
 		</visual>
 		<collision>
-			<geometry>
-				<mesh filename="file://$(find fiveages_w2_description)/meshes/body/link1.glb"/>
+			<origin xyz="0.0 0 0.17"/>
+			<geometry>
+				<box size="0.15 0.145 0.48"/>
 			</geometry>
 		</collision>
@@ -77,6 +73,7 @@
 		</visual>
 		<collision>
-			<geometry>
-				<mesh filename="file://$(find fiveages_w2_description)/meshes/body/link2.glb"/>
+			<origin xyz="0.0 0 0.18"/>
+			<geometry>
+				<box size="0.16 0.2 0.5"/>
 			</geometry>
 		</collision>
@@ -107,6 +104,7 @@
 		</visual>
 		<collision>
-			<geometry>
-				<mesh filename="file://$(find fiveages_w2_description)/meshes/body/link3.glb"/>
+			<origin xyz="0.0 0 0.032"/>
+			<geometry>
+				<box size="0.13 0.13 0.22"/>
 			</geometry>
 		</collision>
@@ -179,9 +177,4 @@
 			</geometry>
 		</visual>
-		<collision>
-			<geometry>
-				<mesh filename="file://$(find fiveages_w2_description)/meshes/body/head_yaw.glb"/>
-			</geometry>
-		</collision>
 	</link>
 	<joint name="head_joint1" type="revolute">
@@ -210,6 +203,7 @@
 		</visual>
 		<collision>
-			<geometry>
-				<mesh filename="file://$(find fiveages_w2_description)/meshes/body/head_pitch.glb"/>
+			<origin xyz="0.025 0 0.04"/>
+			<geometry>
+				<box size="0.15 0.16 0.24"/>
 			</geometry>
 		</collision>

File: xacro/components/arm.xacro (robot description, xacro)
@@ -301,4 +301,20 @@
 					</geometry>
 				</collision>
+				<xacro:if value="${selected_gripper_type == 'rg75'}">
+					<collision>
+						<origin xyz="0 -0.175732 0" rpy="${PI/2} 0 0"/>
+						<geometry>
+							<cylinder length="0.138392" radius="0.041707"/>
+						</geometry>
+					</collision>
+				</xacro:if>
+				<xacro:if value="${selected_gripper_type == 'ag2f90_c' or selected_gripper_type == 'ag2f90_d'}">
+					<collision>
+						<origin xyz="0 -0.175732 0" rpy="${PI/2} 0 0"/>
+						<geometry>
+							<cylinder length="0.138392" radius="0.041707"/>
+						</geometry>
+					</collision>
+				</xacro:if>
 			</xacro:if>
 		</link>

File: xacro/components/linkhou_s2.xacro (robot description, xacro)
@@ -47,4 +47,16 @@
 				</geometry>
 			</collision>
+			<collision>
+				<origin xyz="0 0.195 0.16"/>
+				<geometry>
+					<box size="0.66 0.16 0.3"/>
+				</geometry>
+			</collision>
+			<collision>
+				<origin xyz="0 -0.195 0.16"/>
+				<geometry>
+					<box size="0.66 0.16 0.3"/>
+				</geometry>
+			</collision>
 		</link>
 		<link name="rr_steer">
@@ -301,9 +313,4 @@
 				</geometry>
 			</visual>
-			<collision>
-				<geometry>
-					<mesh filename="file://$(find fiveages_w2_description)/meshes/linkhou_s2/lidar.glb"/>
-				</geometry>
-			</collision>
 		</link>
 		<joint name="rr_lidar_joint" type="fixed">
@@ -329,9 +336,4 @@
 				</geometry>
 			</visual>
-			<collision>
-				<geometry>
-					<mesh filename="file://$(find fiveages_w2_description)/meshes/linkhou_s2/lidar.glb"/>
-				</geometry>
-			</collision>
 		</link>
 		<joint name="fl_lidar_joint" type="fixed">
@@ -346,9 +348,4 @@
 				</geometry>
 			</visual>
-			<collision>
-				<geometry>
-					<mesh filename="file://$(find fiveages_w2_description)/meshes/linkhou_s2/camera.glb"/>
-				</geometry>
-			</collision>
 		</link>
 		<joint name="chassis_camera_joint" type="fixed">
