Commit message: update collision for gripper

File: xacro/robot.xacro (robot description, xacro)
@@ -3,22 +3,4 @@
 	<xacro:arg name="collider" default="convex"/>
 	<xacro:arg name="chassis_joints_movable" default="false"/>
-	<xacro:include filename="$(find fiveages_w2_description)/xacro/components/linkhou_s2.xacro"/>
-	<xacro:linkhou_s2 joints_movable="$(arg chassis_joints_movable)"/>
-	<xacro:include filename="$(find fiveages_w2_description)/xacro/body.xacro"/>
-	<!-- Left Arm -->
-	<joint name="left_arm_base_joint" type="fixed">
-		<parent link="arm_base"/>
-		<child link="left_base_link"/>
-		<origin rpy="-${PI/2} 0 0" xyz="0.0 0.062 0"/>
-	</joint>
-	<!-- Right Arm -->
-	<joint name="right_arm_base_joint" type="fixed">
-		<parent link="arm_base"/>
-		<child link="right_base_link"/>
-		<origin rpy="${PI/2} 0 0" xyz="0 -0.062 0"/>
-	</joint>
-	<xacro:include filename="$(find fiveages_w2_description)/xacro/components/arm.xacro"/>
-	<xacro:M6_CCS name="left" collider="$(arg collider)"/>
-	<xacro:M6_CCS name="right" direction="-1" collider="$(arg collider)"/>
 	<!-- 从 type 参数解析出 hand_type 和 gripper_type -->
 	<xacro:arg name="type" default=""/>
@@ -51,4 +33,22 @@
 		<xacro:property name="selected_hand_type" value="linkerhand_o7"/>
 	</xacro:if>
+	<xacro:include filename="$(find fiveages_w2_description)/xacro/components/linkhou_s2.xacro"/>
+	<xacro:linkhou_s2 joints_movable="$(arg chassis_joints_movable)"/>
+	<xacro:include filename="$(find fiveages_w2_description)/xacro/body.xacro"/>
+	<!-- Left Arm -->
+	<joint name="left_arm_base_joint" type="fixed">
+		<parent link="arm_base"/>
+		<child link="left_base_link"/>
+		<origin rpy="-${PI/2} 0 0" xyz="0.0 0.062 0"/>
+	</joint>
+	<!-- Right Arm -->
+	<joint name="right_arm_base_joint" type="fixed">
+		<parent link="arm_base"/>
+		<child link="right_base_link"/>
+		<origin rpy="${PI/2} 0 0" xyz="0 -0.062 0"/>
+	</joint>
+	<xacro:include filename="$(find fiveages_w2_description)/xacro/components/arm.xacro"/>
+	<xacro:M6_CCS name="left" collider="$(arg collider)"/>
+	<xacro:M6_CCS name="right" direction="-1" collider="$(arg collider)"/>
 	<xacro:include filename="$(find fiveages_w2_description)/xacro/eefs.xacro"/>
 	<xacro:EndEffectors hand_type="${selected_hand_type}" gripper_type="${selected_gripper_type}"/>

Commit message: 调整相机frame

File: urdf/fiveages_w2.urdf (robot description, URDF)
Before this commit: robot FiveAges W2, 45 links, 44 joints
Joints:
- joint body_camera_joint: origin xyz=0.10065 0.024257 0.28812 rpy=3.141592653589793 0.378684973 0 -> xyz=0.10065 0.024257 0.28812 rpy=-1.9494812997948965 0 -1.5707963267948966
- joint head_camera_joint: origin xyz=0.097847  0.046703 0.12364 rpy=3.141592653589793 0.64460396 0 -> xyz=0.097847  0.046703 0.12364 rpy=-2.2154002867948965 0 -1.5707963267948966

File: urdf/fiveages_w2_ag2f90.urdf (robot description, URDF)
Before this commit: robot FiveAges W2, 69 links, 68 joints
Joints:
- joint body_camera_joint: origin xyz=0.10065 0.024257 0.28812 rpy=3.141592653589793 0.378684973 0 -> xyz=0.10065 0.024257 0.28812 rpy=-1.9494812997948965 0 -1.5707963267948966
- joint head_camera_joint: origin xyz=0.097847  0.046703 0.12364 rpy=3.141592653589793 0.64460396 0 -> xyz=0.097847  0.046703 0.12364 rpy=-2.2154002867948965 0 -1.5707963267948966

File: urdf/fiveages_w2_rg75.urdf (robot description, URDF)
Before this commit: robot FiveAges W2, 57 links, 56 joints
Joints:
- joint body_camera_joint: origin xyz=0.10065 0.024257 0.28812 rpy=3.141592653589793 0.378684973 0 -> xyz=0.10065 0.024257 0.28812 rpy=-1.9494812997948965 0 -1.5707963267948966
- joint head_camera_joint: origin xyz=0.097847  0.046703 0.12364 rpy=3.141592653589793 0.64460396 0 -> xyz=0.097847  0.046703 0.12364 rpy=-2.2154002867948965 0 -1.5707963267948966

File: urdf/fiveages_w2_rg75_heavy.urdf (robot description, URDF)
Before this commit: robot FiveAges W2, 57 links, 56 joints
Joints:
- joint body_camera_joint: origin xyz=0.10065 0.024257 0.28812 rpy=3.141592653589793 0.378684973 0 -> xyz=0.10065 0.024257 0.28812 rpy=-1.9494812997948965 0 -1.5707963267948966
- joint head_camera_joint: origin xyz=0.097847  0.046703 0.12364 rpy=3.141592653589793 0.64460396 0 -> xyz=0.097847  0.046703 0.12364 rpy=-2.2154002867948965 0 -1.5707963267948966

File: xacro/components/body.xacro (robot description, xacro)
@@ -156,5 +156,5 @@
 	</link>
 	<joint name="body_camera_joint" type="fixed">
-		<origin xyz="0.10065 0.024257 0.28812" rpy="${PI} 0.378684973 0"/>
+		<origin xyz="0.10065 0.024257 0.28812" rpy="${-PI/2-0.378684973} 0 ${-PI/2}"/>
 		<parent link="body_link4"/>
 		<child link="body_camera"/>
@@ -224,5 +224,5 @@
 	</link>
 	<joint name="head_camera_joint" type="fixed">
-		<origin xyz="0.097847  0.046703 0.12364" rpy="${PI} 0.64460396 0"/>
+		<origin xyz="0.097847  0.046703 0.12364" rpy="${-PI/2-0.64460396} 0 ${-PI/2}"/>
 		<parent link="head_link2"/>
 		<child link="head_camera"/>

Commit message: update sensor path

File: urdf/fiveages_w2.urdf (robot description, URDF)
Before this commit: robot FiveAges W2, 45 links, 44 joints
Links:
- link chassis_camera: geometry 
- link fl_lidar: geometry 
- link rr_lidar: geometry 

File: urdf/fiveages_w2_ag2f90.urdf (robot description, URDF)
Before this commit: robot FiveAges W2, 69 links, 68 joints
Links:
- link chassis_camera: geometry 
- link fl_lidar: geometry 
- link rr_lidar: geometry 

File: urdf/fiveages_w2_rg75.urdf (robot description, URDF)
Before this commit: robot FiveAges W2, 57 links, 56 joints
Links:
- link chassis_camera: geometry 
- link fl_lidar: geometry 
- link rr_lidar: geometry 

File: urdf/fiveages_w2_rg75_heavy.urdf (robot description, URDF)
Before this commit: robot FiveAges W2, 57 links, 56 joints
Links:
- link chassis_camera: geometry 
- link fl_lidar: geometry 
- link rr_lidar: geometry 

File: xacro/components/linkhou_s2.xacro (robot description, xacro)
@@ -310,10 +310,10 @@
 			<visual>
 				<geometry>
-					<mesh filename="file://$(find fiveages_w2_description)/meshes/linkhou_s2/lidar.glb"/>
+					<mesh filename="file://$(find sensor_models)/meshes/robosense/airy.glb"/>
 				</geometry>
 			</visual>
 		</link>
 		<joint name="rr_lidar_joint" type="fixed">
-			<origin xyz="0.21412 0.19406 0.32957" rpy="${PI/2.0} -1.309 0"/>
+			<origin xyz="0.221633 0.200715 0.325074" rpy="0 ${PI*15/180} ${PI}"/>
 			<parent link="chassis_base"/>
 			<child link="rr_lidar"/>
@@ -333,10 +333,10 @@
 			<visual>
 				<geometry>
-					<mesh filename="file://$(find fiveages_w2_description)/meshes/linkhou_s2/lidar.glb"/>
+					<mesh filename="file://$(find sensor_models)/meshes/robosense/airy.glb"/>
 				</geometry>
 			</visual>
 		</link>
 		<joint name="fl_lidar_joint" type="fixed">
-			<origin xyz="-0.21412 -0.19406 0.32957" rpy="${PI/2.0} -1.309 3.1416"/>
+			<origin xyz="-0.221633 -0.200715 0.325074" rpy="0 -${PI*15/180} 0"/>
 			<parent link="chassis_base"/>
 			<child link="fl_lidar"/>
@@ -345,10 +345,10 @@
 			<visual>
 				<geometry>
-					<mesh filename="file://$(find fiveages_w2_description)/meshes/linkhou_s2/camera.glb"/>
+					<mesh filename="file://$(find sensor_models)/meshes/linkhou/ds51.glb"/>
 				</geometry>
 			</visual>
 		</link>
 		<joint name="chassis_camera_joint" type="fixed">
-			<origin xyz="-0.3438 -0.00032028 0.159" rpy="0 0 ${PI}"/>
+			<origin xyz="-0.3438 -0.00032028 0.159" rpy="${-PI/2} 0 ${PI/2}"/>
 			<parent link="chassis_base"/>
 			<child link="chassis_camera"/>

Commit message: remove linkhou

File: urdf/fiveages_w2.urdf (robot description, URDF)
Before this commit: robot FiveAges W2, 45 links, 44 joints
Links:
- removed link head_top_camera
- link body_base: geometry visual mesh filename=package://fiveages_w2_common_description/meshes/body/base.g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
- link body_link1: geometry collision box size=0.15 0.145 0.48; visual mesh filename=package://fiveages_w2_common_description/meshes/body/link1.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
- link body_link2: geometry collision box size=0.16 0.2 0.5; visual mesh filename=package://fiveages_w2_common_description/meshes/body/link2.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
- link body_link3: geometry collision box size=0.13 0.13 0.22; visual mesh filename=package://fiveages_w2_common_description/meshes/body/link3.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
- link body_link4: geometry collision box size=0.2000 0.32 0.5029; visual mesh filename=package://fiveages_w2_common_description/meshes/body/link4.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
- link chassis_base: geometry collision box size=0.5 0.3 0.2; collision box size=0.66 0.16 0.3
- link fl_steer: geometry visual mesh filename=package://fiveages_w2_common_description/meshes/linkhou_s2/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
- link fl_wheel: geometry collision cylinder length=0.046 radius=0.07; visual mesh filename=package://fiveages_w2_common_description/meshes/linkhou_s2/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
- link fr_steer: geometry visual mesh filename=package://fiveages_w2_common_description/meshes/linkhou_s2/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 scale=1 -1 1
- link fr_wheel: geometry collision cylinder length=0.046 radius=0.07; visual mesh filename=package://fiveages_w2_common_description/meshes/linkhou_s2/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 scale=1 -1 1
- link head_link1: geometry visual mesh filename=package://fiveages_w2_common_description/meshes/head/head_y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
- link head_link2: geometry collision box size=0.15 0.16 0.24; visual mesh filename=package://fiveages_w2_common_description/meshes/head/head_p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
- link rl_steer: geometry visual mesh filename=package://fiveages_w2_common_description/meshes/linkhou_s2/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
- link rl_wheel: geometry collision cylinder length=0.046 radius=0.07; visual mesh filename=package://fiveages_w2_common_description/meshes/linkhou_s2/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
- link rr_steer: geometry visual mesh filename=package://fiveages_w2_common_description/meshes/linkhou_s2/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 scale=1 -1 1
- link rr_wheel: geometry collision cylinder length=0.046 radius=0.07; visual mesh filename=package://fiveages_w2_common_description/meshes/linkhou_s2/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 scale=1 -1 1
Joints:
- removed joint head_top_camera_joint

File: urdf/fiveages_w2_ag2f90.urdf (robot description, URDF)
Before this commit: robot FiveAges W2, 69 links, 68 joints
Links:
- removed link head_top_camera
- link body_base: geometry visual mesh filename=package://fiveages_w2_common_description/meshes/body/base.g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
- link body_link1: geometry collision box size=0.15 0.145 0.48; visual mesh filename=package://fiveages_w2_common_description/meshes/body/link1.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
- link body_link2: geometry collision box size=0.16 0.2 0.5; visual mesh filename=package://fiveages_w2_common_description/meshes/body/link2.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
- link body_link3: geometry collision box size=0.13 0.13 0.22; visual mesh filename=package://fiveages_w2_common_description/meshes/body/link3.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
- link body_link4: geometry collision box size=0.2000 0.32 0.5029; visual mesh filename=package://fiveages_w2_common_description/meshes/body/link4.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
- link chassis_base: geometry collision box size=0.5 0.3 0.2; collision box size=0.66 0.16 0.3
- link fl_steer: geometry visual mesh filename=package://fiveages_w2_common_description/meshes/linkhou_s2/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
- link fl_wheel: geometry collision cylinder length=0.046 radius=0.07; visual mesh filename=package://fiveages_w2_common_description/meshes/linkhou_s2/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
- link fr_steer: geometry visual mesh filename=package://fiveages_w2_common_description/meshes/linkhou_s2/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 scale=1 -1 1
- link fr_wheel: geometry collision cylinder length=0.046 radius=0.07; visual mesh filename=package://fiveages_w2_common_description/meshes/linkhou_s2/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 scale=1 -1 1
- link head_link1: geometry visual mesh filename=package://fiveages_w2_common_description/meshes/head/head_y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
- link head_link2: geometry collision box size=0.15 0.16 0.24; visual mesh filename=package://fiveages_w2_common_description/meshes/head/head_p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
- link rl_steer: geometry visual mesh filename=package://fiveages_w2_common_description/meshes/linkhou_s2/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
- link rl_wheel: geometry collision cylinder length=0.046 radius=0.07; visual mesh filename=package://fiveages_w2_common_description/meshes/linkhou_s2/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
- link rr_steer: geometry visual mesh filename=package://fiveages_w2_common_description/meshes/linkhou_s2/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 scale=1 -1 1
- link rr_wheel: geometry collision cylinder length=0.046 radius=0.07; visual mesh filename=package://fiveages_w2_common_description/meshes/linkhou_s2/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 scale=1 -1 1
Joints:
- removed joint head_top_camera_joint

File: urdf/fiveages_w2_rg75.urdf (robot description, URDF)
Before this commit: robot FiveAges W2, 57 links, 56 joints
Links:
- removed link head_top_camera
- link body_base: geometry visual mesh filename=package://fiveages_w2_common_description/meshes/body/base.g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
- link body_link1: geometry collision box size=0.15 0.145 0.48; visual mesh filename=package://fiveages_w2_common_description/meshes/body/link1.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
- link body_link2: geometry collision box size=0.16 0.2 0.5; visual mesh filename=package://fiveages_w2_common_description/meshes/body/link2.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
- link body_link3: geometry collision box size=0.13 0.13 0.22; visual mesh filename=package://fiveages_w2_common_description/meshes/body/link3.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
- link body_link4: geometry collision box size=0.2000 0.32 0.5029; visual mesh filename=package://fiveages_w2_common_description/meshes/body/link4.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
- link chassis_base: geometry collision box size=0.5 0.3 0.2; collision box size=0.66 0.16 0.3
- link fl_steer: geometry visual mesh filename=package://fiveages_w2_common_description/meshes/linkhou_s2/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
- link fl_wheel: geometry collision cylinder length=0.046 radius=0.07; visual mesh filename=package://fiveages_w2_common_description/meshes/linkhou_s2/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
- link fr_steer: geometry visual mesh filename=package://fiveages_w2_common_description/meshes/linkhou_s2/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 scale=1 -1 1
- link fr_wheel: geometry collision cylinder length=0.046 radius=0.07; visual mesh filename=package://fiveages_w2_common_description/meshes/linkhou_s2/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 scale=1 -1 1
- link head_link1: geometry visual mesh filename=package://fiveages_w2_common_description/meshes/head/head_y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
- link head_link2: geometry collision box size=0.15 0.16 0.24; visual mesh filename=package://fiveages_w2_common_description/meshes/head/head_p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
- link rl_steer: geometry visual mesh filename=package://fiveages_w2_common_description/meshes/linkhou_s2/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
- link rl_wheel: geometry collision cylinder length=0.046 radius=0.07; visual mesh filename=package://fiveages_w2_common_description/meshes/linkhou_s2/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
- link rr_steer: geometry visual mesh filename=package://fiveages_w2_common_description/meshes/linkhou_s2/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 scale=1 -1 1
- link rr_wheel: geometry collision cylinder length=0.046 radius=0.07; visual mesh filename=package://fiveages_w2_common_description/meshes/linkhou_s2/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 scale=1 -1 1
Joints:
- removed joint head_top_camera_joint

File: urdf/fiveages_w2_rg75_heavy.urdf (robot description, URDF)
Before this commit: robot FiveAges W2, 57 links, 56 joints
Links:
- removed link head_top_camera
- link body_base: geometry visual mesh filename=package://fiveages_w2_common_description/meshes/body/base.g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
- link body_link1: geometry collision box size=0.15 0.145 0.48; visual mesh filename=package://fiveages_w2_common_description/meshes/body/link1.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
- link body_link2: geometry collision box size=0.16 0.2 0.5; visual mesh filename=package://fiveages_w2_common_description/meshes/body/link2.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
- link body_link3: geometry collision box size=0.13 0.13 0.22; visual mesh filename=package://fiveages_w2_common_description/meshes/body/link3.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
- link body_link4: geometry collision box size=0.2000 0.32 0.5029; visual mesh filename=package://fiveages_w2_common_description/meshes/body/link4.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
- link chassis_base: geometry collision box size=0.5 0.3 0.2; collision box size=0.66 0.16 0.3
- link fl_steer: geometry visual mesh filename=package://fiveages_w2_common_description/meshes/linkhou_s2/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
- link fl_wheel: geometry collision cylinder length=0.046 radius=0.07; visual mesh filename=package://fiveages_w2_common_description/meshes/linkhou_s2/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
- link fr_steer: geometry visual mesh filename=package://fiveages_w2_common_description/meshes/linkhou_s2/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 scale=1 -1 1
- link fr_wheel: geometry collision cylinder length=0.046 radius=0.07; visual mesh filename=package://fiveages_w2_common_description/meshes/linkhou_s2/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 scale=1 -1 1
- link head_link1: geometry visual mesh filename=package://fiveages_w2_common_description/meshes/head/head_y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
- link head_link2: geometry collision box size=0.15 0.16 0.24; visual mesh filename=package://fiveages_w2_common_description/meshes/head/head_p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
- link rl_steer: geometry visual mesh filename=package://fiveages_w2_common_description/meshes/linkhou_s2/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
- link rl_wheel: geometry collision cylinder length=0.046 radius=0.07; visual mesh filename=package://fiveages_w2_common_description/meshes/linkhou_s2/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
- link rr_steer: geometry visual mesh filename=package://fiveages_w2_common_description/meshes/linkhou_s2/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 scale=1 -1 1
- link rr_wheel: geometry collision cylinder length=0.046 radius=0.07; visual mesh filename=package://fiveages_w2_common_description/meshes/linkhou_s2/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 scale=1 -1 1
Joints:
- removed joint head_top_camera_joint

File: xacro/component.xacro (robot description, xacro)
@@ -2,14 +2,5 @@
 <robot name="FiveAges W2" xmlns:xacro="http://www.ros.org/wiki/xacro">
 	<xacro:property name="PI" value="3.1415926535897931"/>
-	<xacro:arg name="type" default="linkhou_s2"/>
-	<xacro:arg name="chassis_joints_movable" default="true"/>
-	<xacro:if value="${'$(arg type)' == 'linkhou_s2'}">
-		<xacro:include filename="$(find fiveages_w2_description)/xacro/components/linkhou_s2.xacro"/>
-		<xacro:linkhou_s2 joints_movable="$(arg chassis_joints_movable)"/>
-	</xacro:if>
-	<xacro:if value="${'$(arg type)' == 'body'}">
-		<link name="base_link"/>
-		<xacro:include filename="$(find fiveages_body_description)/xacro/body.xacro"/>
-	</xacro:if>
+	<xacro:arg name="type" default="arms"/>
 	<xacro:if value="${'$(arg type)' == 'arms'}">
 		<link name="arm_base"/>

File: xacro/robot.xacro (robot description, xacro)
@@ -1,6 +1,7 @@
 <?xml version="1.0"?>
 <robot name="FiveAges W2" xmlns:xacro="http://www.ros.org/wiki/xacro">
-    <xacro:arg name="collider" default="convex"/>
+    <xacro:arg name="collider" default="simple"/>
     <xacro:arg name="chassis_joints_movable" default="false"/>
+    <xacro:arg name="variant" default=""/>
     <!-- 从 type 参数解析出 hand_type 和 gripper_type -->
     <xacro:arg name="type" default=""/>
@@ -38,7 +39,10 @@
         <xacro:property name="selected_hand_type" value="linkerhand_o7"/>
     </xacro:if>
-    <xacro:include filename="$(find fiveages_w2_description)/xacro/components/linkhou_s2.xacro"/>
-    <xacro:linkhou_s2 joints_movable="$(arg chassis_joints_movable)"/>
-    <xacro:include filename="$(find fiveages_body_description)/xacro/body.xacro"/>
+    <xacro:include filename="$(find fiveages_w2_common_description)/xacro/components/linkhou_s2.xacro"/>
+    <xacro:linkhou_s2 joints_movable="$(arg chassis_joints_movable)" variant="$(arg variant)"/>
+    <xacro:include filename="$(find fiveages_w2_common_description)/xacro/components/body.xacro"/>
+    <xacro:body variant="$(arg variant)"/>
+    <xacro:include filename="$(find fiveages_w2_common_description)/xacro/components/head.xacro"/>
+    <xacro:head variant="$(arg variant)"/>
     <!-- Left Arm -->
     <joint name="left_arm_base_joint" type="fixed">

File: xacro/ros2_control/robot.xacro (robot description, xacro)
@@ -6,5 +6,5 @@
 	<xacro:include filename="$(find fiveages_w2_description)/xacro/robot.xacro"/>
 	<xacro:include filename="$(find m6_ccs_description)/xacro/ros2_control/interfaces.xacro"/>
-	<xacro:include filename="$(find fiveages_body_description)/xacro/ros2_control/body.xacro"/>
+	<xacro:include filename="$(find fiveages_w2_common_description)/xacro/ros2_control/body.xacro"/>
 	<xacro:if value="${is_real_hardware}">
 		<!-- 确定传递给 marvin_ros2_control 的 gripper_type 参数 -->
