Commit message: add nav2 config

File: xacro/components/linkhou_s2.xacro (robot description, xacro)
@@ -315,5 +315,5 @@
 		</link>
 		<joint name="rr_lidar_joint" type="fixed">
-			<origin xyz="0.221633 0.200715 0.325074" rpy="0 ${PI*15/180} ${PI}"/>
+			<origin xyz="0.221633 0.200715 0.325074" rpy="0 -${PI*15/180} ${PI}"/>
 			<parent link="chassis_base"/>
 			<child link="rr_lidar"/>

Commit message: Feature/ocs2 wbc bodytest (#5)
* ocs2 wbc config

* update sensor path

* add nav2 config

* add nav2 config

* update german poc nav

* update

* wbc rg75

* update

* update

* 使用full_body.launch.py强制rviz fixed frame为world

* 抬版本号

---------

Co-authored-by: Huang Zhenbiao <biao876990970@hotmail.com>

File: xacro/components/linkhou_s2.xacro (robot description, xacro)
@@ -310,10 +310,10 @@
 			<visual>
 				<geometry>
-					<mesh filename="file://$(find fiveages_w2_description)/meshes/linkhou_s2/lidar.glb"/>
+					<mesh filename="file://$(find sensor_models)/meshes/robosense/airy.glb"/>
 				</geometry>
 			</visual>
 		</link>
 		<joint name="rr_lidar_joint" type="fixed">
-			<origin xyz="0.21412 0.19406 0.32957" rpy="${PI/2.0} -1.309 0"/>
+			<origin xyz="0.221633 0.200715 0.325074" rpy="0 -${PI*15/180} ${PI}"/>
 			<parent link="chassis_base"/>
 			<child link="rr_lidar"/>
@@ -333,10 +333,10 @@
 			<visual>
 				<geometry>
-					<mesh filename="file://$(find fiveages_w2_description)/meshes/linkhou_s2/lidar.glb"/>
+					<mesh filename="file://$(find sensor_models)/meshes/robosense/airy.glb"/>
 				</geometry>
 			</visual>
 		</link>
 		<joint name="fl_lidar_joint" type="fixed">
-			<origin xyz="-0.21412 -0.19406 0.32957" rpy="${PI/2.0} -1.309 3.1416"/>
+			<origin xyz="-0.221633 -0.200715 0.325074" rpy="0 -${PI*15/180} 0"/>
 			<parent link="chassis_base"/>
 			<child link="fl_lidar"/>
@@ -345,10 +345,10 @@
 			<visual>
 				<geometry>
-					<mesh filename="file://$(find fiveages_w2_description)/meshes/linkhou_s2/camera.glb"/>
+					<mesh filename="file://$(find sensor_models)/meshes/linkhou/ds51.glb"/>
 				</geometry>
 			</visual>
 		</link>
 		<joint name="chassis_camera_joint" type="fixed">
-			<origin xyz="-0.3438 -0.00032028 0.159" rpy="0 0 ${PI}"/>
+			<origin xyz="-0.3438 -0.00032028 0.159" rpy="${-PI/2} 0 ${PI/2}"/>
 			<parent link="chassis_base"/>
 			<child link="chassis_camera"/>
