Commit message: Update xacro file to support marvin 485 communication

File: xacro/ros2_control/robot.xacro (robot description, xacro)
@@ -4,21 +4,14 @@
 	<xacro:arg name="device_ip" default="192.168.1.190"/>
 	<xacro:property name="device_ip_arg" value="$(arg device_ip)"/>
+	<xacro:property name="ros2_control_hardware_type_arg" value="$(arg ros2_control_hardware_type)"/>
 	<xacro:include filename="$(find fiveages_w2_description)/xacro/robot.xacro"/>
 	<xacro:include filename="$(find m6_ccs_description)/xacro/ros2_control/interfaces.xacro"/>
 	<xacro:include filename="$(find fiveages_w2_description)/xacro/ros2_control/body.xacro"/>
-	<!-- 宏：创建单个 modbus 灵巧手系统（USB 模式） -->
-	<xacro:macro name="create_modbus_hand_single" params="hand_type system_suffix side serial_port">
-		<ros2_control name="linkerhand_${system_suffix}_${side}_system" type="system">
-			<hardware>
-				<plugin>modbus_ros2_control/DexterousHandHardware</plugin>
-				<param name="serial_port">${serial_port}</param>
-				<param name="hand_type">${hand_type}</param>
-				<param name="hand_side">${side}</param>
-				<param name="max_speed_ratio">1.0</param>
-			</hardware>
-			<xacro:insert_block/>
-		</ros2_control>
-	</xacro:macro>
-	<xacro:if value="${'$(arg ros2_control_hardware_type)' == 'real'}">
+	<!-- quick_start.sh uses hardware:=real (485/marvin) and hardware:=real_usb (USB/modbus hand).
+	     Treat both as "real" branches, but force USB hand mode when hardware==real_usb. -->
+	<xacro:if value="${ros2_control_hardware_type_arg == 'real_usb'}">
+		<xacro:property name="hand_control_mode_arg" value="usb"/>
+	</xacro:if>
+	<xacro:if value="${ros2_control_hardware_type_arg == 'real' or ros2_control_hardware_type_arg == 'real_usb'}">
 		<!-- 确定传递给 marvin_ros2_control 的 gripper_type 参数 -->
 		<!--
@@ -98,38 +91,66 @@
 			<xacro:body_interfaces/>
 		</ros2_control>
-		<!-- 灵巧手接口：USB 模式（modbus_ros2_control） -->
+		<!-- 灵巧手接口：USB 模式（modbus_ros2_control），直接内联 ros2_control 配置 -->
 		<xacro:if value="${selected_hand_type != '' and hand_control_mode_arg == 'usb'}">
 			<!-- O6/L6: 6-DOF 手 -->
 			<xacro:if value="${selected_hand_type == 'linkerhand_o6' or selected_hand_type == 'linkerhand_l6'}">
 				<xacro:include filename="$(find linkerhand_description)/xacro/ros2_control/o6.xacro"/>
-				<xacro:create_modbus_hand_single hand_type="${selected_hand_type}" system_suffix="6" side="left" serial_port="/dev/ttyUSB1">
+				<ros2_control name="linkerhand_6_left_system" type="system">
+					<hardware>
+						<plugin>modbus_ros2_control/DexterousHandHardware</plugin>
+						<param name="serial_port">/dev/ttyUSB1</param>
+						<param name="hand_type">${selected_hand_type}</param>
+						<param name="hand_side">left</param>
+						<param name="max_speed_ratio">1.0</param>
+					</hardware>
 					<xacro:linkerhand_o6_interfaces name="left_hand"/>
-				</xacro:create_modbus_hand_single>
-				<xacro:create_modbus_hand_single hand_type="${selected_hand_type}" system_suffix="6" side="right" serial_port="/dev/ttyUSB0">
+				</ros2_control>
+				<ros2_control name="linkerhand_6_right_system" type="system">
+					<hardware>
+						<plugin>modbus_ros2_control/DexterousHandHardware</plugin>
+						<param name="serial_port">/dev/ttyUSB0</param>
+						<param name="hand_type">${selected_hand_type}</param>
+						<param name="hand_side">right</param>
+						<param name="max_speed_ratio">1.0</param>
+					</hardware>
 					<xacro:linkerhand_o6_interfaces name="right_hand"/>
-				</xacro:create_modbus_hand_single>
+				</ros2_control>
 			</xacro:if>
 			<!-- O7: 7-DOF 手 -->
 			<xacro:if value="${selected_hand_type == 'linkerhand_o7'}">
 				<xacro:include filename="$(find linkerhand_description)/xacro/ros2_control/o7.xacro"/>
-				<xacro:create_modbus_hand_single hand_type="${selected_hand_type}" system_suffix="7" side="left" serial_port="/dev/ttyUSB1">
+				<ros2_control name="linkerhand_7_left_system" type="system">
+					<hardware>
+						<plugin>modbus_ros2_control/DexterousHandHardware</plugin>
+						<param name="serial_port">/dev/ttyUSB1</param>
+						<param name="hand_type">${selected_hand_type}</param>
+						<param name="hand_side">left</param>
+						<param name="max_speed_ratio">1.0</param>
+					</hardware>
 					<xacro:linkerhand_o7_interfaces name="left_hand"/>
-				</xacro:create_modbus_hand_single>
-				<xacro:create_modbus_hand_single hand_type="${selected_hand_type}" system_suffix="7" side="right" serial_port="/dev/ttyUSB0">
+				</ros2_control>
+				<ros2_control name="linkerhand_7_right_system" type="system">
+					<hardware>
+						<plugin>modbus_ros2_control/DexterousHandHardware</plugin>
+						<param name="serial_port">/dev/ttyUSB0</param>
+						<param name="hand_type">${selected_hand_type}</param>
+						<param name="hand_side">right</param>
+						<param name="max_speed_ratio">1.0</param>
+					</hardware>
 					<xacro:linkerhand_o7_interfaces name="right_hand"/>
-				</xacro:create_modbus_hand_single>
+				</ros2_control>
 			</xacro:if>
 		</xacro:if>
 	</xacro:if>
-	<xacro:unless value="${'$(arg ros2_control_hardware_type)' == 'real'}">
+	<xacro:unless value="${ros2_control_hardware_type_arg == 'real' or ros2_control_hardware_type_arg == 'real_usb'}">
 		<ros2_control name="fiveages_w2_system" type="system">
 			<hardware>
-				<xacro:if value="${'$(arg ros2_control_hardware_type)' == 'gz'}">
+				<xacro:if value="${ros2_control_hardware_type_arg == 'gz'}">
 					<plugin>gz_ros2_control/GazeboSimSystem</plugin>
 				</xacro:if>
-				<xacro:if value="${'$(arg ros2_control_hardware_type)' == 'mock_components'}">
+				<xacro:if value="${ros2_control_hardware_type_arg == 'mock_components'}">
 					<plugin>mock_components/GenericSystem</plugin>
 				</xacro:if>
-				<xacro:if value="${'$(arg ros2_control_hardware_type)' == 'isaac'}">
+				<xacro:if value="${ros2_control_hardware_type_arg == 'isaac'}">
 					<plugin>topic_based_ros2_control/TopicBasedSystem</plugin>
 					<param name="joint_commands_topic">/isaac/joint_command</param>
@@ -158,9 +179,4 @@
 				<xacro:linkerhand_o6_interfaces name="left_hand"/>
 				<xacro:linkerhand_o6_interfaces name="right_hand"/>
-			</xacro:if>
-			<xacro:if value="${selected_hand_type == 'linkerhand_o7'}">
-				<xacro:include filename="$(find linkerhand_description)/xacro/ros2_control/o7.xacro"/>
-				<xacro:linkerhand_o7_interfaces name="left_hand"/>
-				<xacro:linkerhand_o7_interfaces name="right_hand"/>
 			</xacro:if>
 			<xacro:if value="${selected_hand_type == 'linkerhand_o7'}">

Commit message: fix xacro hand usb interface selection
Normalize usb hand series comparisons to string values so o6/o7 interface macros are expanded reliably in real_usb mode.

Made-with: Cursor

File: xacro/ros2_control/robot.xacro (robot description, xacro)
@@ -80,9 +80,9 @@
 		<xacro:if value="${ee_drive_type == 'usb'}">
 			<xacro:if value="${selected_hand_type in ('linkerhand_o6', 'linkerhand_l6', 'linkerhand_o7')}">
-				<xacro:property name="usb_hand_series" value="${'7' if selected_hand_type == 'linkerhand_o7' else '6'}"/>
-				<xacro:if value="${usb_hand_series == '6'}">
+				<xacro:property name="usb_hand_series" value="${str('7' if selected_hand_type == 'linkerhand_o7' else '6')}"/>
+				<xacro:if value="${str(usb_hand_series) == '6'}">
 					<xacro:include filename="$(find linkerhand_description)/xacro/ros2_control/o6.xacro"/>
 				</xacro:if>
-				<xacro:if value="${usb_hand_series == '7'}">
+				<xacro:if value="${str(usb_hand_series) == '7'}">
 					<xacro:include filename="$(find linkerhand_description)/xacro/ros2_control/o7.xacro"/>
 				</xacro:if>
@@ -90,13 +90,13 @@
 					<hardware>
 						<plugin>modbus_ros2_control/DexterousHandHardware</plugin>
-						<param name="serial_port">/dev/ttyUSB1</param>
+						<param name="serial_port">/dev/ttyUSB0</param>
 						<param name="hand_type">${selected_hand_type}</param>
 						<param name="hand_side">left</param>
 						<param name="max_speed_ratio">1.0</param>
 					</hardware>
-					<xacro:if value="${usb_hand_series == '6'}">
+					<xacro:if value="${str(usb_hand_series) == '6'}">
 						<xacro:linkerhand_o6_interfaces name="left_hand"/>
 					</xacro:if>
-					<xacro:if value="${usb_hand_series == '7'}">
+					<xacro:if value="${str(usb_hand_series) == '7'}">
 						<xacro:linkerhand_o7_interfaces name="left_hand"/>
 					</xacro:if>
@@ -105,13 +105,13 @@
 					<hardware>
 						<plugin>modbus_ros2_control/DexterousHandHardware</plugin>
-						<param name="serial_port">/dev/ttyUSB0</param>
+						<param name="serial_port">/dev/ttyUSB2</param>
 						<param name="hand_type">${selected_hand_type}</param>
 						<param name="hand_side">right</param>
 						<param name="max_speed_ratio">1.0</param>
 					</hardware>
-					<xacro:if value="${usb_hand_series == '6'}">
+					<xacro:if value="${str(usb_hand_series) == '6'}">
 						<xacro:linkerhand_o6_interfaces name="right_hand"/>
 					</xacro:if>
-					<xacro:if value="${usb_hand_series == '7'}">
+					<xacro:if value="${str(usb_hand_series) == '7'}">
 						<xacro:linkerhand_o7_interfaces name="right_hand"/>
 					</xacro:if>

Commit message: Add configuration files for freedom and inspire robot descriptions

File: xacro/ros2_control/robot.xacro (robot description, xacro)
@@ -15,4 +15,6 @@
 	<xacro:include filename="$(find linkerhand_description)/xacro/ros2_control/o6.xacro"/>
 	<xacro:include filename="$(find linkerhand_description)/xacro/ros2_control/o7.xacro"/>
+	<xacro:include filename="$(find freedom_description)/xacro/ros2_control/freedom.xacro"/>
+	<xacro:include filename="$(find inspire_description)/xacro/ros2_control/RH56E2.xacro"/>
 	<xacro:macro name="side_gripper_joint" params="side">
 		<joint name="${side}_gripper_joint">
@@ -36,8 +38,14 @@
 			<xacro:linkerhand_o7_interfaces name="${side}_hand"/>
 		</xacro:if>
+		<xacro:if value="${hand_type == 'freedom_v1' or hand_type == 'freedom-v1'}">
+			<xacro:freedom_interfaces name="${side}_hand"/>
+		</xacro:if>
+		<xacro:if value="${hand_type == 'inspire_e2' or hand_type == 'inspire-e2'}">
+			<xacro:inspire_rh56e2_interfaces name="${side}_hand"/>
+		</xacro:if>
 	</xacro:macro>
 	<xacro:macro name="side_usb_hand_system" params="side hand_type serial_port">
-		<xacro:property name="usb_hand_series" value="${str('7' if hand_type == 'linkerhand_o7' else '6')}"/>
-		<ros2_control name="linkerhand_${usb_hand_series}_${side}_system" type="system">
+		<xacro:property name="usb_hand_system_name" value="${str('linkerhand_7' if hand_type == 'linkerhand_o7' else ('inspire_e2' if hand_type in ('inspire_e2', 'inspire-e2') else 'linkerhand_6'))}"/>
+		<ros2_control name="${usb_hand_system_name}_${side}_system" type="system">
 			<hardware>
 				<plugin>modbus_ros2_control/DexterousHandHardware</plugin>
@@ -48,4 +56,18 @@
 			</hardware>
 			<xacro:side_hand_interfaces side="${side}" hand_type="${hand_type}"/>
+		</ros2_control>
+	</xacro:macro>
+	<xacro:macro name="side_freedom_usb_hand_system" params="side serial_port">
+		<ros2_control name="freedom_v1_${side}_system" type="system">
+			<hardware>
+				<plugin>modbus_ros2_control/FreedomRS485Hardware</plugin>
+				<param name="serial_port">${serial_port}</param>
+				<param name="hand_side">${side}</param>
+				<param name="slave_id">auto</param>
+				<param name="baudrate">115200</param>
+				<param name="read_feedback">true</param>
+				<param name="feedback_timeout_ms">20</param>
+			</hardware>
+			<xacro:freedom_interfaces name="${side}_hand"/>
 		</ros2_control>
 	</xacro:macro>
@@ -95,9 +117,15 @@
 		</ros2_control>
 		<xacro:if value="${ee_drive_type == 'usb'}">
-			<xacro:if value="${left_hand_type in ('linkerhand_o6', 'linkerhand_l6', 'linkerhand_o7')}">
+			<xacro:if value="${left_hand_type in ('linkerhand_o6', 'linkerhand_l6', 'linkerhand_o7', 'inspire_e2', 'inspire-e2')}">
 				<xacro:side_usb_hand_system side="left" hand_type="${left_hand_type}" serial_port="/dev/ttyUSB0"/>
 			</xacro:if>
-			<xacro:if value="${right_hand_type in ('linkerhand_o6', 'linkerhand_l6', 'linkerhand_o7')}">
+			<xacro:if value="${right_hand_type in ('linkerhand_o6', 'linkerhand_l6', 'linkerhand_o7', 'inspire_e2', 'inspire-e2')}">
 				<xacro:side_usb_hand_system side="right" hand_type="${right_hand_type}" serial_port="/dev/ttyUSB2"/>
+			</xacro:if>
+			<xacro:if value="${left_hand_type in ('freedom_v1', 'freedom-v1')}">
+				<xacro:side_freedom_usb_hand_system side="left" serial_port="/dev/ttyUSB0"/>
+			</xacro:if>
+			<xacro:if value="${right_hand_type in ('freedom_v1', 'freedom-v1')}">
+				<xacro:side_freedom_usb_hand_system side="right" serial_port="/dev/ttyUSB2"/>
 			</xacro:if>
 		</xacro:if>

Commit message: Add can_ros2_control dependency and enhance robot.xacro for drive type handling

File: xacro/ros2_control/robot.xacro (robot description, xacro)
@@ -3,6 +3,10 @@
 	<xacro:arg name="ros2_control_hardware_type" default="mock_components"/>
 	<xacro:arg name="arm_ctrl_mode" default="position"/>
+	<xacro:arg name="left_ee_drive_type" default=""/>
+	<xacro:arg name="right_ee_drive_type" default=""/>
 	<xacro:property name="is_real_hardware" value="${'$(arg ros2_control_hardware_type)' == 'real' or '$(arg ros2_control_hardware_type)' == 'real_usb'}"/>
 	<xacro:property name="ee_drive_type" value="${'usb' if '$(arg ros2_control_hardware_type)' == 'real_usb' else ('marvin' if '$(arg ros2_control_hardware_type)' == 'real' else '')}"/>
+	<xacro:property name="left_drive_type" value="${'$(arg left_ee_drive_type)' if '$(arg left_ee_drive_type)' != '' else ee_drive_type}"/>
+	<xacro:property name="right_drive_type" value="${'$(arg right_ee_drive_type)' if '$(arg right_ee_drive_type)' != '' else ee_drive_type}"/>
 	<xacro:property name="arm_ctrl_mode_value" value="$(arg arm_ctrl_mode)"/>
 	<xacro:property name="left_ee_type" value="${left_hand_type if left_hand_type != '' else left_gripper_type}"/>
@@ -72,4 +76,16 @@
 		</ros2_control>
 	</xacro:macro>
+	<xacro:macro name="side_freedom_usb_can_hand_system" params="side can_interface device_id">
+		<ros2_control name="freedom_v1_${side}_can_system" type="system">
+			<hardware>
+				<plugin>can_ros2_control/FreedomCanHardware</plugin>
+				<param name="can_interface">${can_interface}</param>
+				<param name="device_id">${device_id}</param>
+				<param name="read_feedback">true</param>
+				<param name="feedback_timeout_ms">1</param>
+			</hardware>
+			<xacro:freedom_interfaces name="${side}_hand"/>
+		</ros2_control>
+	</xacro:macro>
 	<xacro:if value="${is_real_hardware}">
 		<ros2_control name="M6_CCS_System" type="system">
@@ -78,9 +94,15 @@
 				<param name="arm_type">dual</param>
 				<param name="ctrl_mode">${arm_ctrl_mode_value}</param>
-				<xacro:if value="${ee_drive_type == 'marvin' and left_ee_type != ''}">
+				<xacro:if value="${(left_drive_type == 'marvin' or left_drive_type == 'tianji_can') and left_ee_type != ''}">
 					<param name="left_ee_type">${left_ee_type}</param>
-				</xacro:if>
-				<xacro:if value="${ee_drive_type == 'marvin' and right_ee_type != ''}">
+					<xacro:if value="${left_drive_type == 'tianji_can'}">
+						<param name="left_ee_channel">1</param>
+					</xacro:if>
+				</xacro:if>
+				<xacro:if value="${(right_drive_type == 'marvin' or right_drive_type == 'tianji_can') and right_ee_type != ''}">
 					<param name="right_ee_type">${right_ee_type}</param>
+					<xacro:if value="${right_drive_type == 'tianji_can'}">
+						<param name="right_ee_channel">1</param>
+					</xacro:if>
 				</xacro:if>
 				<param name="max_joint_speed">50</param>
@@ -98,9 +120,9 @@
 				<xacro:side_gripper_joint side="right"/>
 			</xacro:if>
-			<xacro:if value="${ee_drive_type == 'marvin'}">
-				<xacro:if value="${left_hand_type != ''}">
+			<xacro:if value="${left_drive_type == 'marvin' or right_drive_type == 'marvin' or left_drive_type == 'tianji_can' or right_drive_type == 'tianji_can'}">
+				<xacro:if value="${(left_drive_type == 'marvin' or left_drive_type == 'tianji_can') and left_hand_type != ''}">
 					<xacro:side_hand_interfaces side="left" hand_type="${left_hand_type}"/>
 				</xacro:if>
-				<xacro:if value="${right_hand_type != ''}">
+				<xacro:if value="${(right_drive_type == 'marvin' or right_drive_type == 'tianji_can') and right_hand_type != ''}">
 					<xacro:side_hand_interfaces side="right" hand_type="${right_hand_type}"/>
 				</xacro:if>
@@ -116,16 +138,22 @@
 			<xacro:body_interfaces/>
 		</ros2_control>
-		<xacro:if value="${ee_drive_type == 'usb'}">
-			<xacro:if value="${left_hand_type in ('linkerhand_o6', 'linkerhand_l6', 'linkerhand_o7', 'inspire_e2', 'inspire-e2')}">
+		<xacro:if value="${left_drive_type == 'usb' or right_drive_type == 'usb' or left_drive_type == 'usb_can' or right_drive_type == 'usb_can'}">
+			<xacro:if value="${left_drive_type == 'usb' and left_hand_type in ('linkerhand_o6', 'linkerhand_l6', 'linkerhand_o7', 'inspire_e2', 'inspire-e2')}">
 				<xacro:side_usb_hand_system side="left" hand_type="${left_hand_type}" serial_port="/dev/ttyUSB0"/>
 			</xacro:if>
-			<xacro:if value="${right_hand_type in ('linkerhand_o6', 'linkerhand_l6', 'linkerhand_o7', 'inspire_e2', 'inspire-e2')}">
+			<xacro:if value="${right_drive_type == 'usb' and right_hand_type in ('linkerhand_o6', 'linkerhand_l6', 'linkerhand_o7', 'inspire_e2', 'inspire-e2')}">
 				<xacro:side_usb_hand_system side="right" hand_type="${right_hand_type}" serial_port="/dev/ttyUSB2"/>
 			</xacro:if>
-			<xacro:if value="${left_hand_type in ('freedom_v1', 'freedom-v1')}">
+			<xacro:if value="${left_drive_type == 'usb' and left_hand_type in ('freedom_v1', 'freedom-v1')}">
 				<xacro:side_freedom_usb_hand_system side="left" serial_port="/dev/ttyUSB0"/>
 			</xacro:if>
-			<xacro:if value="${right_hand_type in ('freedom_v1', 'freedom-v1')}">
+			<xacro:if value="${right_drive_type == 'usb' and right_hand_type in ('freedom_v1', 'freedom-v1')}">
 				<xacro:side_freedom_usb_hand_system side="right" serial_port="/dev/ttyUSB2"/>
+			</xacro:if>
+			<xacro:if value="${left_drive_type == 'usb_can' and left_hand_type in ('freedom_v1', 'freedom-v1')}">
+				<xacro:side_freedom_usb_can_hand_system side="left" can_interface="can0" device_id="0"/>
+			</xacro:if>
+			<xacro:if value="${right_drive_type == 'usb_can' and right_hand_type in ('freedom_v1', 'freedom-v1')}">
+				<xacro:side_freedom_usb_can_hand_system side="right" can_interface="can1" device_id="1"/>
 			</xacro:if>
 		</xacro:if>

Commit message: 规范freedom xacro

File: xacro/ros2_control/robot.xacro (robot description, xacro)
@@ -42,13 +42,13 @@
 			<xacro:linkerhand_o7_interfaces name="${side}_hand"/>
 		</xacro:if>
-		<xacro:if value="${hand_type == 'freedom_v1' or hand_type == 'freedom-v1'}">
+		<xacro:if value="${hand_type == 'freedom_v1'}">
 			<xacro:freedom_interfaces name="${side}_hand"/>
 		</xacro:if>
-		<xacro:if value="${hand_type == 'inspire_e2' or hand_type == 'inspire-e2'}">
+		<xacro:if value="${hand_type == 'inspire_e2'}">
 			<xacro:inspire_rh56e2_interfaces name="${side}_hand"/>
 		</xacro:if>
 	</xacro:macro>
 	<xacro:macro name="side_usb_hand_system" params="side hand_type serial_port">
-		<xacro:property name="usb_hand_system_name" value="${str('linkerhand_7' if hand_type == 'linkerhand_o7' else ('inspire_e2' if hand_type in ('inspire_e2', 'inspire-e2') else 'linkerhand_6'))}"/>
+		<xacro:property name="usb_hand_system_name" value="${str('linkerhand_7' if hand_type == 'linkerhand_o7' else ('inspire_e2' if hand_type == 'inspire_e2' else 'linkerhand_6'))}"/>
 		<ros2_control name="${usb_hand_system_name}_${side}_system" type="system">
 			<hardware>
@@ -139,20 +139,20 @@
 		</ros2_control>
 		<xacro:if value="${left_drive_type == 'usb' or right_drive_type == 'usb' or left_drive_type == 'usb_can' or right_drive_type == 'usb_can'}">
-			<xacro:if value="${left_drive_type == 'usb' and left_hand_type in ('linkerhand_o6', 'linkerhand_l6', 'linkerhand_o7', 'inspire_e2', 'inspire-e2')}">
+			<xacro:if value="${left_drive_type == 'usb' and left_hand_type in ('linkerhand_o6', 'linkerhand_l6', 'linkerhand_o7', 'inspire_e2')}">
 				<xacro:side_usb_hand_system side="left" hand_type="${left_hand_type}" serial_port="/dev/ttyUSB0"/>
 			</xacro:if>
-			<xacro:if value="${right_drive_type == 'usb' and right_hand_type in ('linkerhand_o6', 'linkerhand_l6', 'linkerhand_o7', 'inspire_e2', 'inspire-e2')}">
+			<xacro:if value="${right_drive_type == 'usb' and right_hand_type in ('linkerhand_o6', 'linkerhand_l6', 'linkerhand_o7', 'inspire_e2')}">
 				<xacro:side_usb_hand_system side="right" hand_type="${right_hand_type}" serial_port="/dev/ttyUSB2"/>
 			</xacro:if>
-			<xacro:if value="${left_drive_type == 'usb' and left_hand_type in ('freedom_v1', 'freedom-v1')}">
+			<xacro:if value="${left_drive_type == 'usb' and left_hand_type == 'freedom_v1'}">
 				<xacro:side_freedom_usb_hand_system side="left" serial_port="/dev/ttyUSB0"/>
 			</xacro:if>
-			<xacro:if value="${right_drive_type == 'usb' and right_hand_type in ('freedom_v1', 'freedom-v1')}">
+			<xacro:if value="${right_drive_type == 'usb' and right_hand_type == 'freedom_v1'}">
 				<xacro:side_freedom_usb_hand_system side="right" serial_port="/dev/ttyUSB2"/>
 			</xacro:if>
-			<xacro:if value="${left_drive_type == 'usb_can' and left_hand_type in ('freedom_v1', 'freedom-v1')}">
+			<xacro:if value="${left_drive_type == 'usb_can' and left_hand_type == 'freedom_v1'}">
 				<xacro:side_freedom_usb_can_hand_system side="left" can_interface="can0" device_id="0"/>
 			</xacro:if>
-			<xacro:if value="${right_drive_type == 'usb_can' and right_hand_type in ('freedom_v1', 'freedom-v1')}">
+			<xacro:if value="${right_drive_type == 'usb_can' and right_hand_type == 'freedom_v1'}">
 				<xacro:side_freedom_usb_can_hand_system side="right" can_interface="can1" device_id="1"/>
 			</xacro:if>
