Commit message: 添加freedomv2

File: xacro/ros2_control/robot.xacro (robot description, xacro)
@@ -19,5 +19,6 @@
 	<xacro:include filename="$(find linkerhand_description)/xacro/ros2_control/o6.xacro"/>
 	<xacro:include filename="$(find linkerhand_description)/xacro/ros2_control/o7.xacro"/>
-	<xacro:include filename="$(find freedom_description)/xacro/ros2_control/freedom.xacro"/>
+	<xacro:include filename="$(find freedom_description)/xacro/ros2_control/freedomv1.xacro"/>
+	<xacro:include filename="$(find freedom_description)/xacro/ros2_control/freedomv2.xacro"/>
 	<xacro:include filename="$(find inspire_description)/xacro/ros2_control/RH56E2.xacro"/>
 	<xacro:macro name="side_gripper_joint" params="side">
@@ -45,4 +46,7 @@
 			<xacro:freedom_interfaces name="${side}_hand"/>
 		</xacro:if>
+		<xacro:if value="${hand_type == 'freedom_v2'}">
+			<xacro:freedomv2_interfaces name="${side}_hand"/>
+		</xacro:if>
 		<xacro:if value="${hand_type == 'inspire_e2'}">
 			<xacro:inspire_rh56e2_interfaces name="${side}_hand"/>
@@ -62,6 +66,6 @@
 		</ros2_control>
 	</xacro:macro>
-	<xacro:macro name="side_freedom_usb_hand_system" params="side serial_port">
-		<ros2_control name="freedom_v1_${side}_system" type="system">
+	<xacro:macro name="side_freedom_usb_hand_system" params="side serial_port hand_type:=freedom_v1 command_speed:=100">
+		<ros2_control name="${hand_type}_${side}_system" type="system">
 			<hardware>
 				<plugin>modbus_ros2_control/FreedomRS485Hardware</plugin>
@@ -70,8 +74,15 @@
 				<param name="slave_id">auto</param>
 				<param name="baudrate">115200</param>
+				<param name="protocol_version">${hand_type}</param>
+				<param name="command_speed">${command_speed}</param>
 				<param name="read_feedback">true</param>
 				<param name="feedback_timeout_ms">20</param>
 			</hardware>
-			<xacro:freedom_interfaces name="${side}_hand"/>
+			<xacro:if value="${hand_type == 'freedom_v2'}">
+				<xacro:freedomv2_interfaces name="${side}_hand"/>
+			</xacro:if>
+			<xacro:unless value="${hand_type == 'freedom_v2'}">
+				<xacro:freedom_interfaces name="${side}_hand"/>
+			</xacro:unless>
 		</ros2_control>
 	</xacro:macro>
@@ -146,8 +157,14 @@
 			</xacro:if>
 			<xacro:if value="${left_drive_type == 'usb' and left_hand_type == 'freedom_v1'}">
-				<xacro:side_freedom_usb_hand_system side="left" serial_port="/dev/ttyUSB0"/>
+				<xacro:side_freedom_usb_hand_system side="left" serial_port="/dev/ttyUSB0" hand_type="freedom_v1"/>
 			</xacro:if>
 			<xacro:if value="${right_drive_type == 'usb' and right_hand_type == 'freedom_v1'}">
-				<xacro:side_freedom_usb_hand_system side="right" serial_port="/dev/ttyUSB2"/>
+				<xacro:side_freedom_usb_hand_system side="right" serial_port="/dev/ttyUSB2" hand_type="freedom_v1"/>
+			</xacro:if>
+			<xacro:if value="${left_drive_type == 'usb' and left_hand_type == 'freedom_v2'}">
+				<xacro:side_freedom_usb_hand_system side="left" serial_port="/dev/ttyUSB0" hand_type="freedom_v2"/>
+			</xacro:if>
+			<xacro:if value="${right_drive_type == 'usb' and right_hand_type == 'freedom_v2'}">
+				<xacro:side_freedom_usb_hand_system side="right" serial_port="/dev/ttyUSB2" hand_type="freedom_v2"/>
 			</xacro:if>
 			<xacro:if value="${left_drive_type == 'usb_can' and left_hand_type == 'freedom_v1'}">

Commit message: add 120s

File: xacro/ros2_control/robot.xacro (robot description, xacro)
@@ -18,4 +18,5 @@
 	<xacro:include filename="$(find jodell_description)/xacro/ros2_control/RG75-300.xacro"/>
 	<xacro:include filename="$(find changingtek_description)/xacro/ros2_control/AG2F90-C.xacro"/>
+	<xacro:include filename="$(find changingtek_description)/xacro/ros2_control/AG2F120S.xacro"/>
 	<xacro:include filename="$(find linkerhand_description)/xacro/ros2_control/o6.xacro"/>
 	<xacro:include filename="$(find linkerhand_description)/xacro/ros2_control/o7.xacro"/>
@@ -33,4 +34,7 @@
 	<xacro:macro name="side_ag2f90_interfaces" params="side">
 		<xacro:ag2f90c_interfaces name="${side}"/>
+	</xacro:macro>
+	<xacro:macro name="side_ag2f120s_interfaces" params="side">
+		<xacro:ag2f120s_interfaces name="${side}"/>
 	</xacro:macro>
 	<xacro:macro name="side_hand_interfaces" params="side hand_type">
@@ -140,4 +144,10 @@
 				<xacro:side_ag2f90_interfaces side="right"/>
 			</xacro:if>
+			<xacro:if value="${left_gripper_type in ('ag2f120s', 'ag2f120s_d')}">
+				<xacro:side_ag2f120s_interfaces side="left"/>
+			</xacro:if>
+			<xacro:if value="${right_gripper_type in ('ag2f120s', 'ag2f120s_d')}">
+				<xacro:side_ag2f120s_interfaces side="right"/>
+			</xacro:if>
 			<xacro:if value="${left_hand_type != ''}">
 				<xacro:side_hand_interfaces side="left" hand_type="${left_hand_type}"/>

Commit message: refactor readme

File: xacro/ros2_control/robot.xacro (robot description, xacro)
@@ -3,154 +3,36 @@
 	<xacro:arg name="ros2_control_hardware_type" default="mock_components"/>
 	<xacro:arg name="arm_ctrl_mode" default="position"/>
+	<xacro:arg name="device_ip" default="192.168.1.190"/>
 	<xacro:arg name="left_ee_drive_type" default=""/>
 	<xacro:arg name="right_ee_drive_type" default=""/>
 	<xacro:arg name="left_dyn_param" default=""/>
 	<xacro:arg name="right_dyn_param" default=""/>
-	<!-- Marvin joint limits; override via robot.local.yaml hardware: or hardware_max_joint_*:= launch args -->
 	<xacro:arg name="max_joint_speed" default="50"/>
 	<xacro:arg name="max_joint_acceleration" default="30"/>
+	<xacro:arg name="usb_left_port" default="/dev/ttyUSB0"/>
+	<xacro:arg name="usb_right_port" default="/dev/ttyUSB2"/>
 	<xacro:property name="is_real_hardware" value="${'$(arg ros2_control_hardware_type)' == 'real' or '$(arg ros2_control_hardware_type)' == 'real_usb'}"/>
 	<xacro:property name="ee_drive_type" value="${'usb' if '$(arg ros2_control_hardware_type)' == 'real_usb' else ('marvin' if '$(arg ros2_control_hardware_type)' == 'real' else '')}"/>
 	<xacro:property name="left_drive_type" value="${'$(arg left_ee_drive_type)' if '$(arg left_ee_drive_type)' != '' else ee_drive_type}"/>
 	<xacro:property name="right_drive_type" value="${'$(arg right_ee_drive_type)' if '$(arg right_ee_drive_type)' != '' else ee_drive_type}"/>
-	<xacro:property name="arm_ctrl_mode_value" value="$(arg arm_ctrl_mode)"/>
-	<xacro:property name="left_ee_type" value="${left_hand_type if left_hand_type != '' else left_gripper_type}"/>
-	<xacro:property name="right_ee_type" value="${right_hand_type if right_hand_type != '' else right_gripper_type}"/>
 	<xacro:include filename="$(find fiveages_w2_description)/xacro/robot.xacro"/>
-	<xacro:include filename="$(find m6_ccs_description)/xacro/ros2_control/interfaces.xacro"/>
+	<xacro:include filename="$(find robot_common_launch)/xacro/ros2_control/simulation_hardware.xacro"/>
+	<xacro:include filename="$(find m6_ccs_description)/xacro/ros2_control/marvin_hardware.xacro"/>
+	<xacro:include filename="$(find m6_ccs_description)/xacro/ros2_control/end_effector_interfaces.xacro"/>
+	<xacro:include filename="$(find m6_ccs_description)/xacro/ros2_control/external_ee_systems.xacro"/>
 	<xacro:include filename="$(find fiveages_w2_common_description)/xacro/ros2_control/body.xacro"/>
-	<xacro:include filename="$(find jodell_description)/xacro/ros2_control/RG75-300.xacro"/>
-	<xacro:include filename="$(find changingtek_description)/xacro/ros2_control/AG2F90-C.xacro"/>
-	<xacro:include filename="$(find changingtek_description)/xacro/ros2_control/AG2F120S.xacro"/>
-	<xacro:include filename="$(find linkerhand_description)/xacro/ros2_control/o6.xacro"/>
-	<xacro:include filename="$(find linkerhand_description)/xacro/ros2_control/o7.xacro"/>
-	<xacro:include filename="$(find freedom_description)/xacro/ros2_control/freedomv1.xacro"/>
-	<xacro:include filename="$(find freedom_description)/xacro/ros2_control/freedomv2.xacro"/>
-	<xacro:include filename="$(find inspire_description)/xacro/ros2_control/RH56E2.xacro"/>
-	<xacro:include filename="$(find inspire_description)/xacro/ros2_control/side_systems.xacro"/>
-	<xacro:include filename="$(find xhand1_description)/xacro/ros2_control/side_systems.xacro"/>
-	<xacro:macro name="side_gripper_joint" params="side">
-		<joint name="${side}_gripper_joint">
-			<command_interface name="position"/>
-			<state_interface name="position">
-				<param name="initial_value">0</param>
-			</state_interface>
-		</joint>
-	</xacro:macro>
-	<xacro:macro name="side_rg75_interfaces" params="side">
-		<xacro:rg75_interfaces name="${side}"/>
-	</xacro:macro>
-	<xacro:macro name="side_ag2f90_interfaces" params="side">
-		<xacro:ag2f90c_interfaces name="${side}"/>
-	</xacro:macro>
-	<xacro:macro name="side_ag2f120s_interfaces" params="side">
-		<xacro:ag2f120s_interfaces name="${side}"/>
-	</xacro:macro>
-	<xacro:macro name="side_hand_interfaces" params="side hand_type">
-		<xacro:if value="${hand_type in ['linkerhand_o6', 'linkerhand_l6']}">
-			<xacro:linkerhand_o6_interfaces name="${side}_hand"/>
-		</xacro:if>
-		<xacro:if value="${hand_type == 'linkerhand_o7'}">
-			<xacro:linkerhand_o7_interfaces name="${side}_hand"/>
-		</xacro:if>
-		<xacro:if value="${hand_type == 'freedom_v1'}">
-			<xacro:freedom_interfaces name="${side}_hand"/>
-		</xacro:if>
-		<xacro:if value="${hand_type == 'freedom_v2'}">
-			<xacro:freedomv2_interfaces name="${side}_hand"/>
-		</xacro:if>
-		<xacro:if value="${hand_type == 'inspire_e2'}">
-			<xacro:inspire_rh56e2_interfaces name="${side}_hand"/>
-		</xacro:if>
-		<xacro:if value="${hand_type == 'xhand1'}">
-			<xacro:xhand1_interfaces name="${side}_hand"/>
-		</xacro:if>
-	</xacro:macro>
-	<xacro:macro name="side_usb_hand_system" params="side hand_type serial_port">
-		<xacro:property name="usb_hand_system_name" value="${str('linkerhand_7' if hand_type == 'linkerhand_o7' else ('inspire_e2' if hand_type == 'inspire_e2' else 'linkerhand_6'))}"/>
-		<ros2_control name="${usb_hand_system_name}_${side}_system" type="system">
-			<hardware>
-				<plugin>modbus_ros2_control/DexterousHandHardware</plugin>
-				<param name="serial_port">${serial_port}</param>
-				<param name="hand_type">${hand_type}</param>
-				<param name="hand_side">${side}</param>
-				<param name="max_speed_ratio">1.0</param>
-			</hardware>
-			<xacro:side_hand_interfaces side="${side}" hand_type="${hand_type}"/>
-		</ros2_control>
-	</xacro:macro>
-	<xacro:macro name="side_freedom_usb_hand_system" params="side serial_port hand_type:=freedom_v1 command_speed:=100">
-		<ros2_control name="${hand_type}_${side}_system" type="system">
-			<hardware>
-				<plugin>modbus_ros2_control/FreedomRS485Hardware</plugin>
-				<param name="serial_port">${serial_port}</param>
-				<param name="hand_side">${side}</param>
-				<param name="slave_id">auto</param>
-				<param name="baudrate">115200</param>
-				<param name="protocol_version">${hand_type}</param>
-				<param name="command_speed">${command_speed}</param>
-				<param name="read_feedback">true</param>
-				<param name="feedback_timeout_ms">20</param>
-			</hardware>
-			<xacro:if value="${hand_type == 'freedom_v2'}">
-				<xacro:freedomv2_interfaces name="${side}_hand"/>
-			</xacro:if>
-			<xacro:unless value="${hand_type == 'freedom_v2'}">
-				<xacro:freedom_interfaces name="${side}_hand"/>
-			</xacro:unless>
-		</ros2_control>
-	</xacro:macro>
-	<xacro:macro name="side_freedom_usb_can_hand_system" params="side can_interface device_id">
-		<ros2_control name="freedom_v1_${side}_can_system" type="system">
-			<hardware>
-				<plugin>can_ros2_control/FreedomCanHardware</plugin>
-				<param name="can_interface">${can_interface}</param>
-				<param name="device_id">${device_id}</param>
-				<param name="read_feedback">true</param>
-				<param name="feedback_timeout_ms">1</param>
-			</hardware>
-			<xacro:freedom_interfaces name="${side}_hand"/>
-		</ros2_control>
-	</xacro:macro>
 	<xacro:if value="${is_real_hardware}">
 		<ros2_control name="M6_CCS_System" type="system">
 			<hardware>
-				<plugin>marvin_ros2_control/MarvinHardware</plugin>
-				<param name="arm_type">dual</param>
-				<param name="ctrl_mode">${arm_ctrl_mode_value}</param>
-				<xacro:if value="${(left_drive_type == 'marvin' or left_drive_type == 'tianji_can') and left_ee_type != '' and left_ee_type != 'xhand1'}">
-					<param name="left_ee_type">${left_ee_type}</param>
-					<xacro:if value="${left_drive_type == 'tianji_can'}">
-						<param name="left_ee_channel">1</param>
-					</xacro:if>
-				</xacro:if>
-				<xacro:if value="${(right_drive_type == 'marvin' or right_drive_type == 'tianji_can') and right_ee_type != '' and right_ee_type != 'xhand1'}">
-					<param name="right_ee_type">${right_ee_type}</param>
-					<xacro:if value="${right_drive_type == 'tianji_can'}">
-						<param name="right_ee_channel">1</param>
-					</xacro:if>
-				</xacro:if>
-				<param name="max_joint_speed">$(arg max_joint_speed)</param>
-				<param name="max_joint_acceleration">$(arg max_joint_acceleration)</param>
-				<xacro:ee_dyn_param side="left" ee_key="${left_ee_type}" arg_val="$(arg left_dyn_param)"/>
-				<xacro:ee_dyn_param side="right" ee_key="${right_ee_type}" arg_val="$(arg right_dyn_param)"/>
-				<param name="device_ip">192.168.1.190</param>
+				<xacro:marvin_hardware_block
+					arm_type="dual"
+					arm_ctrl_mode="$(arg arm_ctrl_mode)"
+					max_joint_speed="$(arg max_joint_speed)"
+					max_joint_acceleration="$(arg max_joint_acceleration)"
+					device_ip="$(arg device_ip)"
+					left_dyn_param="$(arg left_dyn_param)"
+					right_dyn_param="$(arg right_dyn_param)"/>
 			</hardware>
-			<xacro:m6_interfaces name="left"/>
-			<xacro:m6_interfaces name="right"/>
-			<xacro:if value="${left_gripper_type != ''}">
-				<xacro:side_gripper_joint side="left"/>
-			</xacro:if>
-			<xacro:if value="${right_gripper_type != ''}">
-				<xacro:side_gripper_joint side="right"/>
-			</xacro:if>
-			<xacro:if value="${left_drive_type == 'marvin' or right_drive_type == 'marvin' or left_drive_type == 'tianji_can' or right_drive_type == 'tianji_can'}">
-				<xacro:if value="${(left_drive_type == 'marvin' or left_drive_type == 'tianji_can') and left_hand_type != '' and left_hand_type != 'xhand1'}">
-					<xacro:side_hand_interfaces side="left" hand_type="${left_hand_type}"/>
-				</xacro:if>
-				<xacro:if value="${(right_drive_type == 'marvin' or right_drive_type == 'tianji_can') and right_hand_type != '' and right_hand_type != 'xhand1'}">
-					<xacro:side_hand_interfaces side="right" hand_type="${right_hand_type}"/>
-				</xacro:if>
-			</xacro:if>
+			<xacro:dual_arm_ee_block mode="real"/>
 		</ros2_control>
 		<ros2_control name="juxie_body" type="system">
@@ -163,87 +45,15 @@
 			<xacro:body_interfaces/>
 		</ros2_control>
-		<xacro:if value="${left_drive_type == 'usb' or right_drive_type == 'usb' or left_drive_type == 'usb_can' or right_drive_type == 'usb_can'}">
-			<xacro:if value="${left_drive_type == 'usb' and left_hand_type in ('linkerhand_o6', 'linkerhand_l6', 'linkerhand_o7', 'inspire_e2')}">
-				<xacro:side_usb_hand_system side="left" hand_type="${left_hand_type}" serial_port="/dev/ttyUSB0"/>
-			</xacro:if>
-			<xacro:if value="${right_drive_type == 'usb' and right_hand_type in ('linkerhand_o6', 'linkerhand_l6', 'linkerhand_o7', 'inspire_e2')}">
-				<xacro:side_usb_hand_system side="right" hand_type="${right_hand_type}" serial_port="/dev/ttyUSB2"/>
-			</xacro:if>
-			<xacro:if value="${left_drive_type == 'usb' and left_hand_type == 'freedom_v1'}">
-				<xacro:side_freedom_usb_hand_system side="left" serial_port="/dev/ttyUSB0" hand_type="freedom_v1"/>
-			</xacro:if>
-			<xacro:if value="${right_drive_type == 'usb' and right_hand_type == 'freedom_v1'}">
-				<xacro:side_freedom_usb_hand_system side="right" serial_port="/dev/ttyUSB2" hand_type="freedom_v1"/>
-			</xacro:if>
-			<xacro:if value="${left_drive_type == 'usb' and left_hand_type == 'freedom_v2'}">
-				<xacro:side_freedom_usb_hand_system side="left" serial_port="/dev/ttyUSB0" hand_type="freedom_v2"/>
-			</xacro:if>
-			<xacro:if value="${right_drive_type == 'usb' and right_hand_type == 'freedom_v2'}">
-				<xacro:side_freedom_usb_hand_system side="right" serial_port="/dev/ttyUSB2" hand_type="freedom_v2"/>
-			</xacro:if>
-			<xacro:if value="${left_drive_type == 'usb' and left_hand_type == 'xhand1'}">
-				<xacro:xhand1_rs485_side_system side="left" serial_port="/dev/ttyUSB0"/>
-			</xacro:if>
-			<xacro:if value="${right_drive_type == 'usb' and right_hand_type == 'xhand1'}">
-				<xacro:xhand1_rs485_side_system side="right" serial_port="/dev/ttyUSB2"/>
-			</xacro:if>
-			<xacro:if value="${left_drive_type == 'usb_can' and left_hand_type == 'freedom_v1'}">
-				<xacro:side_freedom_usb_can_hand_system side="left" can_interface="can0" device_id="0"/>
-			</xacro:if>
-			<xacro:if value="${right_drive_type == 'usb_can' and right_hand_type == 'freedom_v1'}">
-				<xacro:side_freedom_usb_can_hand_system side="right" can_interface="can1" device_id="1"/>
-			</xacro:if>
-			<xacro:if value="${left_drive_type == 'usb_can' and left_hand_type == 'inspire_e2'}">
-				<xacro:inspire_canfd_side_system side="left" can_interface="can0"/>
-			</xacro:if>
-			<xacro:if value="${right_drive_type == 'usb_can' and right_hand_type == 'inspire_e2'}">
-				<xacro:inspire_canfd_side_system side="right" can_interface="can1"/>
-			</xacro:if>
-		</xacro:if>
+		<xacro:external_ee_systems
+			usb_left_port="$(arg usb_left_port)"
+			usb_right_port="$(arg usb_right_port)"/>
 	</xacro:if>
 	<xacro:unless value="${is_real_hardware}">
 		<ros2_control name="fiveages_w2_system" type="system">
 			<hardware>
-				<xacro:if value="${'$(arg ros2_control_hardware_type)' == 'gz'}">
-					<plugin>gz_ros2_control/GazeboSimSystem</plugin>
-				</xacro:if>
-				<xacro:if value="${'$(arg ros2_control_hardware_type)' == 'mock_components'}">
-					<plugin>mock_components/GenericSystem</plugin>
-				</xacro:if>
-				<xacro:if value="${'$(arg ros2_control_hardware_type)' == 'isaac'}">
-					<plugin>topic_based_ros2_control/TopicBasedSystem</plugin>
-					<param name="joint_commands_topic">/isaac/joint_command</param>
-					<param name="joint_states_topic">/isaac/joint_states</param>
-					<param name="sum_wrapped_joint_states">false</param>
-					<param name="initialize_commands_from_state">true</param>
-				</xacro:if>
+				<xacro:simulation_hardware_plugin hardware_type="$(arg ros2_control_hardware_type)"/>
 			</hardware>
 			<xacro:body_interfaces/>
-			<xacro:m6_interfaces name="left"/>
-			<xacro:m6_interfaces name="right"/>
-			<xacro:if value="${left_gripper_type == 'rg75'}">
-				<xacro:side_rg75_interfaces side="left"/>
-			</xacro:if>
-			<xacro:if value="${right_gripper_type == 'rg75'}">
-				<xacro:side_rg75_interfaces side="right"/>
-			</xacro:if>
-			<xacro:if value="${left_gripper_type in ('ag2f90_c', 'ag2f90_d')}">
-				<xacro:side_ag2f90_interfaces side="left"/>
-			</xacro:if>
-			<xacro:if value="${right_gripper_type in ('ag2f90_c', 'ag2f90_d')}">
-				<xacro:side_ag2f90_interfaces side="right"/>
-			</xacro:if>
-			<xacro:if value="${left_gripper_type in ('ag2f120s', 'ag2f120s_d')}">
-				<xacro:side_ag2f120s_interfaces side="left"/>
-			</xacro:if>
-			<xacro:if value="${right_gripper_type in ('ag2f120s', 'ag2f120s_d')}">
-				<xacro:side_ag2f120s_interfaces side="right"/>
-			</xacro:if>
-			<xacro:if value="${left_hand_type != ''}">
-				<xacro:side_hand_interfaces side="left" hand_type="${left_hand_type}"/>
-			</xacro:if>
-			<xacro:if value="${right_hand_type != ''}">
-				<xacro:side_hand_interfaces side="right" hand_type="${right_hand_type}"/>
-			</xacro:if>
+			<xacro:dual_arm_ee_block mode="sim"/>
 		</ros2_control>
 	</xacro:unless>
